Commit message: Wrong robotiq gripper

File: mara_description/urdf/mara_robot_camera_top.urdf (robot description, URDF)
Before this commit: robot mara, 24 links, 23 joints
Links:
- link left_inner_finger: geometry collision mesh filename=package://robotiq_arg2f_model_visualization/meshes/robotiq_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 scale=0.001 0.001 0.001; visual mesh filename=package://robotiq_arg2f_model_visualization/meshes/robotiq_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 scale=0.001 0.001 0.001
- link left_inner_knuckle: geometry visual mesh filename=package://robotiq_arg2f_model_visualization/meshes/robotiq_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
- link left_outer_finger: geometry collision mesh filename=package://robotiq_arg2f_model_visualization/meshes/robotiq_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; visual mesh filename=package://robotiq_arg2f_model_visualization/meshes/robotiq_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
- link left_outer_knuckle: geometry collision mesh filename=package://robotiq_arg2f_model_visualization/meshes/robotiq_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; visual mesh filename=package://robotiq_arg2f_model_visualization/meshes/robotiq_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
- link right_inner_finger: geometry collision mesh filename=package://robotiq_arg2f_model_visualization/meshes/robotiq_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 scale=0.001 0.001 0.001; visual mesh filename=package://robotiq_arg2f_model_visualization/meshes/robotiq_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 scale=0.001 0.001 0.001
- link right_inner_knuckle: geometry visual mesh filename=package://robotiq_arg2f_model_visualization/meshes/robotiq_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
- link right_outer_finger: geometry collision mesh filename=package://robotiq_arg2f_model_visualization/meshes/robotiq_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; visual mesh filename=package://robotiq_arg2f_model_visualization/meshes/robotiq_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
- link right_outer_knuckle: geometry collision mesh filename=package://robotiq_arg2f_model_visualization/meshes/robotiq_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; visual mesh filename=package://robotiq_arg2f_model_visualization/meshes/robotiq_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
- link robotiq_arg2f_base_link: geometry collision mesh filename=package://robotiq_arg2f_model_visualization/meshes/GRIPPER_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 scale=0.001 0.001 0.001; visual mesh filename=package://robotiq_arg2f_model_visualization/meshes/GRIPPER_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 scale=0.001 0.001 0.001
