Commit message: Rotating model 90º

File: mara_description/urdf/mara_robot_camera_top.urdf.xacro (robot description, xacro)
@@ -27,5 +27,5 @@
   </joint>
   <joint name="table_to_base_joint" type="fixed">
-    <origin rpy="0 0 0" xyz="0 0 0.62"/>
+    <origin rpy="0 0 -1.57" xyz="0 0 0.62"/>
     <parent link="table"/>
     <child link="base_link"/>

Commit message: Adding gripper to the model

File: mara_description/urdf/mara_robot_camera_top.urdf.xacro (robot description, xacro)
@@ -7,18 +7,16 @@
   <xacro:include filename="$(find mara_description)/urdf/mara.urdf.xacro" />
   <!-- robotiq 140 gripper -->
-  <!-- <xacro:include filename="$(find robotiq_arg2f_model_visualization)/urdf/robotiq_gripper.urdf.xacro" /> -->
-  <!-- <xacro:include filename="$(find mara_description)/urdf/camera_top.urdf.xacro" /> -->
+  <xacro:include filename="$(find robotiq_arg2f_model_visualization)/urdf/robotiq_arg2f_140_model_macro.xacro" />
   <xacro:include filename="$(find mara_description)/urdf/table.urdf.xacro" />
   <!-- arm -->
   <xacro:mara_robot prefix="" joint_limited="false"/>
-  <!-- <xacro:robotiq_gripper prefix="" /> -->
-  <!-- <xacro:mara_camera_top prefix="" /> -->
+  <xacro:robotiq_arg2f_140 prefix="" />
   <xacro:table prefix="" />
   <link name="world" />
-  <!-- <joint name="end_effector_adapter_to_robotiq" type="fixed">
+  <joint name="end_effector_adapter_to_robotiq" type="fixed">
     <origin rpy="0 0 1.57" xyz=" 0 0 0.04659"/>
     <parent link="motor6_link"/>
     <child link="robotiq_arg2f_base_link"/>
-  </joint> -->
+  </joint>
   <joint name="world_to_table_joint" type="fixed">
     <origin rpy="0 0 0" xyz="0 0 0.02"/>

File: robotiq_arg2f_model_visualization/urdf/robotiq_arg2f_140_model_macro.xacro (robot description, xacro)
@@ -1,45 +1,39 @@
 <?xml version="1.0"?>
 <robot xmlns:xacro="http://ros.org/wiki/xacro">
-  <xacro:include filename="$(find robotiq_arg2f_model_visualization)/urdf/robotiq_arg2f_transmission.xacro" />
-  <xacro:macro name="riser">
-    <link name="riser">
-      <origin xyz="-0.15 1.0 0.5" rpy="0 0 0" />
-      <inertial>
-        <origin xyz="0 0 -0.5" rpy="0 0 0" />
-        <mass value="1000.0" />
-        <inertia
-            ixx="0.01"
-            ixy="0.0"
-            ixz="0.0"
-            iyy="0.01"
-            iyz="0.0"
-            izz="0.01" />
-      </inertial>
-      <visual>
-        <origin xyz="0 0 0" rpy="0 0 0" />
-        <geometry>
-          <box size="0.2 0.2 0.1" />
-        </geometry>
-        <material name="">
-          <color rgba="0.792156862745098 0.819607843137255 0.933333333333333 1" />
-        </material>
-      </visual>
-      <collision>
-        <origin xyz="0 0 0" rpy="0 0 0" />
-        <geometry>
-          <box size="0.2 0.2 0.1" />
-        </geometry>
-      </collision>
-    </link>
-  </xacro:macro>
-  <xacro:macro name="outer_knuckle" params="prefix fingerprefix stroke">
-    <link name="${prefix}${fingerprefix}_outer_knuckle">
-      <inertial>
-        <origin xyz="-0.000200000000003065 0.0199435877845359 0.0292245259211331" rpy="0 0 0" />
+  <xacro:macro name="robotiq_arg2f_140"  params="prefix">
+    <link name="robotiq_arg2f_base_link">
+      <inertial>
+        <origin xyz="8.625E-08 -4.6583E-06 0.03145" rpy="0 0 0" />
+        <mass value="0.22652" />
+        <inertia ixx="0.00020005" ixy="0" ixz="0" iyy="0.00017832" iyz="0" izz="0.00013478" />
+      </inertial>
+      <visual>
+        <origin xyz="0 0 0" rpy="0 0 1.57" />
+        <geometry>
+          <mesh filename="package://robotiq_arg2f_model_visualization/meshes/GRIPPER_base_axis.stl" scale="0.001 0.001 0.001"/>
+        </geometry>
+        <material name="">
+          <color rgba="0.1 0.1 0.1 1" />
+        </material>
+      </visual>
+      <collision>
+        <origin xyz="0 0 0" rpy="0 0 1.57" />
+        <geometry>
+          <mesh filename="package://robotiq_arg2f_model_visualization/meshes/GRIPPER_base_axis.stl" scale="0.001 0.001 0.001"/>
+        </geometry>
+      </collision>
+    </link>
+    <gazebo reference="robotiq_arg2f_base_link">
+      <material>Gazebo/Grey</material>
+      <selfCollide>True</selfCollide>
+    </gazebo>
+    <link name="left_outer_knuckle">
+      <inertial>
+        <origin xyz="0 0 0" rpy="0 0 0" />
         <mass value="0.00853198276973456" />
         <inertia
             ixx="2.89328108496468E-06"
-            ixy="-1.57935047237397E-19"
-            ixz="-1.93980378593255E-19"
+            ixy="0"
+            ixz="0"
             iyy="1.86719750325683E-06"
             iyz="-1.21858577871576E-06"
@@ -49,5 +43,5 @@
         <origin xyz="0 0 0" rpy="0 0 0" />
         <geometry>
-          <mesh filename="package://robotiq_arg2f_model_visualization/meshes/robotiq_arg2f_${stroke}_outer_knuckle.stl" />
+          <mesh filename="package://robotiq_arg2f_model_visualization/meshes/robotiq_140_left_outer_knuckle.stl" />
         </geometry>
         <material name="">
@@ -58,11 +52,161 @@
         <origin xyz="0 0 0" rpy="0 0 0" />
         <geometry>
-          <mesh filename="package://robotiq_arg2f_model_visualization/meshes/robotiq_arg2f_${stroke}_outer_knuckle.stl" />
-        </geometry>
-      </collision>
-    </link>
-  </xacro:macro>
-  <xacro:macro name="outer_finger" params="prefix fingerprefix stroke">
-    <link name="${prefix}${fingerprefix}_outer_finger">
+          <mesh filename="package://robotiq_arg2f_model_visualization/meshes/robotiq_140_left_outer_knuckle.stl" />
+        </geometry>
+      </collision>
+    </link>
+    <gazebo reference="left_outer_knuckle">
+      <material>Gazebo/Grey</material>
+      <selfCollide>True</selfCollide>
+    </gazebo>
+    <link name="right_outer_knuckle">
+      <inertial>
+        <origin xyz="0 0 0" rpy="0 0 0" />
+        <mass value="0.00853198276973456" />
+        <inertia
+            ixx="2.89328108496468E-06"
+            ixy="0"
+            ixz="0"
+            iyy="1.86719750325683E-06"
+            iyz="-1.21858577871576E-06"
+            izz="1.21905238907251E-06" />
+      </inertial>
+      <visual>
+        <origin xyz="0 0 0" rpy="0 0 0" />
+        <geometry>
+          <mesh filename="package://robotiq_arg2f_model_visualization/meshes/robotiq_140_right_outer_knuckle.stl" />
+        </geometry>
+        <material name="">
+          <color rgba="0.792156862745098 0.819607843137255 0.933333333333333 1" />
+        </material>
+      </visual>
+      <collision>
+        <origin xyz="0 0 0" rpy="0 0 0" />
+        <geometry>
+          <mesh filename="package://robotiq_arg2f_model_visualization/meshes/robotiq_140_right_outer_knuckle.stl" />
+        </geometry>
+      </collision>
+    </link>
+    <gazebo reference="right_outer_knuckle">
+      <material>Gazebo/Grey</material>
+      <selfCollide>True</selfCollide>
+    </gazebo>
+    <link name="left_inner_knuckle">
+      <inertial>
+        <origin xyz="0.000123011831763771 0.0507850843201817 0.00103968640075166" rpy="0 0 0" />
+        <mass value="0.0271177346495152" />
+        <inertia
+            ixx="2.61910379223783E-05"
+            ixy="-2.43616858946494E-07"
+            ixz="-6.37789906117123E-09"
+            iyy="2.8270243746167E-06"
+            iyz="-5.37200748039765E-07"
+            izz="2.83695868220296E-05" />
+      </inertial>
+      <visual>
+        <origin xyz="0 0 0" rpy="0 0 0" />
+        <geometry>
+          <mesh filename="package://robotiq_arg2f_model_visualization/meshes/robotiq_140_left_inner_knuckle.stl" />
+        </geometry>
+        <material name="">
+          <color rgba="0.1 0.1 0.1 1" />
+        </material>
+      </visual>
+    </link>
+    <gazebo reference="left_inner_knuckle">
+      <material>Gazebo/Grey</material>
+      <selfCollide>True</selfCollide>
+    </gazebo>
+    <link name="right_inner_knuckle">
+      <inertial>
+        <origin xyz="0.000123011831763771 0.0507850843201817 0.00103968640075166" rpy="0 0 0" />
+        <mass value="0.0271177346495152" />
+        <inertia
+            ixx="2.61910379223783E-05"
+            ixy="-2.43616858946494E-07"
+            ixz="-6.37789906117123E-09"
+            iyy="2.8270243746167E-06"
+            iyz="-5.37200748039765E-07"
+            izz="2.83695868220296E-05" />
+      </inertial>
+      <visual>
+        <origin xyz="0 0 0" rpy="0 0 0" />
+        <geometry>
+          <mesh filename="package://robotiq_arg2f_model_visualization/meshes/robotiq_140_right_inner_knuckle.stl" />
+        </geometry>
+        <material name="">
+          <color rgba="0.1 0.1 0.1 1" />
+        </material>
+      </visual>
+    </link>
+    <gazebo reference="right_inner_knuckle">
+      <material>Gazebo/Grey</material>
+      <selfCollide>True</selfCollide>
+    </gazebo>
+    <link name="left_inner_finger">
+      <inertial>
+        <origin xyz="0.0 0.031506174 -0.017648840" rpy="0 0 0" />
+        <mass value="0.0104003125914103" />
+        <inertia
+            ixx="6.06863499e-06"
+            ixy="0"
+            ixz="0"
+            iyy="7.46305064e-07"
+            iyz="0"
+            izz="6.21796490e-06" />
+      </inertial>
+      <visual>
+        <origin xyz="0 0 0" rpy="0 0 0" />
+        <geometry>
+          <mesh filename="package://robotiq_arg2f_model_visualization/meshes/robotiq_140_left_inner_finger.stl" scale="0.001 0.001 0.001" />
+        </geometry>
+        <material name="">
+          <color rgba="0.1 0.1 0.1 1" />
+        </material>
+      </visual>
+      <collision>
+        <origin xyz="0 0 0" rpy="0 0 0" />
+        <geometry>
+          <mesh filename="package://robotiq_arg2f_model_visualization/meshes/robotiq_140_left_inner_finger.stl" scale="0.001 0.001 0.001" />
+        </geometry>
+      </collision>
+    </link>
+    <gazebo reference="left_inner_finger">
+      <material>Gazebo/Grey</material>
+      <selfCollide>True</selfCollide>
+    </gazebo>
+    <link name="right_inner_finger">
+      <inertial>
+        <origin xyz="0.0 0.031506174 -0.017648840" rpy="0 0 0" />
+        <mass value="0.0104003125914103" />
+        <inertia
+            ixx="6.06863499e-06"
+            ixy="0"
+            ixz="0"
+            iyy="7.46305064e-07"
+            iyz="0"
+            izz="6.21796490e-06" />
+      </inertial>
+      <visual>
+        <origin xyz="0 0 0" rpy="0 0 0" />
+        <geometry>
+          <mesh filename="package://robotiq_arg2f_model_visualization/meshes/robotiq_140_right_inner_finger.stl" scale="0.001 0.001 0.001"/>
+        </geometry>
+        <material name="">
+          <color rgba="0.1 0.1 0.1 1" />
+        </material>
+      </visual>
+      <collision>
+        <origin xyz="0 0 0" rpy="0 0 0" />
+        <geometry>
+          <mesh filename="package://robotiq_arg2f_model_visualization/meshes/robotiq_140_right_inner_finger.stl" scale="0.001 0.001 0.001"/>
+        </geometry>
+      </collision>
+    </link>
+    <gazebo reference="right_inner_finger">
+      <material>Gazebo/Grey</material>
+      <selfCollide>True</selfCollide>
+    </gazebo>
+    <link name="left_outer_finger">
       <inertial>
         <origin xyz="0.00030115855001899 0.0373907951953854 -0.0208027427000385" rpy="0 0 0" />
@@ -79,164 +223,140 @@
         <origin xyz="0 0 0" rpy="0 0 0" />
         <geometry>
-          <mesh filename="package://robotiq_arg2f_model_visualization/meshes/robotiq_arg2f_${stroke}_outer_finger.stl" />
-        </geometry>
-        <material name="">
-          <color rgba="0.1 0.1 0.1 1" />
-        </material>
-      </visual>
-      <collision>
-        <origin xyz="0 0 0" rpy="0 0 0" />
-        <geometry>
-          <mesh filename="package://robotiq_arg2f_model_visualization/meshes/robotiq_arg2f_${stroke}_outer_finger.stl" />
-        </geometry>
-      </collision>
-    </link>
-  </xacro:macro>
-  <xacro:macro name="inner_knuckle" params="prefix fingerprefix stroke">
-    <link name="${prefix}${fingerprefix}_inner_knuckle">
-      <inertial>
-        <origin xyz="0.000123011831763771 0.0507850843201817 0.00103968640075166" rpy="0 0 0" />
-        <mass value="0.0271177346495152" />
-        <inertia
-            ixx="2.61910379223783E-05"
-            ixy="-2.43616858946494E-07"
-            ixz="-6.37789906117123E-09"
-            iyy="2.8270243746167E-06"
-            iyz="-5.37200748039765E-07"
-            izz="2.83695868220296E-05" />
-      </inertial>
-      <visual>
-        <origin xyz="0 0 0" rpy="0 0 0" />
-        <geometry>
-          <mesh filename="package://robotiq_arg2f_model_visualization/meshes/robotiq_arg2f_${stroke}_inner_knuckle.stl" />
-        </geometry>
-        <material name="">
-          <color rgba="0.1 0.1 0.1 1" />
-        </material>
-      </visual>
-      <collision>
-        <origin xyz="0 0 0" rpy="0 0 0" />
-        <geometry>
-          <mesh filename="package://robotiq_arg2f_model_visualization/meshes/robotiq_arg2f_${stroke}_inner_knuckle.stl" />
-        </geometry>
-      </collision>
-    </link>
-  </xacro:macro>
-  <xacro:macro name="inner_finger" params="prefix fingerprefix stroke">
-    <link name="${prefix}${fingerprefix}_inner_finger">
-      <inertial>
-        <origin xyz="0.000299999999999317 0.0160078233491243 -0.0136945669206257" rpy="0 0 0" />
-        <mass value="0.0104003125914103" />
-        <inertia
-            ixx="2.71909453810972E-06"
-            ixy="1.35402465472579E-21"
-            ixz="-7.1817349065269E-22"
-            iyy="7.69100314106116E-07"
-            iyz="6.74715432769696E-07"
-            izz="2.30315190420171E-06" />
-      </inertial>
-      <visual>
-        <origin xyz="0 0 0" rpy="0 0 0" />
-        <geometry>
-          <mesh filename="package://robotiq_arg2f_model_visualization/meshes/robotiq_arg2f_${stroke}_inner_finger.stl" />
-        </geometry>
-        <material name="">
-          <color rgba="0.1 0.1 0.1 1" />
-        </material>
-      </visual>
-      <collision>
-        <origin xyz="0 0 0" rpy="0 0 0" />
-        <geometry>
-          <mesh filename="package://robotiq_arg2f_model_visualization/meshes/robotiq_arg2f_${stroke}_inner_finger.stl" />
-        </geometry>
-      </collision>
-    </link>
-  </xacro:macro>
-  <xacro:macro name="outer_finger_joint" params="prefix fingerprefix">
-    <joint name="${prefix}${fingerprefix}_outer_finger_joint" type="fixed">
+          <mesh filename="package://robotiq_arg2f_model_visualization/meshes/robotiq_140_left_outer_finger.stl" />
+        </geometry>
+        <material name="">
+          <color rgba="0.1 0.1 0.1 1" />
+        </material>
+      </visual>
+      <collision>
+        <origin xyz="0 0 0" rpy="0 0 0" />
+        <geometry>
+          <mesh filename="package://robotiq_arg2f_model_visualization/meshes/robotiq_140_left_outer_finger.stl" />
+        </geometry>
+      </collision>
+    </link>
+    <gazebo reference="left_outer_finger">
+      <material>Gazebo/Grey</material>
+      <selfCollide>True</selfCollide>
+    </gazebo>
+    <link name="right_outer_finger">
+      <inertial>
+        <origin xyz="0.00030115855001899 0.0373907951953854 -0.0208027427000385" rpy="0 0 0" />
+        <mass value="0.022614240507152" />
+        <inertia
+            ixx="1.52518312458174E-05"
+            ixy="9.76583423954399E-10"
+            ixz="-5.43838577022588E-10"
+            iyy="6.17694243867776E-06"
+            iyz="6.78636130740228E-06"
+            izz="1.16494917907219E-05" />
+      </inertial>
+      <visual>
+        <origin xyz="0 0 0" rpy="0 0 0" />
+        <geometry>
+          <mesh filename="package://robotiq_arg2f_model_visualization/meshes/robotiq_140_right_outer_finger.stl" />
+        </geometry>
+        <material name="">
+          <color rgba="0.1 0.1 0.1 1" />
+        </material>
+      </visual>
+      <collision>
+        <origin xyz="0 0 0" rpy="0 0 0" />
+        <geometry>
+          <mesh filename="package://robotiq_arg2f_model_visualization/meshes/robotiq_140_right_outer_finger.stl" />
+        </geometry>
+      </collision>
+    </link>
+    <gazebo reference="right_outer_finger">
+      <material>Gazebo/Grey</material>
+      <selfCollide>True</selfCollide>
+    </gazebo>
+    <joint name="left_outer_knuckle_joint" type="revolute">
+      <origin xyz="0 -0.030601 0.054905" rpy="2.31 0 0" />
+      <parent link="robotiq_arg2f_base_link" />
+      <child link="left_outer_knuckle" />
+      <axis xyz="-1 0 0" />
+      <limit lower="0" upper="0.875"  velocity="2.0" effort="1000" />
+    </joint>
+    <joint name="right_outer_knuckle_joint" type="revolute">
+      <origin xyz="0 0.030601 0.054905" rpy="2.31 0 3.14159265359" />
+      <parent link="robotiq_arg2f_base_link" />
+      <child link="right_outer_knuckle" />
+      <axis xyz="-1 0 0" />
+      <limit lower="0" upper="0.875" velocity="2.0" effort="1000" />
+    </joint>
+    <joint name="left_inner_knuckle_joint" type="revolute">
+      <origin xyz="0 -0.0127 0.06142" rpy="2.29 0 0" />
+      <parent link="robotiq_arg2f_base_link" />
+      <child link="left_inner_knuckle" />
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
Commit message: fix urdf

File: mara_description/urdf/mara_robot_camera_top.urdf.xacro (robot description, xacro)
@@ -7,13 +7,13 @@
   <xacro:include filename="$(find mara_description)/urdf/mara.urdf.xacro" />
   <!-- robotiq 140 gripper -->
-  <xacro:include filename="$(find robotiq_arg2f_model_visualization)/urdf/robotiq_arg2f_140_model_macro.xacro" />
+  <xacro:include filename="$(find robotiq_140_gripper_description)/urdf/robotiq_140.urdf.xacro" />
   <xacro:include filename="$(find mara_description)/urdf/table.urdf.xacro" />
   <!-- arm -->
-  <xacro:mara_robot prefix="" joint_limited="false"/>
-  <xacro:robotiq_arg2f_140 prefix="" />
+  <xacro:mara_robot prefix="" ee_link_distance="0.24"/>
+  <xacro:robotiq_gripper prefix="" />
   <xacro:table prefix="" />
   <link name="world" />
   <joint name="end_effector_adapter_to_robotiq" type="fixed">
-    <origin rpy="0 0 1.57" xyz=" 0 0 0.04659"/>
+    <origin rpy="0 0 1.57" xyz=" 0 0 0.0353"/>
     <parent link="motor6_link"/>
     <child link="robotiq_arg2f_base_link"/>
