Commit message: Adding new adpater and updating gimatic

File: mara_description/urdf/mara_robot_gripper_ur_j.urdf.xacro (robot description, xacro)
@@ -15,5 +15,5 @@
   <link name="world" />
   <joint name="end_effector_adapter_to_robotiq" type="fixed">
-    <origin rpy="0 0 0" xyz=" 0 0 0.03653"/>
+    <origin rpy="0 0 0" xyz=" 0 0 0.0"/>
     <parent link="motor6_link"/>
     <child link="body"/>
