Commit message: Updating robotiq URDFs

File: mara_description/urdf/mara_robot_gripper_140.urdf.xacro (robot description, xacro)
@@ -4,15 +4,20 @@
   <!-- common stuff -->
   <xacro:include filename="$(find mara_description)/urdf/mara_gazebo.urdf.xacro" />
+  <!-- mara -->
   <xacro:include filename="$(find mara_description)/urdf/mara.urdf.xacro" />
+  <!-- robotiq 140 gripper -->
   <xacro:include filename="$(find robotiq_140_gripper_description)/urdf/robotiq_140.urdf.xacro" />
+  <!-- <xacro:include filename="$(find mara_description)/urdf/camera_top.urdf.xacro" /> -->
   <xacro:include filename="$(find mara_description)/urdf/table.urdf.xacro" />
+  <!-- arm -->
   <xacro:mara_robot prefix="" ee_link_distance="0.24"/>
   <xacro:robotiq_gripper prefix="mara" />
+  <!-- <xacro:mara_camera_top prefix="" /> -->
   <xacro:table prefix="" />
   <link name="world" />
   <joint name="end_effector_adapter_to_robotiq" type="fixed">
-    <origin rpy="0 0 1.57" xyz=" 0 0 0.0353"/>
+    <origin rpy="0 0 1.57" xyz=" 0 0 0.0"/>
     <parent link="motor6_link"/>
-    <child link="robotiq_arg2f_base_link"/>
+    <child link="robotiq_adapter_link"/>
   </joint>
   <joint name="world_to_table_joint" type="fixed">

File: mara_description/urdf/mara_robot_gripper_85.urdf.xacro (robot description, xacro)
@@ -15,7 +15,7 @@
   <link name="world" />
   <joint name="end_effector_adapter_to_robotiq" type="fixed">
-    <origin rpy="0 0 0" xyz=" 0 0 0.03653"/>
+    <origin rpy="0 0 0" xyz=" 0 0 0.0"/>
     <parent link="motor6_link"/>
-    <child link="robotiq_arg2f_base"/>
+    <child link="robotiq_adapter_link"/>
   </joint>
   <joint name="world_to_table_joint" type="fixed">

File: mara_description/urdf/mara_robot_gripper_hande.urdf.xacro (robot description, xacro)
@@ -15,7 +15,7 @@
   <link name="world" />
   <joint name="end_effector_adapter_to_robotiq" type="fixed">
-    <origin rpy="0 1.57 0" xyz=" 0 0 0.13"/>
+    <origin rpy="0 0 0" xyz=" 0 0 0.0"/>
     <parent link="motor6_link"/>
-    <child link="robotiq_hande_base_link"/>
+    <child link="robotiq_adapter_link"/>
   </joint>
   <joint name="world_to_table_joint" type="fixed">

File: robotiq_140_gripper_description/urdf/robotiq_140.urdf.xacro (robot description, xacro)
@@ -2,4 +2,35 @@
 <robot xmlns:xacro="http://ros.org/wiki/xacro">
   <xacro:macro name="robotiq_gripper"  params="prefix">
+    <link name="robotiq_adapter_link">
+      <inertial>
+        <origin xyz="8.625E-08 -4.6583E-06 0.03145" rpy="0 0 0" />
+        <mass value="0.22652" />
+        <inertia ixx="0.00020005" ixy="0" ixz="0" iyy="0.00017832" iyz="0" izz="0.00013478" />
+      </inertial>
+      <visual>
+        <origin xyz="0 0 0" rpy="0 0 1.57" />
+        <geometry>
+          <mesh filename="package://robotiq_140_gripper_description/meshes/hros_robotiq_adapter.dae" scale="0.001 0.001 0.001"/>
+        </geometry>
+        <material name="Gazebo/Black">
+          <color rgba="0.0 0.0 0.0 1" />
+        </material>
+      </visual>
+      <collision>
+        <origin xyz="0 0 0" rpy="0 0 1.57" />
+        <geometry>
+          <mesh filename="package://robotiq_140_gripper_description/meshes/hros_robotiq_adapter.dae" scale="0.001 0.001 0.001"/>
+        </geometry>
+      </collision>
+    </link>
+    <gazebo reference="robotiq_adapter_link">
+      <material>Gazebo/Black</material>
+      <selfCollide>False</selfCollide>
+    </gazebo>
+    <joint name="base_adapter_to_base_robotiq_joint" type="fixed">
+      <origin rpy="0 0 0" xyz=" 0 0 0.03653"/>
+      <parent link="robotiq_adapter_link" />
+      <child link="robotiq_arg2f_base_link"/>
+    </joint>
     <link name="robotiq_arg2f_base_link">
       <inertial>
@@ -358,4 +389,10 @@
         </axis>
       </joint>
+      <plugin filename="librobotiq_gripper_gazebo_plugin.so" name="robotiq_140_gripper">
+        <joint>left_inner_knuckle_joint</joint>
+        <joint>left_outer_knuckle_joint</joint>
+        <joint>right_inner_knuckle_joint</joint>
+        <joint>joint_finger</joint>
+      </plugin>
     </gazebo>
   </xacro:macro>

File: robotiq_85_gripper_description/urdf/robotiq_85.urdf.xacro (robot description, xacro)
@@ -2,4 +2,35 @@
 <robot xmlns:xacro="http://ros.org/wiki/xacro">
   <xacro:macro name="robotiq_85"  params="prefix">
+    <link name="robotiq_adapter_link">
+      <inertial>
+        <origin xyz="8.625E-08 -4.6583E-06 0.03145" rpy="0 0 0" />
+        <mass value="0.22652" />
+        <inertia ixx="0.00020005" ixy="0" ixz="0" iyy="0.00017832" iyz="0" izz="0.00013478" />
+      </inertial>
+      <visual>
+        <origin xyz="0 0 0" rpy="0 0 1.57" />
+        <geometry>
+          <mesh filename="package://robotiq_85_gripper_description/meshes/hros_robotiq_adapter.dae" scale="0.001 0.001 0.001"/>
+        </geometry>
+        <material name="Gazebo/Black">
+          <color rgba="0.0 0.0 0.0 1" />
+        </material>
+      </visual>
+      <collision>
+        <origin xyz="0 0 0" rpy="0 0 1.57" />
+        <geometry>
+          <mesh filename="package://robotiq_85_gripper_description/meshes/hros_robotiq_adapter.dae" scale="0.001 0.001 0.001"/>
+        </geometry>
+      </collision>
+    </link>
+    <gazebo reference="robotiq_adapter_link">
+      <material>Gazebo/Black</material>
+      <selfCollide>False</selfCollide>
+    </gazebo>
+    <joint name="base_adapter_to_base_robotiq_joint" type="fixed">
+      <origin rpy="0 0 0" xyz=" 0 0 0.03653"/>
+      <parent link="robotiq_adapter_link" />
+      <child link="robotiq_arg2f_base"/>
+    </joint>
     <link name="robotiq_arg2f_base">
       <inertial>
@@ -322,4 +353,10 @@
         </axis>
       </joint>
+      <plugin filename="librobotiq_gripper_gazebo_plugin.so" name="robotiq_85_gripper">
+        <joint>left_inner_knuckle_joint</joint>
+        <joint>left_outer_knuckle_joint</joint>
+        <joint>right_inner_knuckle_joint</joint>
+        <joint>joint_finger</joint>
+      </plugin>
     </gazebo>
   </xacro:macro>

File: robotiq_hande_gripper_description/urdf/robotiq_hande.urdf.xacro (robot description, xacro)
@@ -2,4 +2,30 @@
 <robot xmlns:xacro="http://ros.org/wiki/xacro">
   <xacro:macro name="robotiq_hande"  params="prefix">
+    <link name="robotiq_adapter_link">
+      <inertial>
+        <origin xyz="8.625E-08 -4.6583E-06 0.03145" rpy="0 0 0" />
+        <mass value="0.22652" />
+        <inertia ixx="0.00020005" ixy="0" ixz="0" iyy="0.00017832" iyz="0" izz="0.00013478" />
+      </inertial>
+      <visual>
+        <origin xyz="0 0 0" rpy="0 0 1.57" />
+        <geometry>
+          <mesh filename="package://robotiq_hande_gripper_description/meshes/hros_robotiq_adapter.dae" scale="0.001 0.001 0.001"/>
+        </geometry>
+        <material name="Gazebo/Black">
+          <color rgba="0.0 0.0 0.0 1" />
+        </material>
+      </visual>
+      <collision>
+        <origin xyz="0 0 0" rpy="0 0 1.57" />
+        <geometry>
+          <mesh filename="package://robotiq_hande_gripper_description/meshes/hros_robotiq_adapter.dae" scale="0.001 0.001 0.001"/>
+        </geometry>
+      </collision>
+    </link>
+    <gazebo reference="robotiq_adapter_link">
+      <material>Gazebo/Black</material>
+      <selfCollide>False</selfCollide>
+    </gazebo>
     <link name="robotiq_hande_base_link">
       <inertial>
@@ -81,9 +107,17 @@
     </gazebo>
     <gazebo>
-      <plugin filename="librobotiq_linear_gripper_gazebo_plugin.so" name="robotiq_hande_gripper">
-        <left_joint>joint_finger</left_joint>
-        <right_joint>finger2_joint</right_joint>
+      <plugin filename="librobotiq_gripper_gazebo_plugin.so" name="robotiq_hande_gripper">
+        <kp>10</kp>
+        <ki>3</ki>
+        <kd>5</kd>
+        <joint>joint_finger</joint>
+        <joint>finger2_joint</joint>
       </plugin>
     </gazebo>
+    <joint name="base_adapter_to_base_robotiq_joint" type="fixed">
+      <origin rpy="0 1.57 0" xyz=" 0 0 0.10653"/>
+      <parent link="robotiq_adapter_link" />
+      <child link="robotiq_hande_base_link"/>
+    </joint>
     <joint name="joint_finger" type="prismatic">
       <origin rpy="0 0 0" xyz="0 0 0.0"/>

Commit message: fixing the rotation between the robot and the base

File: mara_description/urdf/mara_robot_gripper_140.urdf.xacro (robot description, xacro)
@@ -27,5 +27,5 @@
   </joint>
   <joint name="table_to_base_joint" type="fixed">
-    <origin rpy="0 0 1.57" xyz="0 0 0.62"/>
+    <origin rpy="0 0 0" xyz="0 0 0.62"/>
     <parent link="table"/>
     <child link="base_link"/>

File: mara_description/urdf/mara_robot_gripper_85.urdf.xacro (robot description, xacro)
@@ -25,5 +25,5 @@
   </joint>
   <joint name="table_to_base_joint" type="fixed">
-    <origin rpy="0 0 1.57" xyz="0 0 0.62"/>
+    <origin rpy="0 0 0" xyz="0 0 0.62"/>
     <parent link="table"/>
     <child link="base_link"/>

File: mara_description/urdf/mara_robot_gripper_hande.urdf.xacro (robot description, xacro)
@@ -25,5 +25,5 @@
   </joint>
   <joint name="table_to_base_joint" type="fixed">
-    <origin rpy="0 0 1.57" xyz="0 0 0.62"/>
+    <origin rpy="0 0 0" xyz="0 0 0.62"/>
     <parent link="table"/>
     <child link="base_link"/>

File: mara_description/urdf/mara_robot_gripper_ur_j.urdf.xacro (robot description, xacro)
@@ -25,5 +25,5 @@
   </joint>
   <joint name="table_to_base_joint" type="fixed">
-    <origin rpy="0 0 1.57" xyz="0 0 0.62"/>
+    <origin rpy="0 0 0" xyz="0 0 0.62"/>
     <parent link="table"/>
     <child link="base_link"/>
