Commit message: Updating MARA description with the new model

File: mara_description/urdf/mara.urdf.xacro (robot description, xacro)
@@ -5,5 +5,5 @@
 -->
   <xacro:include filename="$(find mara_description)/urdf/mara.transmission.xacro" />
-  <xacro:include filename="$(find mara_description)/urdf/mara.gazebo.xacro" />
+  <xacro:include filename="$(find mara_description)/urdf/mara_gazebo.urdf.xacro" />
   <xacro:macro name="mara_robot"  params="prefix joint_limited">
     <link name="${prefix}base_link">
@@ -16,5 +16,5 @@
         <origin rpy="0 0 0" xyz="0 0 0"/>
         <geometry>
-          <mesh filename="package://mara_description/meshes/H-ROS_Robot_BASE.stl" scale="0.001 0.001 0.001"/>
+          <mesh filename="package://mara_description/meshes/Base_plancha.stl" scale="0.001 0.001 0.001"/>
         </geometry>
         <material name="Gazebo/Grey">
@@ -25,5 +25,5 @@
         <origin rpy="0 0 0" xyz="0 0 0"/>
         <geometry>
-          <mesh filename="package://mara_description/meshes/H-ROS_Robot_BASE.stl" scale="0.001 0.001 0.001"/>
+          <mesh filename="package://mara_description/meshes/Base_plancha.stl" scale="0.001 0.001 0.001"/>
         </geometry>
       </collision>
@@ -33,14 +33,40 @@
       <selfCollide>True</selfCollide>
     </gazebo>
+    <link name="${prefix}base_robot">
+      <inertial>
+        <origin rpy="0 0 0" xyz="8.625E-08 -4.6583E-06 0.03145"/>
+        <mass value="7.033"/>
+        <inertia ixx="0.1478344" ixy="-0.00001" ixz="0.0" iyy="0.14782335" iyz="0.0" izz="0.29471799"/>
+      </inertial>
+      <visual>
+        <origin rpy="0 0 0" xyz="0 0 0"/>
+        <geometry>
+          <mesh filename="package://mara_description/meshes/Base.stl" scale="0.001 0.001 0.001"/>
+        </geometry>
+        <material name="Gazebo/Grey">
+          <color rgba="0. 0. 0. 1"/>
+        </material>
+      </visual>
+      <collision>
+        <origin rpy="0 0 0" xyz="0 0 0"/>
+        <geometry>
+          <mesh filename="package://mara_description/meshes/Base.stl" scale="0.001 0.001 0.001"/>
+        </geometry>
+      </collision>
+    </link>
+    <gazebo reference="${prefix}base_robot">
+      <material>Gazebo/Grey</material>
+      <selfCollide>True</selfCollide>
+    </gazebo>
     <link name="${prefix}motor1_link">
       <inertial>
         <origin rpy="0 0 0" xyz="8.625E-08 -4.6583E-06 0.03145"/>
-        <mass value="5.8"/>
-        <inertia ixx="0.10105893" ixy="0.000211" ixz="-0.004" iyy="0.09386624" iyz="-0.01698537" izz="0.01449937"/>
-      </inertial>
-      <visual>
-        <origin rpy="0 0 0" xyz="0 0 0"/>
-        <geometry>
-          <mesh filename="package://mara_description/meshes/H-ROS_Robot_mara1.stl" scale="0.001 0.001 0.001"/>
+        <mass value="7.033"/>
+        <inertia ixx="0.1478344" ixy="-0.00001" ixz="0.0" iyy="0.14782335" iyz="0.0" izz="0.29471799"/>
+      </inertial>
+      <visual>
+        <origin rpy="0 0 0" xyz="0 0 0"/>
+        <geometry>
+          <mesh filename="package://mara_description/meshes/MARA_T49.stl" scale="0.001 0.001 0.001"/>
         </geometry>
         <material name="Gazebo/White">
@@ -51,5 +77,5 @@
         <origin rpy="0 0 0" xyz="0 0 0"/>
         <geometry>
-          <mesh filename="package://mara_description/meshes/H-ROS_Robot_mara1.stl" scale="0.001 0.001 0.001"/>
+          <mesh filename="package://mara_description/meshes/MARA_T49.stl" scale="0.001 0.001 0.001"/>
         </geometry>
       </collision>
@@ -59,23 +85,49 @@
       <selfCollide>True</selfCollide>
     </gazebo>
+    <link name="${prefix}motor1_cover">
+      <inertial>
+        <origin rpy="0 0 0" xyz="8.625E-08 -4.6583E-06 0.03145"/>
+        <mass value="7.033"/>
+        <inertia ixx="0.1478344" ixy="-0.00001" ixz="0.0" iyy="0.14782335" iyz="0.0" izz="0.29471799"/>
+      </inertial>
+      <visual>
+        <origin rpy="0 0 0" xyz="0 0 0"/>
+        <geometry>
+          <mesh filename="package://mara_description/meshes/MARA_T49_Black.stl" scale="0.001 0.001 0.001"/>
+        </geometry>
+        <material name="Gazebo/Black">
+          <color rgba="0. 0. 0. 1"/>
+        </material>
+      </visual>
+      <collision>
+        <origin rpy="0 0 0" xyz="0 0 0"/>
+        <geometry>
+          <mesh filename="package://mara_description/meshes/MARA_T49_Black.stl" scale="0.001 0.001 0.001"/>
+        </geometry>
+      </collision>
+    </link>
+    <gazebo reference="${prefix}motor1_cover">
+      <material>Gazebo/Black</material>
+      <selfCollide>True</selfCollide>
+    </gazebo>
     <link name="${prefix}motor2_link">
       <inertial>
         <origin rpy="0 0 0" xyz="8.625E-08 -4.6583E-06 0.03145"/>
-        <mass value="1.03237"/>
-        <inertia ixx="0.014865226" ixy="0.0" ixz="0.0" iyy="0.01557" iyz="0.00071" izz="0.00092"/>
-      </inertial>
-      <visual>
-        <origin rpy="0 0 0" xyz="0 0 0"/>
-        <geometry>
-          <mesh filename="package://mara_description/meshes/H-ROS_Robot_LINK1.stl" scale="0.001 0.001 0.001"/>
-        </geometry>
-        <material name="Gazebo/Black">
-          <color rgba="0. 0. 0. 1"/>
-        </material>
-      </visual>
-      <collision>
-        <origin rpy="0 0 0" xyz="0 0 0"/>
-        <geometry>
-          <mesh filename="package://mara_description/meshes/H-ROS_Robot_LINK1.stl" scale="0.001 0.001 0.001"/>
+        <mass value="7.033"/>
+        <inertia ixx="0.1478344" ixy="-0.00001" ixz="0.0" iyy="0.14782335" iyz="0.0" izz="0.29471799"/>
+      </inertial>
+      <visual>
+        <origin rpy="0 0 0" xyz="0 0 0"/>
+        <geometry>
+          <mesh filename="package://mara_description/meshes/MARA_Link1.stl" scale="0.001 0.001 0.001"/>
+        </geometry>
+        <material name="Gazebo/Black">
+          <color rgba="0. 0. 0. 1"/>
+        </material>
+      </visual>
+      <collision>
+        <origin rpy="0 0 0" xyz="0 0 0"/>
+        <geometry>
+          <mesh filename="package://mara_description/meshes/MARA_Link1.stl" scale="0.001 0.001 0.001"/>
         </geometry>
       </collision>
@@ -88,11 +140,11 @@
       <inertial>
         <origin rpy="0 0 0" xyz="8.625E-08 -4.6583E-06 0.03145"/>
-        <mass value="3.8"/>
-        <inertia ixx="0.04517" ixy="0.00002" ixz="0.0" iyy="0.01587" iyz="0.01444" izz="0.03303"/>
-      </inertial>
-      <visual>
-        <origin rpy="0 0 0" xyz="0 0 0"/>
-        <geometry>
-          <mesh filename="package://mara_description/meshes/H-ROS_Robot_mara2.stl" scale="0.001 0.001 0.001"/>
+        <mass value="7.033"/>
+        <inertia ixx="0.1478344" ixy="-0.00001" ixz="0.0" iyy="0.14782335" iyz="0.0" izz="0.29471799"/>
+      </inertial>
+      <visual>
+        <origin rpy="0 0 0" xyz="0 0 0"/>
+        <geometry>
+          <mesh filename="package://mara_description/meshes/MARA_T30.stl" scale="0.001 0.001 0.001"/>
         </geometry>
         <material name="Gazebo/White">
@@ -103,5 +155,5 @@
         <origin rpy="0 0 0" xyz="0 0 0"/>
         <geometry>
-          <mesh filename="package://mara_description/meshes/H-ROS_Robot_mara2.stl" scale="0.001 0.001 0.001"/>
+          <mesh filename="package://mara_description/meshes/MARA_T30.stl" scale="0.001 0.001 0.001"/>
         </geometry>
       </collision>
@@ -111,23 +163,49 @@
       <selfCollide>True</selfCollide>
     </gazebo>
+    <link name="${prefix}motor3_cover">
+      <inertial>
+        <origin rpy="0 0 0" xyz="8.625E-08 -4.6583E-06 0.03145"/>
+        <mass value="7.033"/>
+        <inertia ixx="0.1478344" ixy="-0.00001" ixz="0.0" iyy="0.14782335" iyz="0.0" izz="0.29471799"/>
+      </inertial>
+      <visual>
+        <origin rpy="0 0 0" xyz="0 0 0"/>
+        <geometry>
+          <mesh filename="package://mara_description/meshes/MARA_T30_Black.stl" scale="0.001 0.001 0.001"/>
+        </geometry>
+        <material name="Gazebo/Black">
+          <color rgba="0. 0. 0. 1"/>
+        </material>
+      </visual>
+      <collision>
+        <origin rpy="0 0 0" xyz="0 0 0"/>
+        <geometry>
+          <mesh filename="package://mara_description/meshes/MARA_T30_Black.stl" scale="0.001 0.001 0.001"/>
+        </geometry>
+      </collision>
+    </link>
+    <gazebo reference="${prefix}motor3_cover">
+      <material>Gazebo/Black</material>
+      <selfCollide>True</selfCollide>
+    </gazebo>
     <link name="${prefix}motor4_link">
       <inertial>
         <origin rpy="0 0 0" xyz="8.625E-08 -4.6583E-06 0.03145"/>
-        <mass value="1.1"/>
-        <inertia ixx="0.01464" ixy="0.0" ixz="0.0" iyy="0.00895" iyz="-0.00631" izz="0.00725"/>
-      </inertial>
-      <visual>
-        <origin rpy="0 0 0" xyz="0 0 0"/>
-        <geometry>
-          <mesh filename="package://mara_description/meshes/H-ROS_Robot_LINK2.stl" scale="0.001 0.001 0.001"/>
-        </geometry>
-        <material name="Gazebo/Black">
-          <color rgba="0. 0. 0. 1"/>
-        </material>
-      </visual>
-      <collision>
-        <origin rpy="0 0 0" xyz="0 0 0"/>
-        <geometry>
-          <mesh filename="package://mara_description/meshes/H-ROS_Robot_LINK2.stl" scale="0.001 0.001 0.001"/>
+        <mass value="7.033"/>
+        <inertia ixx="0.1478344" ixy="-0.00001" ixz="0.0" iyy="0.14782335" iyz="0.0" izz="0.29471799"/>
+      </inertial>
+      <visual>
+        <origin rpy="0 0 0" xyz="0 0 0"/>
+        <geometry>
+          <mesh filename="package://mara_description/meshes/MARA_Link2.stl" scale="0.001 0.001 0.001"/>
+        </geometry>
+        <material name="Gazebo/Black">
+          <color rgba="0. 0. 0. 1"/>
+        </material>
+      </visual>
+      <collision>
+        <origin rpy="0 0 0" xyz="0 0 0"/>
+        <geometry>
+          <mesh filename="package://mara_description/meshes/MARA_Link2.stl" scale="0.001 0.001 0.001"/>
         </geometry>
       </collision>
@@ -140,11 +218,11 @@
       <inertial>
         <origin rpy="0 0 0" xyz="8.625E-08 -4.6583E-06 0.03145"/>
-        <mass value="2.9"/>
-        <inertia ixx="0.03406" ixy="0.0" ixz="0.0" iyy="0.01066" iyz="0.00989" izz="0.02563"/>
-      </inertial>
-      <visual>
-        <origin rpy="0 0 0" xyz="0 0 0"/>
-        <geometry>
-          <mesh filename="package://mara_description/meshes/H-ROS_Robot_mara3.stl" scale="0.001 0.001 0.001"/>
+        <mass value="7.033"/>
+        <inertia ixx="0.1478344" ixy="-0.00001" ixz="0.0" iyy="0.14782335" iyz="0.0" izz="0.29471799"/>
+      </inertial>
+      <visual>
+        <origin rpy="0 0 0" xyz="0 0 0"/>
+        <geometry>
+          <mesh filename="package://mara_description/meshes/MARA_T5.4.stl" scale="0.001 0.001 0.001"/>
         </geometry>
         <material name="Gazebo/White">
@@ -155,5 +233,5 @@
         <origin rpy="0 0 0" xyz="0 0 0"/>
         <geometry>
-          <mesh filename="package://mara_description/meshes/H-ROS_Robot_mara3.stl" scale="0.001 0.001 0.001"/>
+          <mesh filename="package://mara_description/meshes/MARA_T5.4.stl" scale="0.001 0.001 0.001"/>
         </geometry>
       </collision>
@@ -163,23 +241,49 @@
       <selfCollide>True</selfCollide>
     </gazebo>
+    <link name="${prefix}motor5_cover">
+      <inertial>
+        <origin rpy="0 0 0" xyz="8.625E-08 -4.6583E-06 0.03145"/>
+        <mass value="7.033"/>
+        <inertia ixx="0.1478344" ixy="-0.00001" ixz="0.0" iyy="0.14782335" iyz="0.0" izz="0.29471799"/>
+      </inertial>
+      <visual>
+        <origin rpy="0 0 0" xyz="0 0 0"/>
+        <geometry>
+          <mesh filename="package://mara_description/meshes/MARA_T5.4_black.stl" scale="0.001 0.001 0.001"/>
+        </geometry>
+        <material name="Gazebo/Black">
+          <color rgba="0. 0. 0. 1"/>
+        </material>
+      </visual>
+      <collision>
+        <origin rpy="0 0 0" xyz="0 0 0"/>
+        <geometry>
+          <mesh filename="package://mara_description/meshes/MARA_T5.4_black.stl" scale="0.001 0.001 0.001"/>
+        </geometry>
+      </collision>
+    </link>
+    <gazebo reference="${prefix}motor5_cover">
+      <material>Gazebo/Black</material>
+      <selfCollide>True</selfCollide>
+    </gazebo>
     <link name="${prefix}motor6_link">
       <inertial>
         <origin rpy="0 0 0" xyz="8.625E-08 -4.6583E-06 0.03145"/>
-        <mass value="2.9"/>
-        <inertia ixx="0.0005" ixy="0.0" ixz="0.0" iyy="0.0005" iyz="0.0000" izz="0.0003"/>
-      </inertial>
-      <visual>
-        <origin rpy="0 0 ${60*3.14/180}" xyz="0 0 0"/>
-        <geometry>
-          <mesh filename="package://mara_description/meshes/gripper_support.stl" scale="0.001 0.001 0.001"/>
-        </geometry>
-        <material name="Gazebo/Black">
-          <color rgba="0. 0. 0. 1"/>
-        </material>
-      </visual>
-      <collision>
-        <origin rpy="0 0 ${60*3.14/180}" xyz="0 0 0"/>
-        <geometry>
-          <mesh filename="package://mara_description/meshes/gripper_support.stl" scale="0.001 0.001 0.001"/>
+        <mass value="7.033"/>
+        <inertia ixx="0.1478344" ixy="-0.00001" ixz="0.0" iyy="0.14782335" iyz="0.0" izz="0.29471799"/>
+      </inertial>
+      <visual>
+        <origin rpy="0 0 0" xyz="0 0 0"/>
+        <geometry>
+          <mesh filename="package://mara_description/meshes/MARA_GripperAdapter.stl" scale="0.001 0.001 0.001"/>
+        </geometry>
+        <material name="Gazebo/Black">
+          <color rgba="0. 0. 0. 1"/>
+        </material>
+      </visual>
+      <collision>
+        <origin rpy="0 0 0" xyz="0 0 0"/>
+        <geometry>
+          <mesh filename="package://mara_description/meshes/MARA_GripperAdapter.stl" scale="0.001 0.001 0.001"/>
         </geometry>
       </collision>
@@ -195,7 +299,12 @@
       <selfCollide>False</selfCollide>
     </gazebo>
+    <joint name="${prefix}joint_bases" type="fixed">
+      <origin rpy="0 0 0" xyz="0 0 0.04"/>
+      <parent link="${prefix}base_link"/>
+      <child link="${prefix}base_robot"/>
+    </joint>
     <joint name="${prefix}motor1" type="revolute">
-      <origin rpy="0 0 0" xyz="0 0 0.00625"/>
-      <parent link="${prefix}base_link"/>
+      <origin rpy="0 0 0" xyz="0 0 0.05122"/>
+      <parent link="${prefix}base_robot"/>
       <child link="${prefix}motor1_link"/>
       <axis xyz="0 0 -1"/>
@@ -203,42 +312,57 @@
       <dynamics damping="0" friction="0"/>
     </joint>
+    <joint name="${prefix}motor1_cover_joint" type="fixed">
+      <origin rpy="0 0 0" xyz="0 0 0.0"/>
+      <parent link="${prefix}motor1_link"/>
+      <child link="${prefix}motor1_cover"/>
+    </joint>
     <joint name="${prefix}motor2" type="revolute">
-      <origin rpy="0 0 0" xyz="0 -0.100499999 0.1545"/>
+      <origin rpy="0 0 0" xyz="0.118 0 0.1637"/>
       <parent link="${prefix}motor1_link"/>
       <child link="${prefix}motor2_link"/>
-      <axis xyz="0 1 0"/>
-      <limit effort="330.0" lower="-3.13" upper="3.13" velocity="3.1416"/>
+      <axis xyz="1 0 0"/>
+      <limit effort="330.0" lower="-2.3562" upper="2.3562" velocity="3.1416"/>
       <dynamics damping="0" friction="0"/>
     </joint>
     <joint name="${prefix}motor3" type="revolute">
-      <origin rpy="0 0 0" xyz="0 -0.000499999 0.2"/>
+      <origin rpy="0 0 0" xyz="-0.009 0 0.2"/>
       <parent link="${prefix}motor2_link"/>
       <child link="${prefix}motor3_link"/>
-      <axis xyz="0 -1 0"/>
-      <limit effort="330" lower="-3.13" upper="3.13" velocity="3.1416"/>
-      <dynamics damping="0" friction="0"/>
+      <axis xyz="1 0 0"/>
+      <limit effort="330.0" lower="-2.3562" upper="2.3562" velocity="3.1416"/>
+      <dynamics damping="0" friction="0"/>
+    </joint>
+    <joint name="${prefix}motor3_cover_joint" type="fixed">
+      <origin rpy="0 0 0" xyz="0 0 0.0"/>
+      <parent link="${prefix}motor3_link"/>
+      <child link="${prefix}motor3_cover"/>
     </joint>
     <joint name="${prefix}motor4" type="revolute">
-      <origin rpy="0 0 0" xyz="0 0.09999 0.12999997"/>
+      <origin rpy="0 0 0" xyz="-0.109255 0 0.149255"/>
       <parent link="${prefix}motor3_link"/>
       <child link="${prefix}motor4_link"/>
-      <axis xyz="0 0 -1"/>
-      <limit effort="330" lower="-3.13" upper="3.13" velocity="3.1416"/>
+      <axis xyz="0 0 1"/>
+      <limit effort="330.0" lower="-2.3562" upper="2.3562" velocity="3.1416"/>
       <dynamics damping="0" friction="0"/>
     </joint>
     <joint name="${prefix}motor5" type="revolute">
-      <origin rpy="0 0 0" xyz="0 -0.096999 0.15906"/>
+      <origin rpy="0 0 0" xyz="0.1054570 0 0.16074"/>
       <parent link="${prefix}motor4_link"/>
       <child link="${prefix}motor5_link"/>
-      <axis xyz="0 -1 0"/>
-      <limit effort="330" lower="-3.13" upper="3.13" velocity="3.1416"/>
-      <dynamics damping="0" friction="0"/>
+      <axis xyz="1 0 0"/>
+      <limit effort="330.0" lower="-2.3562" upper="2.3562" velocity="3.1416"/>
+      <dynamics damping="0" friction="0"/>
+    </joint>
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
File: mara_description/urdf/mara_robot_camera_top.urdf.xacro (robot description, xacro)
@@ -3,22 +3,22 @@
        name="mara" >
   <!-- common stuff -->
-  <xacro:include filename="$(find mara_description)/urdf/common.gazebo.xacro" />
+  <xacro:include filename="$(find mara_description)/urdf/mara_gazebo.urdf.xacro" />
   <!-- mara -->
   <xacro:include filename="$(find mara_description)/urdf/mara.urdf.xacro" />
   <!-- robotiq 140 gripper -->
-  <xacro:include filename="$(find mara_description)/urdf/robotiq_gripper.urdf.xacro" />
+  <!-- <xacro:include filename="$(find robotiq_arg2f_model_visualization)/urdf/robotiq_gripper.urdf.xacro" /> -->
   <!-- <xacro:include filename="$(find mara_description)/urdf/camera_top.urdf.xacro" /> -->
   <xacro:include filename="$(find mara_description)/urdf/table.urdf.xacro" />
   <!-- arm -->
   <xacro:mara_robot prefix="" joint_limited="false"/>
-  <xacro:robotiq_gripper prefix="" />
+  <!-- <xacro:robotiq_gripper prefix="" /> -->
   <!-- <xacro:mara_camera_top prefix="" /> -->
   <xacro:table prefix="" />
   <link name="world" />
-  <joint name="end_effector_adapter_to_robotiq" type="fixed">
-    <origin rpy="0 0 0" xyz=" 0 0 0.05375"/>
+  <!-- <joint name="end_effector_adapter_to_robotiq" type="fixed">
+    <origin rpy="0 0 1.57" xyz=" 0 0 0.04659"/>
     <parent link="motor6_link"/>
     <child link="robotiq_arg2f_base_link"/>
-  </joint>
+  </joint> -->
   <joint name="world_to_table_joint" type="fixed">
     <origin rpy="0 0 0" xyz="0 0 0.02"/>
@@ -27,5 +27,5 @@
   </joint>
   <joint name="table_to_base_joint" type="fixed">
-    <origin rpy="0 0 0" xyz="0 0 0.65"/>
+    <origin rpy="0 0 0" xyz="0 0 0.62"/>
     <parent link="table"/>
     <child link="base_link"/>

File: mara_description/urdf/mara_robot_nogripper.urdf.xacro (robot description, xacro)
@@ -5,10 +5,10 @@
   <xacro:include filename="$(find mara_description)/urdf/common.gazebo.xacro" />
   <!-- mara -->
-  <xacro:include filename="$(find mara_description)/urdf/mara_nogripper.urdf.xacro" />
-  <xacro:include filename="$(find mara_description)/urdf/camera_top.urdf.xacro" />
+  <xacro:include filename="$(find mara_description)/urdf/mara.urdf.xacro" />
+  <!-- robotiq 140 gripper -->
+  <xacro:include filename="$(find mara_description)/urdf/robotiq_gripper.urdf.xacro" />
   <xacro:include filename="$(find mara_description)/urdf/table.urdf.xacro" />
   <!-- arm -->
   <xacro:mara_robot prefix="" joint_limited="false"/>
-  <xacro:mara_camera_top prefix="" />
   <xacro:table prefix="" />
   <link name="world" />

File: mara_description/urdf/table.urdf.xacro (robot description, xacro)
@@ -8,6 +8,6 @@
       <inertial>
         <origin rpy="0 0 0" xyz="0 0 0"/>
-         <mass value=".0"/>
-         <inertia ixx="1" ixy="0" ixz="0" iyy="1" iyz="0" izz="1"/>
+         <mass value="0.00001"/>
+         <inertia ixx="0.001" ixy="0" ixz="0" iyy="0.001" iyz="0" izz="0.001"/>
       </inertial>
       <visual>

Commit message: Fixing axis

File: mara_description/urdf/mara.urdf.xacro (robot description, xacro)
@@ -321,5 +321,5 @@
       <parent link="${prefix}motor1_link"/>
       <child link="${prefix}motor2_link"/>
-      <axis xyz="1 0 0"/>
+      <axis xyz="-1 0 0"/>
       <limit effort="330.0" lower="-2.3562" upper="2.3562" velocity="3.1416"/>
       <dynamics damping="0" friction="0"/>
@@ -342,5 +342,5 @@
       <parent link="${prefix}motor3_link"/>
       <child link="${prefix}motor4_link"/>
-      <axis xyz="0 0 1"/>
+      <axis xyz="0 0 -1"/>
       <limit effort="330.0" lower="-2.3562" upper="2.3562" velocity="3.1416"/>
       <dynamics damping="0" friction="0"/>
@@ -363,5 +363,5 @@
       <parent link="${prefix}motor5_link"/>
       <child link="${prefix}motor6_link"/>
-      <axis xyz="0 0 1"/>
+      <axis xyz="0 0 -1"/>
       <limit effort="330.0" lower="-2.3562" upper="2.3562" velocity="3.1416"/>
       <dynamics damping="0" friction="0"/>
