Commit message: fixng names in the .xacro

File: mara_description/urdf/mara.urdf.xacro (robot description, xacro)
@@ -16,5 +16,5 @@
         <origin rpy="0 0 0" xyz="0 0 0"/>
         <geometry>
-          <mesh filename="package://mara_description/meshes/Base_plancha.stl" scale="0.001 0.001 0.001"/>
+          <mesh filename="package://mara_description/meshes/Base_plancha.dae" scale="0.001 0.001 0.001"/>
         </geometry>
         <material name="Gazebo/Grey">
@@ -25,5 +25,5 @@
         <origin rpy="0 0 0" xyz="0 0 0"/>
         <geometry>
-          <mesh filename="package://mara_description/meshes/Base_plancha.stl" scale="0.001 0.001 0.001"/>
+          <mesh filename="package://mara_description/meshes/Base_plancha.dae" scale="0.001 0.001 0.001"/>
         </geometry>
       </collision>
@@ -42,14 +42,14 @@
         <origin rpy="0 0 0" xyz="0 0 0"/>
         <geometry>
-          <mesh filename="package://mara_description/meshes/Base.stl" scale="0.001 0.001 0.001"/>
+          <mesh filename="package://mara_description/meshes/Base.dae" scale="0.001 0.001 0.001"/>
         </geometry>
         <material name="Gazebo/Grey">
-          <color rgba="0. 0. 0. 1"/>
-        </material>
-      </visual>
-      <collision>
-        <origin rpy="0 0 0" xyz="0 0 0"/>
-        <geometry>
-          <mesh filename="package://mara_description/meshes/Base.stl" scale="0.001 0.001 0.001"/>
+          <color rgba="1. 0. 0. 1.0"/>
+        </material>
+      </visual>
+      <collision>
+        <origin rpy="0 0 0" xyz="0 0 0"/>
+        <geometry>
+          <mesh filename="package://mara_description/meshes/Base.dae" scale="0.001 0.001 0.001"/>
         </geometry>
       </collision>
@@ -68,5 +68,5 @@
         <origin rpy="0 0 0" xyz="0 0 0"/>
         <geometry>
-          <mesh filename="package://mara_description/meshes/MARA_T49.stl" scale="0.001 0.001 0.001"/>
+          <mesh filename="package://mara_description/meshes/MARA_T49.dae" scale="0.001 0.001 0.001"/>
         </geometry>
         <material name="Gazebo/White">
@@ -77,5 +77,5 @@
         <origin rpy="0 0 0" xyz="0 0 0"/>
         <geometry>
-          <mesh filename="package://mara_description/meshes/MARA_T49.stl" scale="0.001 0.001 0.001"/>
+          <mesh filename="package://mara_description/meshes/MARA_T49.dae" scale="0.001 0.001 0.001"/>
         </geometry>
       </collision>
@@ -94,14 +94,14 @@
         <origin rpy="0 0 0" xyz="0 0 0"/>
         <geometry>
-          <mesh filename="package://mara_description/meshes/MARA_T49_Black.stl" scale="0.001 0.001 0.001"/>
-        </geometry>
-        <material name="Gazebo/Black">
-          <color rgba="0. 0. 0. 1"/>
-        </material>
-      </visual>
-      <collision>
-        <origin rpy="0 0 0" xyz="0 0 0"/>
-        <geometry>
-          <mesh filename="package://mara_description/meshes/MARA_T49_Black.stl" scale="0.001 0.001 0.001"/>
+          <mesh filename="package://mara_description/meshes/MARA_T49_Black.dae" scale="0.001 0.001 0.001"/>
+        </geometry>
+        <material name="Gazebo/Black">
+          <color rgba="0. 0. 0. 1"/>
+        </material>
+      </visual>
+      <collision>
+        <origin rpy="0 0 0" xyz="0 0 0"/>
+        <geometry>
+          <mesh filename="package://mara_description/meshes/MARA_T49_Black.dae" scale="0.001 0.001 0.001"/>
         </geometry>
       </collision>
@@ -120,14 +120,14 @@
         <origin rpy="0 0 0" xyz="0 0 0"/>
         <geometry>
-          <mesh filename="package://mara_description/meshes/MARA_Link1.stl" scale="0.001 0.001 0.001"/>
-        </geometry>
-        <material name="Gazebo/Black">
-          <color rgba="0. 0. 0. 1"/>
-        </material>
-      </visual>
-      <collision>
-        <origin rpy="0 0 0" xyz="0 0 0"/>
-        <geometry>
-          <mesh filename="package://mara_description/meshes/MARA_Link1.stl" scale="0.001 0.001 0.001"/>
+          <mesh filename="package://mara_description/meshes/MARA_Link1.dae" scale="0.001 0.001 0.001"/>
+        </geometry>
+        <material name="Gazebo/Black">
+          <color rgba="0. 0. 0. 1"/>
+        </material>
+      </visual>
+      <collision>
+        <origin rpy="0 0 0" xyz="0 0 0"/>
+        <geometry>
+          <mesh filename="package://mara_description/meshes/MARA_Link1.dae" scale="0.001 0.001 0.001"/>
         </geometry>
       </collision>
@@ -146,5 +146,5 @@
         <origin rpy="0 0 0" xyz="0 0 0"/>
         <geometry>
-          <mesh filename="package://mara_description/meshes/MARA_T30.stl" scale="0.001 0.001 0.001"/>
+          <mesh filename="package://mara_description/meshes/MARA_T30.dae" scale="0.001 0.001 0.001"/>
         </geometry>
         <material name="Gazebo/White">
@@ -155,5 +155,5 @@
         <origin rpy="0 0 0" xyz="0 0 0"/>
         <geometry>
-          <mesh filename="package://mara_description/meshes/MARA_T30.stl" scale="0.001 0.001 0.001"/>
+          <mesh filename="package://mara_description/meshes/MARA_T30.dae" scale="0.001 0.001 0.001"/>
         </geometry>
       </collision>
@@ -172,14 +172,14 @@
         <origin rpy="0 0 0" xyz="0 0 0"/>
         <geometry>
-          <mesh filename="package://mara_description/meshes/MARA_T30_Black.stl" scale="0.001 0.001 0.001"/>
-        </geometry>
-        <material name="Gazebo/Black">
-          <color rgba="0. 0. 0. 1"/>
-        </material>
-      </visual>
-      <collision>
-        <origin rpy="0 0 0" xyz="0 0 0"/>
-        <geometry>
-          <mesh filename="package://mara_description/meshes/MARA_T30_Black.stl" scale="0.001 0.001 0.001"/>
+          <mesh filename="package://mara_description/meshes/MARA_T30_Black.dae" scale="0.001 0.001 0.001"/>
+        </geometry>
+        <material name="Gazebo/Black">
+          <color rgba="0. 0. 0. 1"/>
+        </material>
+      </visual>
+      <collision>
+        <origin rpy="0 0 0" xyz="0 0 0"/>
+        <geometry>
+          <mesh filename="package://mara_description/meshes/MARA_T30_Black.dae" scale="0.001 0.001 0.001"/>
         </geometry>
       </collision>
@@ -198,14 +198,14 @@
         <origin rpy="0 0 0" xyz="0 0 0"/>
         <geometry>
-          <mesh filename="package://mara_description/meshes/MARA_Link2.stl" scale="0.001 0.001 0.001"/>
-        </geometry>
-        <material name="Gazebo/Black">
-          <color rgba="0. 0. 0. 1"/>
-        </material>
-      </visual>
-      <collision>
-        <origin rpy="0 0 0" xyz="0 0 0"/>
-        <geometry>
-          <mesh filename="package://mara_description/meshes/MARA_Link2.stl" scale="0.001 0.001 0.001"/>
+          <mesh filename="package://mara_description/meshes/MARA_Link2.dae" scale="0.001 0.001 0.001"/>
+        </geometry>
+        <material name="Gazebo/Black">
+          <color rgba="0. 0. 0. 1"/>
+        </material>
+      </visual>
+      <collision>
+        <origin rpy="0 0 0" xyz="0 0 0"/>
+        <geometry>
+          <mesh filename="package://mara_description/meshes/MARA_Link2.dae" scale="0.001 0.001 0.001"/>
         </geometry>
       </collision>
@@ -224,5 +224,5 @@
         <origin rpy="0 0 0" xyz="0 0 0"/>
         <geometry>
-          <mesh filename="package://mara_description/meshes/MARA_T5.4.stl" scale="0.001 0.001 0.001"/>
+          <mesh filename="package://mara_description/meshes/MARA_T5.4.dae" scale="0.001 0.001 0.001"/>
         </geometry>
         <material name="Gazebo/White">
@@ -233,5 +233,5 @@
         <origin rpy="0 0 0" xyz="0 0 0"/>
         <geometry>
-          <mesh filename="package://mara_description/meshes/MARA_T5.4.stl" scale="0.001 0.001 0.001"/>
+          <mesh filename="package://mara_description/meshes/MARA_T5.4.dae" scale="0.001 0.001 0.001"/>
         </geometry>
       </collision>
@@ -250,14 +250,14 @@
         <origin rpy="0 0 0" xyz="0 0 0"/>
         <geometry>
-          <mesh filename="package://mara_description/meshes/MARA_T5.4_black.stl" scale="0.001 0.001 0.001"/>
-        </geometry>
-        <material name="Gazebo/Black">
-          <color rgba="0. 0. 0. 1"/>
-        </material>
-      </visual>
-      <collision>
-        <origin rpy="0 0 0" xyz="0 0 0"/>
-        <geometry>
-          <mesh filename="package://mara_description/meshes/MARA_T5.4_black.stl" scale="0.001 0.001 0.001"/>
+          <mesh filename="package://mara_description/meshes/MARA_T5.4_black.dae" scale="0.001 0.001 0.001"/>
+        </geometry>
+        <material name="Gazebo/Black">
+          <color rgba="0. 0. 0. 1"/>
+        </material>
+      </visual>
+      <collision>
+        <origin rpy="0 0 0" xyz="0 0 0"/>
+        <geometry>
+          <mesh filename="package://mara_description/meshes/MARA_T5.4_black.dae" scale="0.001 0.001 0.001"/>
         </geometry>
       </collision>
@@ -276,14 +276,14 @@
         <origin rpy="0 0 0" xyz="0 0 0"/>
         <geometry>
-          <mesh filename="package://mara_description/meshes/MARA_GripperAdapter.stl" scale="0.001 0.001 0.001"/>
-        </geometry>
-        <material name="Gazebo/Black">
-          <color rgba="0. 0. 0. 1"/>
-        </material>
-      </visual>
-      <collision>
-        <origin rpy="0 0 0" xyz="0 0 0"/>
-        <geometry>
-          <mesh filename="package://mara_description/meshes/MARA_GripperAdapter.stl" scale="0.001 0.001 0.001"/>
+          <mesh filename="package://mara_description/meshes/MARA_GripperAdapter.dae" scale="0.001 0.001 0.001"/>
+        </geometry>
+        <material name="Gazebo/Black">
+          <color rgba="0. 0. 0. 1"/>
+        </material>
+      </visual>
+      <collision>
+        <origin rpy="0 0 0" xyz="0 0 0"/>
+        <geometry>
+          <mesh filename="package://mara_description/meshes/MARA_GripperAdapter.dae" scale="0.001 0.001 0.001"/>
         </geometry>
       </collision>

Commit message: Updating urdf model

File: mara_description/urdf/mara.urdf.xacro (robot description, xacro)
@@ -44,5 +44,5 @@
           <mesh filename="package://mara_description/meshes/Base.dae" scale="0.001 0.001 0.001"/>
         </geometry>
-        <material name="Gazebo/Grey">
+        <material name="Gazebo/Black">
           <color rgba="1. 0. 0. 1.0"/>
         </material>
@@ -56,5 +56,5 @@
     </link>
     <gazebo reference="${prefix}base_robot">
-      <material>Gazebo/Grey</material>
+      <material>Gazebo/Black</material>
       <selfCollide>True</selfCollide>
     </gazebo>

File: mara_description/urdf/mara_robot_camera_top.urdf (robot description, URDF)
Before this commit: robot mara, 24 links, 23 joints
Joints:
- joint motor6: limit lower=-2.3562 upper=2.3562 effort=330.0 velocity=3.1416 -> lower=-3.1416 upper=3.1416 effort=330.0 velocity=3.1416

Commit message: include param to locate ee_link

File: mara_description/urdf/mara.urdf.xacro (robot description, xacro)
@@ -6,5 +6,5 @@
   <xacro:include filename="$(find mara_description)/urdf/mara.transmission.xacro" />
   <xacro:include filename="$(find mara_description)/urdf/mara_gazebo.urdf.xacro" />
-  <xacro:macro name="mara_robot"  params="prefix joint_limited">
+  <xacro:macro name="mara_robot"  params="prefix ee_link_distance">
     <link name="${prefix}base_link">
       <inertial>
@@ -368,5 +368,5 @@
     </joint>
     <joint name="${prefix}ee_link" type="fixed">
-      <origin rpy="0 -1.57 0" xyz="0 0.0 0.24"/>
+      <origin rpy="0 -1.57 0" xyz="0 0.0 ${ee_link_distance}"/>
       <parent link="${prefix}motor6_link"/>
       <child link="${prefix}ee_link"/>
@@ -374,5 +374,5 @@
     <link name="${prefix}tool0"/>
     <joint name="${prefix}${prefix}motor6_link-tool0_fixed_joint" type="fixed">
-      <origin rpy="0 -1.57 0" xyz="0 0.0 0.24"/>
+      <origin rpy="0 -1.57 0" xyz="0 0.0 ${ee_link_distance}"/>
       <parent link="${prefix}${prefix}motor6_link"/>
       <child link="${prefix}tool0"/>

Commit message: Modified axis signs

File: mara_description/urdf/mara.urdf.xacro (robot description, xacro)
@@ -308,5 +308,5 @@
       <parent link="${prefix}base_robot"/>
       <child link="${prefix}motor1_link"/>
-      <axis xyz="0 0 -1"/>
+      <axis xyz="0 0 1"/>
       <limit effort="330.0" lower="-2.3562" upper="2.3562" velocity="3.1416"/>
       <dynamics damping="0" friction="0"/>
@@ -321,5 +321,5 @@
       <parent link="${prefix}motor1_link"/>
       <child link="${prefix}motor2_link"/>
-      <axis xyz="-1 0 0"/>
+      <axis xyz="1 0 0"/>
       <limit effort="330.0" lower="-2.3562" upper="2.3562" velocity="3.1416"/>
       <dynamics damping="0" friction="0"/>
@@ -329,5 +329,5 @@
       <parent link="${prefix}motor2_link"/>
       <child link="${prefix}motor3_link"/>
-      <axis xyz="1 0 0"/>
+      <axis xyz="-1 0 0"/>
       <limit effort="330.0" lower="-2.3562" upper="2.3562" velocity="3.1416"/>
       <dynamics damping="0" friction="0"/>
@@ -342,5 +342,5 @@
       <parent link="${prefix}motor3_link"/>
       <child link="${prefix}motor4_link"/>
-      <axis xyz="0 0 -1"/>
+      <axis xyz="0 0 1"/>
       <limit effort="330.0" lower="-2.3562" upper="2.3562" velocity="3.1416"/>
       <dynamics damping="0" friction="0"/>
@@ -350,5 +350,5 @@
       <parent link="${prefix}motor4_link"/>
       <child link="${prefix}motor5_link"/>
-      <axis xyz="1 0 0"/>
+      <axis xyz="-1 0 0"/>
       <limit effort="330.0" lower="-2.3562" upper="2.3562" velocity="3.1416"/>
       <dynamics damping="0" friction="0"/>
@@ -363,5 +363,5 @@
       <parent link="${prefix}motor5_link"/>
       <child link="${prefix}motor6_link"/>
-      <axis xyz="0 0 -1"/>
+      <axis xyz="0 0 1"/>
       <limit effort="330.0" lower="-2.3562" upper="2.3562" velocity="3.1416"/>
       <dynamics damping="0" friction="0"/>

Commit message: Updating inertia and efforts

File: mara_description/urdf/mara.urdf.xacro (robot description, xacro)
@@ -37,5 +37,5 @@
         <origin rpy="0 0 0" xyz="8.625E-08 -4.6583E-06 0.03145"/>
         <mass value="7.033"/>
-        <inertia ixx="0.1478344" ixy="-0.00001" ixz="0.0" iyy="0.14782335" iyz="0.0" izz="0.29471799"/>
+        <inertia ixx="0.1478344" ixy="0.00001" ixz="0.0" iyy="0.14782335" iyz="0.0" izz="0.29471799"/>
       </inertial>
       <visual>
@@ -61,7 +61,7 @@
     <link name="${prefix}motor1_link">
       <inertial>
-        <origin rpy="0 0 0" xyz="8.625E-08 -4.6583E-06 0.03145"/>
-        <mass value="7.033"/>
-        <inertia ixx="0.1478344" ixy="-0.00001" ixz="0.0" iyy="0.14782335" iyz="0.0" izz="0.29471799"/>
+        <origin rpy="0 0 0" xyz="0.02066 0 0.12051"/>
+        <mass value="5.6"/>
+        <inertia ixx="0.0200769278" ixy="-7.72273E-006" ixz="0.0050158708" iyy="0.0257088151" iyz="5.49229E-006" izz="0.0120821377"/>
       </inertial>
       <visual>
@@ -88,6 +88,6 @@
       <inertial>
         <origin rpy="0 0 0" xyz="8.625E-08 -4.6583E-06 0.03145"/>
-        <mass value="7.033"/>
-        <inertia ixx="0.1478344" ixy="-0.00001" ixz="0.0" iyy="0.14782335" iyz="0.0" izz="0.29471799"/>
+        <mass value="0.0"/>
+        <inertia ixx="0.0" ixy="0.0" ixz="0.0" iyy="0.0" iyz="0.0" izz="0.0"/>
       </inertial>
       <visual>
@@ -113,7 +113,7 @@
     <link name="${prefix}motor2_link">
       <inertial>
-        <origin rpy="0 0 0" xyz="8.625E-08 -4.6583E-06 0.03145"/>
-        <mass value="7.033"/>
-        <inertia ixx="0.1478344" ixy="-0.00001" ixz="0.0" iyy="0.14782335" iyz="0.0" izz="0.29471799"/>
+        <origin rpy="0 0 0" xyz="-0.01665 0.0 0.09639"/>
+        <mass value="1.236"/>
+        <inertia ixx="0.0079614839" ixy="0.000000037" ixz="-0.0003203013" iyy="0.007135338" iyz="-0.000001062" izz="0.001111114"/>
       </inertial>
       <visual>
@@ -139,7 +139,7 @@
     <link name="${prefix}motor3_link">
       <inertial>
-        <origin rpy="0 0 0" xyz="8.625E-08 -4.6583E-06 0.03145"/>
-        <mass value="7.033"/>
-        <inertia ixx="0.1478344" ixy="-0.00001" ixz="0.0" iyy="0.14782335" iyz="0.0" izz="0.29471799"/>
+        <origin rpy="0 0 0" xyz="-0.08963 0.0 0.0403"/>
+        <mass value="3.95"/>
+        <inertia ixx="0.0115136615" ixy="-1.231046E-005" ixz="-0.003148516" iyy="0.0149841676" iyz="-8.81378E-006" izz="0.0070387807"/>
       </inertial>
       <visual>
@@ -166,6 +166,6 @@
       <inertial>
         <origin rpy="0 0 0" xyz="8.625E-08 -4.6583E-06 0.03145"/>
-        <mass value="7.033"/>
-        <inertia ixx="0.1478344" ixy="-0.00001" ixz="0.0" iyy="0.14782335" iyz="0.0" izz="0.29471799"/>
+        <mass value="0.0"/>
+        <inertia ixx="0.0" ixy="0.0" ixz="0.0" iyy="0.0" iyz="0.0" izz="0.0"/>
       </inertial>
       <visual>
@@ -191,7 +191,7 @@
     <link name="${prefix}motor4_link">
       <inertial>
-        <origin rpy="0 0 0" xyz="8.625E-08 -4.6583E-06 0.03145"/>
-        <mass value="7.033"/>
-        <inertia ixx="0.1478344" ixy="-0.00001" ixz="0.0" iyy="0.14782335" iyz="0.0" izz="0.29471799"/>
+        <origin rpy="0 0 0" xyz="0.06357 0.0 0.05698"/>
+        <mass value="1.258"/>
+        <inertia ixx="0.005919676" ixy="0.000000923" ixz="0.0022280208" iyy="0.0068807393" iyz="6.1373E-007" izz="0.00257485"/>
       </inertial>
       <visual>
@@ -217,7 +217,7 @@
     <link name="${prefix}motor5_link">
       <inertial>
-        <origin rpy="0 0 0" xyz="8.625E-08 -4.6583E-06 0.03145"/>
-        <mass value="7.033"/>
-        <inertia ixx="0.1478344" ixy="-0.00001" ixz="0.0" iyy="0.14782335" iyz="0.0" izz="0.29471799"/>
+        <origin rpy="0 0 0" xyz="-0.09105 0.0 0.03676"/>
+        <mass value="2.85"/>
+        <inertia ixx="0.0072829492" ixy="3.77994E-006" ixz="-0.0015682105" iyy="0.0098263499" iyz="2.52745E-006" izz="0.0045615321"/>
       </inertial>
       <visual>
@@ -244,6 +244,6 @@
       <inertial>
         <origin rpy="0 0 0" xyz="8.625E-08 -4.6583E-06 0.03145"/>
-        <mass value="7.033"/>
-        <inertia ixx="0.1478344" ixy="-0.00001" ixz="0.0" iyy="0.14782335" iyz="0.0" izz="0.29471799"/>
+        <mass value="0.0"/>
+        <inertia ixx="0.0" ixy="0.0" ixz="0.0" iyy="0.0" iyz="0.0" izz="0.0"/>
       </inertial>
       <visual>
@@ -269,7 +269,7 @@
     <link name="${prefix}motor6_link">
       <inertial>
-        <origin rpy="0 0 0" xyz="8.625E-08 -4.6583E-06 0.03145"/>
-        <mass value="7.033"/>
-        <inertia ixx="0.1478344" ixy="-0.00001" ixz="0.0" iyy="0.14782335" iyz="0.0" izz="0.29471799"/>
+        <origin rpy="0 0 0" xyz="0.0 0.0 -0.0173"/>
+        <mass value="0.14"/>
+        <inertia ixx="9.22e-05" ixy="6.35e-7" ixz="2.00e-11" iyy="9.73e-5" iyz="2.36e-9" izz="1.77e-4"/>
       </inertial>
       <visual>
@@ -309,5 +309,5 @@
       <child link="${prefix}motor1_link"/>
       <axis xyz="0 0 1"/>
-      <limit effort="330.0" lower="-2.3562" upper="2.3562" velocity="3.1416"/>
+      <limit effort="104.0" lower="-3.1416" upper="3.1416" velocity="1.57"/>
       <dynamics damping="0" friction="0"/>
     </joint>
@@ -322,5 +322,5 @@
       <child link="${prefix}motor2_link"/>
       <axis xyz="1 0 0"/>
-      <limit effort="330.0" lower="-2.3562" upper="2.3562" velocity="3.1416"/>
+      <limit effort="104.0" lower="-2.35" upper="2.35" velocity="1.57"/>
       <dynamics damping="0" friction="0"/>
     </joint>
@@ -330,5 +330,5 @@
       <child link="${prefix}motor3_link"/>
       <axis xyz="-1 0 0"/>
-      <limit effort="330.0" lower="-2.3562" upper="2.3562" velocity="3.1416"/>
+      <limit effort="69" lower="-2.61" upper="2.61" velocity="1.57"/>
       <dynamics damping="0" friction="0"/>
     </joint>
@@ -343,5 +343,5 @@
       <child link="${prefix}motor4_link"/>
       <axis xyz="0 0 1"/>
-      <limit effort="330.0" lower="-2.3562" upper="2.3562" velocity="3.1416"/>
+      <limit effort="69" lower="-3.14" upper="3.14" velocity="1.57"/>
       <dynamics damping="0" friction="0"/>
     </joint>
@@ -351,5 +351,5 @@
       <child link="${prefix}motor5_link"/>
       <axis xyz="-1 0 0"/>
-      <limit effort="330.0" lower="-2.3562" upper="2.3562" velocity="3.1416"/>
+      <limit effort="34" lower="-2.56" upper="2.56" velocity="1.57"/>
       <dynamics damping="0" friction="0"/>
     </joint>
@@ -364,5 +364,5 @@
       <child link="${prefix}motor6_link"/>
       <axis xyz="0 0 1"/>
-      <limit effort="330.0" lower="-2.3562" upper="2.3562" velocity="3.1416"/>
+      <limit effort="34" lower="-3.14" upper="3.14" velocity="1.57"/>
       <dynamics damping="0" friction="0"/>
     </joint>

Commit message: Adapting axis to ros2

File: mara_description/urdf/mara.urdf.xacro (robot description, xacro)
@@ -101,5 +101,5 @@
       </visual>
       <collision>
-        <origin rpy="0 0 0" xyz="0 0 0"/>
+        <origin rpy="0 0 3.1416" xyz="0 0 0"/>
         <geometry>
           <mesh filename="package://mara_description/meshes/MARA_T49_Black.dae" scale="0.001 0.001 0.001"/>
@@ -308,5 +308,5 @@
       <parent link="${prefix}base_robot"/>
       <child link="${prefix}motor1_link"/>
-      <axis xyz="0 0 1"/>
+      <axis xyz="0 0 -1"/>
       <limit effort="104.0" lower="-3.1416" upper="3.1416" velocity="1.57"/>
       <dynamics damping="0" friction="0"/>
@@ -321,5 +321,5 @@
       <parent link="${prefix}motor1_link"/>
       <child link="${prefix}motor2_link"/>
-      <axis xyz="1 0 0"/>
+      <axis xyz="-1 0 0"/>
       <limit effort="104.0" lower="-2.35" upper="2.35" velocity="1.57"/>
       <dynamics damping="0" friction="0"/>
@@ -329,5 +329,5 @@
       <parent link="${prefix}motor2_link"/>
       <child link="${prefix}motor3_link"/>
-      <axis xyz="-1 0 0"/>
+      <axis xyz="1 0 0"/>
       <limit effort="69" lower="-2.61" upper="2.61" velocity="1.57"/>
       <dynamics damping="0" friction="0"/>
@@ -342,5 +342,5 @@
       <parent link="${prefix}motor3_link"/>
       <child link="${prefix}motor4_link"/>
-      <axis xyz="0 0 1"/>
+      <axis xyz="0 0 -1"/>
       <limit effort="69" lower="-3.14" upper="3.14" velocity="1.57"/>
       <dynamics damping="0" friction="0"/>
@@ -350,5 +350,5 @@
       <parent link="${prefix}motor4_link"/>
       <child link="${prefix}motor5_link"/>
-      <axis xyz="-1 0 0"/>
+      <axis xyz="1 0 0"/>
       <limit effort="34" lower="-2.56" upper="2.56" velocity="1.57"/>
       <dynamics damping="0" friction="0"/>
@@ -363,5 +363,5 @@
       <parent link="${prefix}motor5_link"/>
       <child link="${prefix}motor6_link"/>
-      <axis xyz="0 0 1"/>
+      <axis xyz="0 0 -1"/>
       <limit effort="34" lower="-3.14" upper="3.14" velocity="1.57"/>
       <dynamics damping="0" friction="0"/>
