Commit message: Axis according ROS 2 and real one

File: mara_description/urdf/mara.urdf.xacro (robot description, xacro)
@@ -308,5 +308,5 @@
       <parent link="${prefix}base_robot"/>
       <child link="${prefix}motor1_link"/>
-      <axis xyz="0 0 -1"/>
+      <axis xyz="0 0 1"/>
       <limit effort="104.0" lower="-3.1416" upper="3.1416" velocity="1.57"/>
       <dynamics damping="0" friction="0"/>
@@ -321,5 +321,5 @@
       <parent link="${prefix}motor1_link"/>
       <child link="${prefix}motor2_link"/>
-      <axis xyz="-1 0 0"/>
+      <axis xyz="1 0 0"/>
       <limit effort="104.0" lower="-2.35" upper="2.35" velocity="1.57"/>
       <dynamics damping="0" friction="0"/>
@@ -329,5 +329,5 @@
       <parent link="${prefix}motor2_link"/>
       <child link="${prefix}motor3_link"/>
-      <axis xyz="1 0 0"/>
+      <axis xyz="-1 0 0"/>
       <limit effort="69" lower="-2.61" upper="2.61" velocity="1.57"/>
       <dynamics damping="0" friction="0"/>
@@ -342,5 +342,5 @@
       <parent link="${prefix}motor3_link"/>
       <child link="${prefix}motor4_link"/>
-      <axis xyz="0 0 -1"/>
+      <axis xyz="0 0 1"/>
       <limit effort="69" lower="-3.14" upper="3.14" velocity="1.57"/>
       <dynamics damping="0" friction="0"/>
@@ -350,5 +350,5 @@
       <parent link="${prefix}motor4_link"/>
       <child link="${prefix}motor5_link"/>
-      <axis xyz="1 0 0"/>
+      <axis xyz="-1 0 0"/>
       <limit effort="34" lower="-2.56" upper="2.56" velocity="1.57"/>
       <dynamics damping="0" friction="0"/>
@@ -363,5 +363,5 @@
       <parent link="${prefix}motor5_link"/>
       <child link="${prefix}motor6_link"/>
-      <axis xyz="0 0 -1"/>
+      <axis xyz="0 0 1"/>
       <limit effort="34" lower="-3.14" upper="3.14" velocity="1.57"/>
       <dynamics damping="0" friction="0"/>

Commit message: fix mara_description after having updated the grippers

File: mara_description/urdf/mara.urdf.xacro (robot description, xacro)
@@ -101,5 +101,5 @@
       </visual>
       <collision>
-        <origin rpy="0 0 3.1416" xyz="0 0 0"/>
+        <origin rpy="0 0 0" xyz="0 0 0"/>
         <geometry>
           <mesh filename="package://mara_description/meshes/MARA_T49_Black.dae" scale="0.001 0.001 0.001"/>
@@ -267,36 +267,25 @@
       <selfCollide>True</selfCollide>
     </gazebo>
+    <!-- dummy link with the required tags-->
     <link name="${prefix}motor6_link">
       <inertial>
-        <origin rpy="0 0 0" xyz="0.0 0.0 -0.0173"/>
-        <mass value="0.14"/>
-        <inertia ixx="9.22e-05" ixy="6.35e-7" ixz="2.00e-11" iyy="9.73e-5" iyz="2.36e-9" izz="1.77e-4"/>
-      </inertial>
-      <visual>
-        <origin rpy="0 0 0" xyz="0 0 0"/>
-        <geometry>
-          <mesh filename="package://mara_description/meshes/MARA_GripperAdapter.dae" scale="0.001 0.001 0.001"/>
-        </geometry>
-        <material name="Gazebo/Black">
-          <color rgba="0. 0. 0. 1"/>
-        </material>
-      </visual>
-      <collision>
-        <origin rpy="0 0 0" xyz="0 0 0"/>
-        <geometry>
-          <mesh filename="package://mara_description/meshes/MARA_GripperAdapter.dae" scale="0.001 0.001 0.001"/>
-        </geometry>
-      </collision>
-    </link>
-    <gazebo reference="${prefix}motor6_link">
-      <material>Gazebo/Black</material>
-      <selfCollide>True</selfCollide>
-    </gazebo>
-    <link name="${prefix}ee_link">
-    </link>
-    <gazebo reference="${prefix}ee_link">
-      <material>Gazebo/Blue</material>
-      <selfCollide>False</selfCollide>
-    </gazebo>
+        <origin rpy="0 0 0" xyz="0 0 0"/>
+        <mass value="0.00001"/>
+        <inertia ixx="0" ixy="0" ixz="0" iyy="0" iyz="0" izz="0"/>
+      </inertial>
+      <visual>
+        <origin rpy="0 0 0" xyz="0 0 0"/>
+        <geometry>
+          <sphere radius="0"/>
+        </geometry>
+      </visual>
+      <collision>
+        <origin rpy="0 0 0" xyz="0 0 0"/>
+        <geometry>
+          <sphere radius="0"/>
+        </geometry>
+      </collision>
+    </link>
+    <link name="${prefix}ee_link"/>
     <joint name="${prefix}joint_bases" type="fixed">
       <origin rpy="0 0 0" xyz="0 0 0.04"/>

File: mara_description/urdf/mara_gazebo.urdf.xacro (robot description, xacro)
@@ -14,12 +14,9 @@
     		<joint_name>motor5</joint_name>
         <joint_name>motor6</joint_name>
-        <joint_name>left_inner_knuckle_joint</joint_name>
-        <joint_name>left_outer_knuckle_joint</joint_name>
-        <joint_name>left_outer_finger_joint</joint_name>
-        <joint_name>left_inner_finger_joint</joint_name>
-        <joint_name>right_inner_knuckle_joint</joint_name>
-        <joint_name>right_outer_knuckle_joint</joint_name>
-        <joint_name>right_outer_finger_joint</joint_name>
-        <joint_name>right_inner_finger_joint</joint_name>
+        <joint_name>robotiq_arg2f_base_to_left_inner_knuckle</joint_name>
+        <joint_name>robotiq_arg2f_base_to_left_outer_knuckle</joint_name>
+        <joint_name>left_outer_knuckle_to_finger</joint_name>
+        <joint_name>left_outer_finger_to_inner</joint_name>
+        <joint_name>robotiq_arg2f_base_to_right_inner_knuckle</joint_name>
     	</plugin>
       <plugin name="hros_actuation_servomotor_000000000001" filename="libmara_gazebo_joint_plugin.so">

File: mara_description/urdf/mara_robot_gripper_140.urdf.xacro (robot description, xacro)
@@ -1,5 +1,4 @@
 <?xml version="1.0"?>
-<robot xmlns:xacro="http://ros.org/wiki/xacro"
-       name="mara" >
+<robot xmlns:xacro="http://ros.org/wiki/xacro" name="mara" >
   <!-- common stuff -->
   <xacro:include filename="$(find mara_description)/urdf/mara_gazebo.urdf.xacro" />
@@ -8,26 +7,86 @@
   <!-- robotiq 140 gripper -->
   <xacro:include filename="$(find robotiq_140_gripper_description)/urdf/robotiq_140.urdf.xacro" />
-  <!-- <xacro:include filename="$(find mara_description)/urdf/camera_top.urdf.xacro" /> -->
   <xacro:include filename="$(find mara_description)/urdf/table.urdf.xacro" />
   <!-- arm -->
-  <xacro:mara_robot prefix="" ee_link_distance="0.24"/>
+  <xacro:mara_robot prefix="" ee_link_distance="0.24497"/>
   <xacro:robotiq_gripper prefix="mara" />
-  <!-- <xacro:mara_camera_top prefix="" /> -->
   <xacro:table prefix="" />
   <link name="world" />
-  <joint name="end_effector_adapter_to_robotiq" type="fixed">
-    <origin rpy="0 0 1.57" xyz=" 0 0 0.0"/>
-    <parent link="motor6_link"/>
-    <child link="robotiq_adapter_link"/>
-  </joint>
-  <joint name="world_to_table_joint" type="fixed">
-    <origin rpy="0 0 0" xyz="0 0 0.02"/>
+  <link name="gripper_adapter">
+    <inertial>
+      <origin rpy="0 0 0" xyz="8.625E-08 -4.6583E-06 0.03145"/>
+      <mass value="0.13969"/>
+      <inertia ixx="91283.23E-9" ixy="634.87E-9" ixz="-0.02E-9" iyy="97239.94E-9" iyz="93.72E-9" izz="175963.64E-9"/>
+    </inertial>
+    <visual>
+      <origin rpy="0 0 0" xyz="0 0 0"/>
+      <geometry>
+        <mesh filename="package://mara_description/meshes/gripper_adapter.dae" scale="0.001 0.001 0.001"/>
+      </geometry>
+      <material name="Gazebo/Wood">
+        <color rgba="0. 0. 0. 1"/>
+      </material>
+    </visual>
+    <collision>
+      <origin rpy="0 0 0" xyz="0 0 0"/>
+      <geometry>
+        <mesh filename="package://mara_description/meshes/gripper_adapter.dae" scale="0.001 0.001 0.001"/>
+      </geometry>
+    </collision>
+  </link>
+  <gazebo reference="gripper_adapter">
+    <material>Gazebo/Black</material>
+    <selfCollide>True</selfCollide>
+  </gazebo>
+  <link name="robotiq_adapter_link">
+    <inertial>
+      <origin xyz="8.625E-08 -4.6583E-06 0.03145" rpy="0 0 0" />
+      <mass value="0.22652" />
+      <inertia ixx="0.00020005" ixy="0" ixz="0" iyy="0.00017832" iyz="0" izz="0.00013478" />
+    </inertial>
+    <visual>
+      <origin xyz="0 0 0" rpy="0 0 0" />
+      <geometry>
+        <mesh filename="package://mara_description/meshes/robotiq_adapter.dae" scale="0.001 0.001 0.001"/>
+      </geometry>
+      <material name="Gazebo/Black">
+        <color rgba="0.0 0.0 0.0 1" />
+      </material>
+    </visual>
+    <collision>
+      <origin xyz="0 0 0" rpy="0 0 0" />
+      <geometry>
+        <mesh filename="package://mara_description/meshes/robotiq_adapter.dae" scale="0.001 0.001 0.001"/>
+      </geometry>
+    </collision>
+  </link>
+  <gazebo reference="robotiq_adapter_link">
+    <material>Gazebo/Black</material>
+    <selfCollide>False</selfCollide>
+  </gazebo>
+  <joint name="world_to_table" type="fixed">
+    <origin rpy="0 0 0" xyz="0 0 0"/>
     <parent link="world"/>
     <child link="table"/>
   </joint>
-  <joint name="table_to_base_joint" type="fixed">
+  <joint name="table_to_base" type="fixed">
     <origin rpy="0 0 0" xyz="0 0 0.62"/>
     <parent link="table"/>
     <child link="base_link"/>
   </joint>
+  <joint name="motor6_to_gripper_adapter" type="fixed">
+    <origin rpy="0 0 0" xyz=" 0 0 -0.02026"/>
+    <parent link="motor6_link"/>
+    <child link="gripper_adapter"/>
+  </joint>
+  <joint name="gripper_adapter_to_robotiq_adapter" type="fixed">
+    <origin rpy="0 0 0" xyz=" 0 0 0.05679"/>
+    <parent link="gripper_adapter"/>
+    <child link="robotiq_adapter_link"/>
+  </joint>
+  <joint name="robotiq_adapter_to_arg2f_base" type="fixed">
+    <origin rpy="0 0 0" xyz=" 0 0 0"/>
+    <parent link="robotiq_adapter_link"/>
+    <child link="robotiq_arg2f_base_link"/>
+  </joint>
 </robot>

File: mara_description/urdf/mara_robot_gripper_140_no_table.urdf.xacro (robot description, xacro)
@@ -8,16 +8,78 @@
   <xacro:include filename="$(find robotiq_140_gripper_description)/urdf/robotiq_140.urdf.xacro" />
   <!-- arm -->
-  <xacro:mara_robot prefix="" ee_link_distance="0.24"/>
+  <xacro:mara_robot prefix="" ee_link_distance="0.24497"/>
   <xacro:robotiq_gripper prefix="mara" />
   <link name="world" />
-  <joint name="end_effector_adapter_to_robotiq" type="fixed">
-    <origin rpy="0 0 1.57" xyz=" 0 0 0.0"/>
-    <parent link="motor6_link"/>
-    <child link="robotiq_adapter_link"/>
-  </joint>
-  <joint name="world_to_base_joint" type="fixed">
-    <origin rpy="0 0 0" xyz="0 0 0.02"/>
+  <link name="gripper_adapter">
+    <inertial>
+      <origin rpy="0 0 0" xyz="8.625E-08 -4.6583E-06 0.03145"/>
+      <mass value="0.13969"/>
+      <inertia ixx="91283.23E-9" ixy="634.87E-9" ixz="-0.02E-9" iyy="97239.94E-9" iyz="93.72E-9" izz="175963.64E-9"/>
+    </inertial>
+    <visual>
+      <origin rpy="0 0 0" xyz="0 0 0"/>
+      <geometry>
+        <mesh filename="package://mara_description/meshes/gripper_adapter.dae" scale="0.001 0.001 0.001"/>
+      </geometry>
+      <material name="Gazebo/Wood">
+        <color rgba="0. 0. 0. 1"/>
+      </material>
+    </visual>
+    <collision>
+      <origin rpy="0 0 0" xyz="0 0 0"/>
+      <geometry>
+        <mesh filename="package://mara_description/meshes/gripper_adapter.dae" scale="0.001 0.001 0.001"/>
+      </geometry>
+    </collision>
+  </link>
+  <gazebo reference="gripper_adapter">
+    <material>Gazebo/Black</material>
+    <selfCollide>True</selfCollide>
+  </gazebo>
+  <link name="robotiq_adapter_link">
+    <inertial>
+      <origin xyz="8.625E-08 -4.6583E-06 0.03145" rpy="0 0 0" />
+      <mass value="0.22652" />
+      <inertia ixx="0.00020005" ixy="0" ixz="0" iyy="0.00017832" iyz="0" izz="0.00013478" />
+    </inertial>
+    <visual>
+      <origin xyz="0 0 0" rpy="0 0 0" />
+      <geometry>
+        <mesh filename="package://mara_description/meshes/robotiq_adapter.dae" scale="0.001 0.001 0.001"/>
+      </geometry>
+      <material name="Gazebo/Black">
+        <color rgba="0.0 0.0 0.0 1" />
+      </material>
+    </visual>
+    <collision>
+      <origin xyz="0 0 0" rpy="0 0 0" />
+      <geometry>
+        <mesh filename="package://mara_description/meshes/robotiq_adapter.dae" scale="0.001 0.001 0.001"/>
+      </geometry>
+    </collision>
+  </link>
+  <gazebo reference="robotiq_adapter_link">
+    <material>Gazebo/Black</material>
+    <selfCollide>False</selfCollide>
+  </gazebo>
+  <joint name="world_to_table" type="fixed">
+    <origin rpy="0 0 0" xyz="0 0 0"/>
     <parent link="world"/>
     <child link="base_link"/>
   </joint>
+  <joint name="motor6_to_gripper_adapter" type="fixed">
+    <origin rpy="0 0 0" xyz=" 0 0 -0.02026"/>
+    <parent link="motor6_link"/>
+    <child link="gripper_adapter"/>
+  </joint>
+  <joint name="gripper_adapter_to_robotiq_adapter" type="fixed">
+    <origin rpy="0 0 0" xyz=" 0 0 0.05679"/>
+    <parent link="gripper_adapter"/>
+    <child link="robotiq_adapter_link"/>
+  </joint>
+  <joint name="robotiq_adapter_to_arg2f_base" type="fixed">
+    <origin rpy="0 0 0" xyz=" 0 0 0"/>
+    <parent link="robotiq_adapter_link"/>
+    <child link="robotiq_arg2f_base_link"/>
+  </joint>
 </robot>

File: mara_description/urdf/mara_robot_gripper_85.urdf.xacro (robot description, xacro)
@@ -1,5 +1,4 @@
 <?xml version="1.0"?>
-<robot xmlns:xacro="http://ros.org/wiki/xacro"
-       name="mara" >
+<robot xmlns:xacro="http://ros.org/wiki/xacro" name="mara" >
   <!-- common stuff -->
   <xacro:include filename="$(find mara_description)/urdf/mara_gazebo.urdf.xacro" />
@@ -10,22 +9,84 @@
   <xacro:include filename="$(find mara_description)/urdf/table.urdf.xacro" />
   <!-- arm -->
-  <xacro:mara_robot prefix="" ee_link_distance="0.165"/>
+  <xacro:mara_robot prefix="" ee_link_distance="0.18491"/>
   <xacro:robotiq_85 prefix="mara" />
   <xacro:table prefix="" />
   <link name="world" />
-  <joint name="end_effector_adapter_to_robotiq" type="fixed">
-    <origin rpy="0 0 0" xyz=" 0 0 0.0"/>
-    <parent link="motor6_link"/>
-    <child link="robotiq_adapter_link"/>
-  </joint>
-  <joint name="world_to_table_joint" type="fixed">
-    <origin rpy="0 0 0" xyz="0 0 0.02"/>
+  <link name="gripper_adapter">
+    <inertial>
+      <origin rpy="0 0 0" xyz="8.625E-08 -4.6583E-06 0.03145"/>
+      <mass value="0.13969"/>
+      <inertia ixx="91283.23E-9" ixy="634.87E-9" ixz="-0.02E-9" iyy="97239.94E-9" iyz="93.72E-9" izz="175963.64E-9"/>
+    </inertial>
+    <visual>
+      <origin rpy="0 0 0" xyz="0 0 0"/>
+      <geometry>
+        <mesh filename="package://mara_description/meshes/gripper_adapter.dae" scale="0.001 0.001 0.001"/>
+      </geometry>
+      <material name="Gazebo/Wood">
+        <color rgba="0. 0. 0. 1"/>
+      </material>
+    </visual>
+    <collision>
+      <origin rpy="0 0 0" xyz="0 0 0"/>
+      <geometry>
+        <mesh filename="package://mara_description/meshes/gripper_adapter.dae" scale="0.001 0.001 0.001"/>
+      </geometry>
+    </collision>
+  </link>
+  <gazebo reference="gripper_adapter">
+    <material>Gazebo/Black</material>
+    <selfCollide>True</selfCollide>
+  </gazebo>
+  <link name="robotiq_adapter_link">
+    <inertial>
+      <origin xyz="8.625E-08 -4.6583E-06 0.03145" rpy="0 0 0" />
+      <mass value="0.22652" />
+      <inertia ixx="0.00020005" ixy="0" ixz="0" iyy="0.00017832" iyz="0" izz="0.00013478" />
+    </inertial>
+    <visual>
+      <origin xyz="0 0 0" rpy="0 0 0" />
+      <geometry>
+        <mesh filename="package://mara_description/meshes/robotiq_adapter.dae" scale="0.001 0.001 0.001"/>
+      </geometry>
+      <material name="Gazebo/Black">
+        <color rgba="0.0 0.0 0.0 1" />
+      </material>
+    </visual>
+    <collision>
+      <origin xyz="0 0 0" rpy="0 0 0" />
+      <geometry>
+        <mesh filename="package://mara_description/meshes/robotiq_adapter.dae" scale="0.001 0.001 0.001"/>
+      </geometry>
+    </collision>
+  </link>
+  <gazebo reference="robotiq_adapter_link">
+    <material>Gazebo/Black</material>
+    <selfCollide>False</selfCollide>
+  </gazebo>
+  <joint name="world_to_table" type="fixed">
+    <origin rpy="0 0 0" xyz="0 0 0"/>
     <parent link="world"/>
     <child link="table"/>
   </joint>
-  <joint name="table_to_base_joint" type="fixed">
+  <joint name="table_to_base" type="fixed">
     <origin rpy="0 0 0" xyz="0 0 0.62"/>
     <parent link="table"/>
     <child link="base_link"/>
   </joint>
+  <joint name="motor6_to_gripper_adapter" type="fixed">
+    <origin rpy="0 0 0" xyz=" 0 0 -0.02026"/>
+    <parent link="motor6_link"/>
+    <child link="gripper_adapter"/>
+  </joint>
+  <joint name="gripper_adapter_to_robotiq_adapter" type="fixed">
+    <origin rpy="0 0 0" xyz=" 0 0 0.05679"/>
+    <parent link="gripper_adapter"/>
+    <child link="robotiq_adapter_link"/>
+  </joint>
+  <joint name="robotiq_adapter_to_arg2f_base" type="fixed">
+    <origin rpy="0 0 0" xyz=" 0 0 0"/>
+    <parent link="robotiq_adapter_link"/>
+    <child link="robotiq_arg2f_base_link"/>
+  </joint>
 </robot>

File: mara_description/urdf/mara_robot_gripper_hande.urdf.xacro (robot description, xacro)
@@ -1,22 +1,68 @@
 <?xml version="1.0"?>
-<robot xmlns:xacro="http://ros.org/wiki/xacro"
-       name="mara" >
+<robot xmlns:xacro="http://ros.org/wiki/xacro" name="mara" >
   <!-- common stuff -->
   <xacro:include filename="$(find mara_description)/urdf/mara_gazebo.urdf.xacro" />
   <!-- mara -->
   <xacro:include filename="$(find mara_description)/urdf/mara.urdf.xacro" />
-  <!-- robotiq 140 gripper -->
+  <!-- robotiq hande gripper -->
   <xacro:include filename="$(find robotiq_hande_gripper_description)/urdf/robotiq_hande.urdf.xacro" />
   <xacro:include filename="$(find mara_description)/urdf/table.urdf.xacro" />
   <!-- arm -->
-  <xacro:mara_robot prefix="" ee_link_distance="0.18"/>
+  <xacro:mara_robot prefix="" ee_link_distance="0.18253"/>
   <xacro:robotiq_hande prefix="mara" />
   <xacro:table prefix="" />
   <link name="world" />
-  <joint name="end_effector_adapter_to_robotiq" type="fixed">
-    <origin rpy="0 0 0" xyz=" 0 0 0.0"/>
-    <parent link="motor6_link"/>
-    <child link="robotiq_adapter_link"/>
-  </joint>
+  <link name="gripper_adapter">
+    <inertial>
+      <origin rpy="0 0 0" xyz="8.625E-08 -4.6583E-06 0.03145"/>
+      <mass value="0.13969"/>
+      <inertia ixx="91283.23E-9" ixy="634.87E-9" ixz="-0.02E-9" iyy="97239.94E-9" iyz="93.72E-9" izz="175963.64E-9"/>
+    </inertial>
+    <visual>
+      <origin rpy="0 0 0" xyz="0 0 0"/>
+      <geometry>
+        <mesh filename="package://mara_description/meshes/gripper_adapter.dae" scale="0.001 0.001 0.001"/>
+      </geometry>
+      <material name="Gazebo/Wood">
+        <color rgba="0. 0. 0. 1"/>
+      </material>
+    </visual>
+    <collision>
+      <origin rpy="0 0 0" xyz="0 0 0"/>
+      <geometry>
+        <mesh filename="package://mara_description/meshes/gripper_adapter.dae" scale="0.001 0.001 0.001"/>
+      </geometry>
+    </collision>
+  </link>
+  <gazebo reference="gripper_adapter">
+    <material>Gazebo/Black</material>
+    <selfCollide>False</selfCollide>
+  </gazebo>
+  <link name="robotiq_adapter_link">
+    <inertial>
+      <origin xyz="8.625E-08 -4.6583E-06 0.03145" rpy="0 0 0" />
+      <mass value="0.22652" />
+      <inertia ixx="0.00020005" ixy="0" ixz="0" iyy="0.00017832" iyz="0" izz="0.00013478" />
+    </inertial>
+    <visual>
+      <origin xyz="0 0 0" rpy="0 0 0" />
+      <geometry>
+        <mesh filename="package://mara_description/meshes/robotiq_adapter.dae" scale="0.001 0.001 0.001"/>
+      </geometry>
+      <material name="Gazebo/Black">
+        <color rgba="0.0 0.0 0.0 1" />
+      </material>
+    </visual>
+    <collision>
+      <origin xyz="0 0 0" rpy="0 0 0" />
+      <geometry>
+        <mesh filename="package://mara_description/meshes/robotiq_adapter.dae" scale="0.001 0.001 0.001"/>
+      </geometry>
+    </collision>
+  </link>
+  <gazebo reference="robotiq_adapter_link">
+    <material>Gazebo/Black</material>
+    <selfCollide>False</selfCollide>
+  </gazebo>
   <joint name="world_to_table_joint" type="fixed">
     <origin rpy="0 0 0" xyz="0 0 0.02"/>
@@ -29,3 +75,18 @@
     <child link="base_link"/>
   </joint>
+  <joint name="motor6_to_gripper_adapter" type="fixed">
+    <origin rpy="0 0 0" xyz=" 0 0 0.0"/>
+    <parent link="motor6_link"/>
+    <child link="gripper_adapter"/>
+  </joint>
+  <joint name="gripper_adapter_to_robotiq_adapter" type="fixed">
+    <origin rpy="0 0 0" xyz=" 0 0 0.0"/>
+    <parent link="gripper_adapter"/>
+    <child link="robotiq_adapter_link"/>
+  </joint>
+  <joint name="robotiq_adapter_to_hande_base" type="fixed">
+    <origin rpy="0 0 0" xyz=" 0 0 0"/>
+    <parent link="robotiq_adapter_link"/>
+    <child link="robotiq_hande_base_link"/>
+  </joint>
 </robot>

Commit message: Update mara.urdf.xacro

File: mara_description/urdf/mara.urdf.xacro (robot description, xacro)
@@ -101,5 +101,5 @@
       </visual>
       <collision>
-        <origin rpy="0 0 3.1416" xyz="0 0 0"/>
+        <origin rpy="0 0 0" xyz="0 0 0"/>
         <geometry>
           <mesh filename="package://mara_description/meshes/MARA_T49_Black.dae" scale="0.001 0.001 0.001"/>
