Commit message: enable multiple S140 robots

File: mara_description/urdf/mara.urdf.xacro (robot description, xacro)
@@ -6,5 +6,5 @@
   <xacro:include filename="$(find mara_description)/urdf/mara.transmission.xacro" />
   <xacro:include filename="$(find mara_description)/urdf/mara_gazebo.urdf.xacro" />
-  <xacro:macro name="mara_robot"  params="prefix ee_link_distance">
+  <xacro:macro name="mara_robot"  params="prefix ee_link_distance MAC1 MAC2 MAC3">
     <link name="${prefix}base_link">
       <inertial>
@@ -362,11 +362,11 @@
     </joint>
     <link name="${prefix}tool0"/>
-    <joint name="${prefix}${prefix}motor6_link-tool0_fixed_joint" type="fixed">
+    <joint name="${prefix}motor6_link-tool0_fixed_joint" type="fixed">
       <origin rpy="0 -1.57 0" xyz="0 0.0 ${ee_link_distance}"/>
-      <parent link="${prefix}${prefix}motor6_link"/>
+      <parent link="${prefix}motor6_link"/>
       <child link="${prefix}tool0"/>
     </joint>
     <xacro:mara_transmission prefix="${prefix}"/>
-    <xacro:mara_gazebo prefix="${prefix}"/>
+    <xacro:mara_gazebo prefix="${prefix}" MAC1="${MAC1}" MAC2="${MAC2}" MAC3="${MAC3}"/>
   </xacro:macro>
 </robot>

File: mara_description/urdf/mara_gazebo.urdf.xacro (robot description, xacro)
@@ -1,5 +1,5 @@
 <?xml version="1.0"?>
 <robot xmlns:xacro="http://ros.org/wiki/xacro">
-  <xacro:macro name="mara_gazebo" params="prefix">
+  <xacro:macro name="mara_gazebo" params="prefix MAC1 MAC2 MAC3">
     <gazebo>
       <plugin name="mara_joint_state" filename="libgazebo_ros_joint_state_publisher.so">
@@ -8,28 +8,28 @@
         </ros>
         <update_rate>25</update_rate>
-        <joint_name>motor1</joint_name>
-        <joint_name>motor2</joint_name>
-        <joint_name>motor3</joint_name>
-        <joint_name>motor4</joint_name>
-        <joint_name>motor5</joint_name>
-        <joint_name>motor6</joint_name>
-        <joint_name>joint_finger</joint_name>
+        <joint_name>${prefix}motor1</joint_name>
+        <joint_name>${prefix}motor2</joint_name>
+        <joint_name>${prefix}motor3</joint_name>
+        <joint_name>${prefix}motor4</joint_name>
+        <joint_name>${prefix}motor5</joint_name>
+        <joint_name>${prefix}motor6</joint_name>
+        <joint_name>${prefix}joint_finger</joint_name>
       </plugin>
-      <plugin name="hros_actuation_servomotor_000000000001" filename="libmara_gazebo_joint_plugin.so">
+      <plugin name="hros_actuation_servomotor${MAC1}" filename="libmara_gazebo_joint_plugin.so">
         <ros></ros>
-        <axis1>motor2</axis1>
-        <axis2>motor1</axis2>
+        <axis1>${prefix}motor2</axis1>
+        <axis2>${prefix}motor1</axis2>
         <type>series14</type>
       </plugin>
-      <plugin name="hros_actuation_servomotor_000000000002" filename="libmara_gazebo_joint_plugin.so">
+      <plugin name="hros_actuation_servomotor${MAC2}" filename="libmara_gazebo_joint_plugin.so">
         <ros></ros>
-        <axis1>motor3</axis1>
-        <axis2>motor4</axis2>
+        <axis1>${prefix}motor3</axis1>
+        <axis2>${prefix}motor4</axis2>
         <type>series17</type>
       </plugin>
-      <plugin name="hros_actuation_servomotor_000000000003" filename="libmara_gazebo_joint_plugin.so">
+      <plugin name="hros_actuation_servomotor${MAC3}" filename="libmara_gazebo_joint_plugin.so">
         <ros></ros>
-        <axis1>motor5</axis1>
-        <axis2>motor6</axis2>
+        <axis1>${prefix}motor5</axis1>
+        <axis2>${prefix}motor6</axis2>
         <type>series20</type>
       </plugin>

File: robotiq_140_gripper_description/urdf/robotiq_140.urdf.xacro (robot description, xacro)
@@ -1,6 +1,6 @@
 <?xml version="1.0"?>
 <robot xmlns:xacro="http://ros.org/wiki/xacro">
-  <xacro:macro name="robotiq_gripper"  params="prefix">
-    <link name="robotiq_arg2f_base_link">
+  <xacro:macro name="robotiq_gripper"  params="prefix MAC">
+    <link name="${prefix}robotiq_arg2f_base_link">
       <inertial>
         <origin xyz="-0.00013 0.00011 0.03284" rpy="0 0 0" />
@@ -24,9 +24,9 @@
       </collision>
     </link>
-    <gazebo reference="robotiq_arg2f_base_link">
-      <material>Gazebo/Black</material>
-      <selfCollide>True</selfCollide>
-    </gazebo>
-    <link name="left_outer_knuckle">
+    <gazebo reference="${prefix}robotiq_arg2f_base_link">
+      <material>Gazebo/Black</material>
+      <selfCollide>True</selfCollide>
+    </gazebo>
+    <link name="${prefix}left_outer_knuckle">
       <inertial>
         <origin xyz="0.01616 0 -0.00133" rpy="0 0 0" />
@@ -50,9 +50,9 @@
       </collision>
     </link>
-    <gazebo reference="left_outer_knuckle">
+    <gazebo reference="${prefix}left_outer_knuckle">
       <material>Gazebo/Grey</material>
       <selfCollide>True</selfCollide>
     </gazebo>
-    <link name="right_outer_knuckle">
+    <link name="${prefix}right_outer_knuckle">
       <inertial>
         <origin xyz="-0.01616 0 -0.00133" rpy="0 0 0" />
@@ -76,9 +76,9 @@
       </collision>
     </link>
-    <gazebo reference="right_outer_knuckle">
+    <gazebo reference="${prefix}right_outer_knuckle">
       <material>Gazebo/Grey</material>
       <selfCollide>True</selfCollide>
     </gazebo>
-    <link name="left_inner_knuckle">
+    <link name="${prefix}left_inner_knuckle">
       <inertial>
         <origin xyz="0.03332 0 0.0379" rpy="0 0 0" />
@@ -102,9 +102,9 @@
       </collision>
     </link>
-    <gazebo reference="left_inner_knuckle">
+    <gazebo reference="${prefix}left_inner_knuckle">
       <material>Gazebo/Black</material>
       <selfCollide>False</selfCollide>
     </gazebo>
-    <link name="right_inner_knuckle">
+    <link name="${prefix}right_inner_knuckle">
       <inertial>
         <origin xyz="-0.03332 0 0.0379" rpy="0 0 0" />
@@ -128,9 +128,9 @@
       </collision>
     </link>
-    <gazebo reference="right_inner_knuckle">
+    <gazebo reference="${prefix}right_inner_knuckle">
       <material>Gazebo/Black</material>
       <selfCollide>False</selfCollide>
     </gazebo>
-    <link name="left_inner_finger">
+    <link name="${prefix}left_inner_finger">
       <inertial>
         <origin xyz="-0.01563 0 0.02522" rpy="0 0 0" />
@@ -154,9 +154,9 @@
       </collision>
     </link>
-    <gazebo reference="left_inner_finger">
+    <gazebo reference="${prefix}left_inner_finger">
       <material>Gazebo/Black</material>
       <selfCollide>False</selfCollide>
     </gazebo>
-    <link name="right_inner_finger">
+    <link name="${prefix}right_inner_finger">
       <inertial>
         <origin xyz="0.01563 0 0.02522" rpy="0 0 0" />
@@ -180,9 +180,9 @@
       </collision>
     </link>
-    <gazebo reference="right_inner_finger">
+    <gazebo reference="${prefix}right_inner_finger">
       <material>Gazebo/Black</material>
       <selfCollide>False</selfCollide>
     </gazebo>
-    <link name="left_outer_finger">
+    <link name="${prefix}left_outer_finger">
       <inertial>
         <origin xyz="0.01482 0 0.03451" rpy="0 0 0" />
@@ -206,9 +206,9 @@
       </collision>
     </link>
-    <gazebo reference="left_outer_finger">
-      <material>Gazebo/Black</material>
-      <selfCollide>True</selfCollide>
-    </gazebo>
-    <link name="right_outer_finger">
+    <gazebo reference="${prefix}left_outer_finger">
+      <material>Gazebo/Black</material>
+      <selfCollide>True</selfCollide>
+    </gazebo>
+    <link name="${prefix}right_outer_finger">
       <inertial>
         <origin xyz="-0.01482 0 0.03451" rpy="0 0 0" />
@@ -232,70 +232,70 @@
       </collision>
     </link>
-    <gazebo reference="right_outer_finger">
-      <material>Gazebo/Black</material>
-      <selfCollide>True</selfCollide>
-    </gazebo>
-    <joint name="robotiq_arg2f_base_to_left_outer_knuckle" type="revolute">
+    <gazebo reference="${prefix}right_outer_finger">
+      <material>Gazebo/Black</material>
+      <selfCollide>True</selfCollide>
+    </gazebo>
+    <joint name="robotiq_arg2f_base_to_${prefix}left_outer_knuckle" type="revolute">
       <origin xyz="0.0306 0 0.05466" rpy="0 0 0" />
-      <parent link="robotiq_arg2f_base_link" />
-      <child link="left_outer_knuckle" />
+      <parent link="${prefix}robotiq_arg2f_base_link" />
+      <child link="${prefix}left_outer_knuckle" />
       <axis xyz="0 -1 0" />
       <limit lower="0" upper="0.78574722925"  velocity="2.0" effort="18.65" />
-      <mimic joint="joint_finger" multiplier="1" offset="0"/>
-    </joint>
-    <joint name="joint_finger" type="revolute">
+      <mimic joint="${prefix}joint_finger" multiplier="1" offset="0"/>
+    </joint>
+    <joint name="${prefix}joint_finger" type="revolute">
       <origin xyz="-0.0306 0 0.05466" rpy="0 0 0" />
-      <parent link="robotiq_arg2f_base_link" />
-      <child link="right_outer_knuckle" />
+      <parent link="${prefix}robotiq_arg2f_base_link" />
+      <child link="${prefix}right_outer_knuckle" />
       <axis xyz="0 1 0" />
       <limit lower="0" upper="0.78574722925" velocity="3.54" effort="18.65" />
     </joint>
-    <joint name="robotiq_arg2f_base_to_left_inner_knuckle" type="revolute">
+    <joint name="robotiq_arg2f_base_to_${prefix}left_inner_knuckle" type="revolute">
       <origin xyz="0.0127 0 0.06118" rpy="0 0 0" />
-      <parent link="robotiq_arg2f_base_link" />
-      <child link="left_inner_knuckle" />
+      <parent link="${prefix}robotiq_arg2f_base_link" />
+      <child link="${prefix}left_inner_knuckle" />
       <axis xyz="0 -1 0" />
       <limit lower="0" upper="0.78574722925" velocity="3.54" effort="18.65" />
-      <mimic joint="joint_finger" multiplier="1" offset="0"/>
-    </joint>
-    <joint name="robotiq_arg2f_base_to_right_inner_knuckle" type="revolute">
+      <mimic joint="${prefix}joint_finger" multiplier="1" offset="0"/>
+    </joint>
+    <joint name="robotiq_arg2f_base_to_${prefix}right_inner_knuckle" type="revolute">
       <origin xyz="-0.0127 0 0.06118" rpy="0 0 0" />
-      <parent link="robotiq_arg2f_base_link" />
-      <child link="right_inner_knuckle" />
+      <parent link="${prefix}robotiq_arg2f_base_link" />
+      <child link="${prefix}right_inner_knuckle" />
       <axis xyz="0 1 0" />
       <limit lower="0" upper="0.78574722925" velocity="3.54" effort="18.65" />
-      <mimic joint="joint_finger" multiplier="1" offset="0"/>
-    </joint>
-    <joint name="left_outer_knuckle_to_finger" type="fixed">
+      <mimic joint="${prefix}joint_finger" multiplier="1" offset="0"/>
+    </joint>
+    <joint name="${prefix}left_outer_knuckle_to_finger" type="fixed">
       <origin xyz="0.03142 0 -0.00453" rpy="0 0 0" />
-      <parent link="left_outer_knuckle" />
-      <child link="left_outer_finger" />
-    </joint>
-    <joint name="right_outer_knuckle_to_finger" type="fixed">
+      <parent link="${prefix}left_outer_knuckle" />
+      <child link="${prefix}left_outer_finger" />
+    </joint>
+    <joint name="${prefix}right_outer_knuckle_to_finger" type="fixed">
       <origin xyz="-0.03142 0 -0.00453" rpy="0 0 0" />
-      <parent link="right_outer_knuckle" />
-      <child link="right_outer_finger" />
-    </joint>
-    <joint name="left_outer_finger_to_inner" type="revolute">
+      <parent link="${prefix}right_outer_knuckle" />
+      <child link="${prefix}right_outer_finger" />
+    </joint>
+    <joint name="${prefix}left_outer_finger_to_inner" type="revolute">
       <origin xyz="0.03543 0 0.0789" rpy="0 0 0" />
-      <parent link="left_outer_finger" />
-      <child link="left_inner_finger" />
+      <parent link="${prefix}left_outer_finger" />
+      <child link="${prefix}left_inner_finger" />
       <axis xyz="0 1 0" />
       <limit lower="0" upper="0.78574722925" velocity="3.54" effort="18.65" />
-      <mimic joint="joint_finger" multiplier="1" offset="0"/>
-    </joint>
-    <joint name="right_outer_finger_to_inner" type="revolute">
+      <mimic joint="${prefix}joint_finger" multiplier="1" offset="0"/>
+    </joint>
+    <joint name="${prefix}right_outer_finger_to_inner" type="revolute">
       <origin xyz="-0.03543 0 0.0789" rpy="0 0 0" />
-      <parent link="right_outer_finger" />
-      <child link="right_inner_finger" />
+      <parent link="${prefix}right_outer_finger" />
+      <child link="${prefix}right_inner_finger" />
       <axis xyz="0 -1 0" />
       <limit lower="0" upper="0.78574722925" velocity="3.54" effort="18.65" />
-      <mimic joint="joint_finger" multiplier="1" offset="0"/>
+      <mimic joint="${prefix}joint_finger" multiplier="1" offset="0"/>
     </joint>
     <gazebo>
-      <joint name="left_inner_knuckle_to_finger" type="revolute">
+      <joint name="${prefix}left_inner_knuckle_to_finger" type="revolute">
         <pose frame="">-0.0179 0 0.00652 0 0 0</pose>
-        <parent>${prefix}::left_inner_knuckle</parent>
-        <child>${prefix}::left_inner_finger</child>
+        <parent>${prefix}left_inner_knuckle</parent>
+        <child>${prefix}left_inner_finger</child>
         <axis>
           <xyz>0 1 0</xyz>
@@ -308,8 +308,8 @@
         </axis>
       </joint>
-      <joint name="right_inner_knuckle_to_finger" type="revolute">
+      <joint name="${prefix}right_inner_knuckle_to_finger" type="revolute">
         <pose frame="">0.0179 0 0.00652 0 0 0</pose>
-        <parent>${prefix}::right_inner_knuckle</parent>
-        <child>${prefix}::right_inner_finger</child>
+        <parent>${prefix}right_inner_knuckle</parent>
+        <child>${prefix}right_inner_finger</child>
         <axis>
           <xyz>0 -1 0</xyz>
@@ -322,12 +322,12 @@
         </axis>
       </joint>
-      <plugin filename="librobotiq_gripper_gazebo_plugin.so" name="robotiq_140_gripper">
+      <plugin filename="librobotiq_gripper_gazebo_plugin.so" name="hrim_actuator_gripper${MAC}">
         <kp>1000</kp>
         <ki>0.1</ki>
         <kd>0.01</kd>
-        <joint>robotiq_arg2f_base_to_left_inner_knuckle</joint>
-        <joint>robotiq_arg2f_base_to_left_outer_knuckle</joint>
-        <joint>robotiq_arg2f_base_to_right_inner_knuckle</joint>
-        <joint>joint_finger</joint>
+        <joint>robotiq_arg2f_base_to_${prefix}left_inner_knuckle</joint>
+        <joint>robotiq_arg2f_base_to_${prefix}left_outer_knuckle</joint>
+        <joint>robotiq_arg2f_base_to_${prefix}right_inner_knuckle</joint>
+        <joint>${prefix}joint_finger</joint>
       </plugin>
     </gazebo>
