Commit message: enable multiple S85 and hande robots

File: mara_description/urdf/mara_robot_gripper_85.urdf.xacro (robot description, xacro)
@@ -9,6 +9,6 @@
   <xacro:include filename="$(find mara_description)/urdf/table.urdf.xacro" />
   <!-- arm -->
-  <xacro:mara_robot prefix="" ee_link_distance="0.18491"/>
-  <xacro:robotiq_85 prefix="mara" />
+  <xacro:mara_robot prefix="" ee_link_distance="0.18491" MAC1="_000000000001" MAC2="_000000000002" MAC3="_000000000003"/>
+  <xacro:robotiq_85 prefix="" MAC="_000000000004"/>
   <xacro:table prefix="" />
   <link name="world" />

File: mara_description/urdf/mara_robot_gripper_hande.urdf.xacro (robot description, xacro)
@@ -9,6 +9,6 @@
   <xacro:include filename="$(find mara_description)/urdf/table.urdf.xacro" />
   <!-- arm -->
-  <xacro:mara_robot prefix="" ee_link_distance="0.18253"/>
-  <xacro:robotiq_hande prefix="mara" />
+  <xacro:mara_robot prefix="" ee_link_distance="0.18253" MAC1="_000000000001" MAC2="_000000000002" MAC3="_000000000003"/>
+  <xacro:robotiq_hande prefix="" MAC="_000000000004"/>
   <xacro:table prefix="" />
   <link name="world" />

File: robotiq_85_gripper_description/urdf/robotiq_85.urdf.xacro (robot description, xacro)
@@ -1,6 +1,6 @@
 <?xml version="1.0"?>
 <robot xmlns:xacro="http://ros.org/wiki/xacro">
-  <xacro:macro name="robotiq_85"  params="prefix">
-    <link name="robotiq_arg2f_base_link">
+  <xacro:macro name="robotiq_85"  params="prefix MAC">
+    <link name="${prefix}robotiq_arg2f_base_link">
       <inertial>
         <origin xyz="-0.00013 -0.00011 0.03284" rpy="0 0 0" />
@@ -24,9 +24,9 @@
       </collision>
     </link>
-    <gazebo reference="robotiq_arg2f_base_link">
-      <material>Gazebo/Black</material>
-      <selfCollide>True</selfCollide>
-    </gazebo>
-    <link name="left_outer_knuckle">
+    <gazebo reference="${prefix}robotiq_arg2f_base_link">
+      <material>Gazebo/Black</material>
+      <selfCollide>True</selfCollide>
+    </gazebo>
+    <link name="${prefix}left_outer_knuckle">
       <inertial>
         <origin xyz="0.01545 0 -0.00118" rpy="0 0 0" />
@@ -50,9 +50,9 @@
       </collision>
     </link>
-    <gazebo reference="left_outer_knuckle">
+    <gazebo reference="${prefix}left_outer_knuckle">
       <material>Gazebo/Grey</material>
       <selfCollide>True</selfCollide>
     </gazebo>
-    <link name="right_outer_knuckle">
+    <link name="${prefix}right_outer_knuckle">
       <inertial>
         <origin xyz="-0.01545 0 -0.00118" rpy="0 0 0" />
@@ -76,9 +76,9 @@
       </collision>
     </link>
-    <gazebo reference="right_outer_knuckle">
+    <gazebo reference="${prefix}right_outer_knuckle">
       <material>Gazebo/Grey</material>
       <selfCollide>True</selfCollide>
     </gazebo>
-    <link name="left_outer_finger">
+    <link name="${prefix}left_outer_finger">
       <inertial>
         <origin xyz="0.004 0 0.01892" rpy="0 0 0" />
@@ -102,9 +102,9 @@
       </collision>
     </link>
-    <gazebo reference="left_outer_finger">
-      <material>Gazebo/Black</material>
-      <selfCollide>True</selfCollide>
-    </gazebo>
-    <link name="right_outer_finger">
+    <gazebo reference="${prefix}left_outer_finger">
+      <material>Gazebo/Black</material>
+      <selfCollide>True</selfCollide>
+    </gazebo>
+    <link name="${prefix}right_outer_finger">
       <inertial>
         <origin xyz="-0.004 0 0.01892" rpy="0 0 0" />
@@ -128,9 +128,9 @@
       </collision>
     </link>
-    <gazebo reference="right_outer_finger">
-      <material>Gazebo/Black</material>
-      <selfCollide>True</selfCollide>
-    </gazebo>
-    <link name="left_inner_knuckle">
+    <gazebo reference="${prefix}right_outer_finger">
+      <material>Gazebo/Black</material>
+      <selfCollide>True</selfCollide>
+    </gazebo>
+    <link name="${prefix}left_inner_knuckle">
       <inertial>
         <origin xyz="0.01952 0 0.022" rpy="0 0 0" />
@@ -154,9 +154,9 @@
       </collision>
     </link>
-    <gazebo reference="left_inner_knuckle">
+    <gazebo reference="${prefix}left_inner_knuckle">
       <material>Gazebo/Black</material>
       <selfCollide>False</selfCollide>
     </gazebo>
-    <link name="right_inner_knuckle">
+    <link name="${prefix}right_inner_knuckle">
       <inertial>
         <origin xyz="-0.01952 0 0.022" rpy="0 0 0" />
@@ -180,9 +180,9 @@
       </collision>
     </link>
-    <gazebo reference="right_inner_knuckle">
+    <gazebo reference="${prefix}right_inner_knuckle">
       <material>Gazebo/Black</material>
       <selfCollide>False</selfCollide>
     </gazebo>
-    <link name="left_inner_finger">
+    <link name="${prefix}left_inner_finger">
       <inertial>
         <origin xyz="-0.01409 0 0.01569" rpy="0 0 0" />
@@ -206,9 +206,9 @@
       </collision>
     </link>
-    <gazebo reference="left_inner_finger">
+    <gazebo reference="${prefix}left_inner_finger">
       <material>Gazebo/Black</material>
       <selfCollide>False</selfCollide>
     </gazebo>
-    <link name="right_inner_finger">
+    <link name="${prefix}right_inner_finger">
       <inertial>
         <origin xyz="0.01409 0 0.01569" rpy="0 0 0" />
@@ -232,70 +232,70 @@
       </collision>
     </link>
-    <gazebo reference="right_inner_finger">
+    <gazebo reference="${prefix}right_inner_finger">
       <material>Gazebo/Black</material>
       <selfCollide>False</selfCollide>
     </gazebo>
-    <joint name="robotiq_arg2f_base_link_to_left_outer_knuckle" type="revolute">
+    <joint name="${prefix}robotiq_arg2f_base_link_to_${prefix}left_outer_knuckle" type="revolute">
       <origin xyz="0.0306 0 0.05466" rpy="0 0 0" />
-      <parent link="robotiq_arg2f_base_link" />
-      <child link="left_outer_knuckle" />
+      <parent link="${prefix}robotiq_arg2f_base_link" />
+      <child link="${prefix}left_outer_knuckle" />
       <axis xyz="0 -1 0" />
       <limit lower="0" upper="0.82589" velocity="3.87" effort="21.03" />
       <mimic joint="joint_finger" multiplier="1" offset="0"/>
     </joint>
-    <joint name="joint_finger" type="revolute">
+    <joint name="${prefix}joint_finger" type="revolute">
       <origin xyz="-0.0306 0 0.05466" rpy="0 0 0" />
-      <parent link="robotiq_arg2f_base_link" />
-      <child link="right_outer_knuckle" />
+      <parent link="${prefix}robotiq_arg2f_base_link" />
+      <child link="${prefix}right_outer_knuckle" />
       <axis xyz="0 1 0" />
       <limit lower="0" upper="0.82589" velocity="3.87" effort="21.03" />
     </joint>
-    <joint name="robotiq_arg2f_base_link_to_left_inner_knuckle" type="revolute">
+    <joint name="${prefix}robotiq_arg2f_base_link_to_${prefix}left_inner_knuckle" type="revolute">
       <origin xyz="0.0127 0 0.06118" rpy="0 0 0" />
-      <parent link="robotiq_arg2f_base_link" />
-      <child link="left_inner_knuckle" />
+      <parent link="${prefix}robotiq_arg2f_base_link" />
+      <child link="${prefix}left_inner_knuckle" />
       <axis xyz="0 -1 0" />
       <limit lower="0" upper="0.82589" velocity="3.87" effort="21.03" />
       <mimic joint="joint_finger" multiplier="1" offset="0"/>
     </joint>
-    <joint name="robotiq_arg2f_base_link_to_right_inner_knuckle" type="revolute">
+    <joint name="${prefix}robotiq_arg2f_base_link_to_${prefix}right_inner_knuckle" type="revolute">
       <origin xyz="-0.0127 0 0.06118" rpy="0 0 0" />
-      <parent link="robotiq_arg2f_base_link" />
-      <child link="right_inner_knuckle" />
+      <parent link="${prefix}robotiq_arg2f_base_link" />
+      <child link="${prefix}right_inner_knuckle" />
       <axis xyz="0 1 0" />
       <limit lower="0" upper="0.82589" velocity="3.87" effort="21.03" />
       <mimic joint="joint_finger" multiplier="1" offset="0"/>
     </joint>
-    <joint name="left_outer_finger_to_inner" type="revolute">
+    <joint name="${prefix}left_outer_finger_to_inner" type="revolute">
       <origin xyz="0.00678 0 0.04703" rpy="0 0 0" />
-      <parent link="left_outer_finger" />
-      <child link="left_inner_finger" />
+      <parent link="${prefix}left_outer_finger" />
+      <child link="${prefix}left_inner_finger" />
       <axis xyz="0 1 0" />
       <limit lower="0" upper="0.82589" velocity="3.87" effort="21.03" />
       <mimic joint="joint_finger" multiplier="1" offset="0"/>
     </joint>
-    <joint name="right_outer_finger_to_inner" type="revolute">
+    <joint name="${prefix}right_outer_finger_to_inner" type="revolute">
       <origin xyz="-0.00678 0 0.04703" rpy="0 0 0" />
-      <parent link="right_outer_finger" />
-      <child link="right_inner_finger" />
+      <parent link="${prefix}right_outer_finger" />
+      <child link="${prefix}right_inner_finger" />
       <axis xyz="0 -1 0" />
       <limit lower="0" upper="0.82589" velocity="3.87" effort="21.03" />
       <mimic joint="joint_finger" multiplier="1" offset="0"/>
     </joint>
-    <joint name="left_outer_knuckle_to_finger" type="fixed">
+    <joint name="${prefix}left_outer_knuckle_to_finger" type="fixed">
       <origin xyz="0.03142 0 -0.00453" rpy="0 0 0" />
-      <parent link="left_outer_knuckle" />
-      <child link="left_outer_finger" />
-    </joint>
-    <joint name="right_outer_knuckle_to_finger" type="fixed">
+      <parent link="${prefix}left_outer_knuckle" />
+      <child link="${prefix}left_outer_finger" />
+    </joint>
+    <joint name="${prefix}right_outer_knuckle_to_finger" type="fixed">
       <origin xyz="-0.03142 0 -0.00453" rpy="0 0 0" />
-      <parent link="right_outer_knuckle" />
-      <child link="right_outer_finger" />
+      <parent link="${prefix}right_outer_knuckle" />
+      <child link="${prefix}right_outer_finger" />
     </joint>
     <gazebo>
-      <joint name="left_inner_knuckle_to_finger" type="revolute">
+      <joint name="${prefix}left_inner_knuckle_to_finger" type="revolute">
         <pose frame="">-0.0179 0 0.00652 0 0 0</pose>
-        <parent>${prefix}::left_inner_knuckle</parent>
-        <child>${prefix}::left_inner_finger</child>
+        <parent>${prefix}left_inner_knuckle</parent>
+        <child>${prefix}left_inner_finger</child>
         <axis>
           <xyz>0 1 0</xyz>
@@ -308,8 +308,8 @@
         </axis>
       </joint>
-      <joint name="right_inner_knuckle_to_finger" type="revolute">
+      <joint name="${prefix}right_inner_knuckle_to_finger" type="revolute">
         <pose frame="">0.0179 0 0.00652 0 0 0</pose>
-        <parent>${prefix}::right_inner_knuckle</parent>
-        <child>${prefix}::right_inner_finger</child>
+        <parent>${prefix}right_inner_knuckle</parent>
+        <child>${prefix}right_inner_finger</child>
         <axis>
           <xyz>0 -1 0</xyz>
@@ -322,12 +322,12 @@
         </axis>
       </joint>
-      <plugin filename="librobotiq_gripper_gazebo_plugin.so" name="robotiq_85_gripper">
+      <plugin filename="librobotiq_gripper_gazebo_plugin.so" name="hrim_actuator_gripper${MAC}">
         <kp>10</kp>
         <ki>10</ki>
         <kd>0.1</kd>
-        <joint>robotiq_arg2f_base_link_to_left_inner_knuckle</joint>
-        <joint>robotiq_arg2f_base_link_to_left_outer_knuckle</joint>
-        <joint>robotiq_arg2f_base_link_to_right_inner_knuckle</joint>
-        <joint>joint_finger</joint>
+        <joint>${prefix}robotiq_arg2f_base_link_to_${prefix}left_inner_knuckle</joint>
+        <joint>${prefix}robotiq_arg2f_base_link_to_${prefix}left_outer_knuckle</joint>
+        <joint>${prefix}robotiq_arg2f_base_link_to_${prefix}right_inner_knuckle</joint>
+        <joint>${prefix}joint_finger</joint>
       </plugin>
     </gazebo>

File: robotiq_85_gripper_description/urdf/robotiq_85_world.urdf.xacro (robot description, xacro)
@@ -2,5 +2,5 @@
 <robot xmlns:xacro="http://ros.org/wiki/xacro" name="robotiq_85" >
   <xacro:include filename="$(find robotiq_85_gripper_description)/urdf/robotiq_85.urdf.xacro" />
-  <xacro:robotiq_85 prefix="robotiq85"/>
+  <xacro:robotiq_85 prefix="robotiq85" MAC="_000000000004"/>
   <link name="world" />
   <joint name="world_to_robotiq_arg2f_base" type="fixed">

File: robotiq_hande_gripper_description/urdf/robotiq_hande.urdf.xacro (robot description, xacro)
@@ -1,6 +1,6 @@
 <?xml version="1.0"?>
 <robot xmlns:xacro="http://ros.org/wiki/xacro">
-  <xacro:macro name="robotiq_hande"  params="prefix">
-    <link name="robotiq_hande_base_link">
+  <xacro:macro name="robotiq_hande"  params="prefix MAC">
+    <link name="${prefix}robotiq_hande_base_link">
       <inertial>
         <origin xyz="0 0 0.04607" rpy="0 0 0" />
@@ -24,9 +24,9 @@
       </collision>
     </link>
-    <gazebo reference="robotiq_hande_base_link">
+    <gazebo reference="${prefix}robotiq_hande_base_link">
       <material>Gazebo/Black</material>
       <selfCollide>True</selfCollide>
     </gazebo>
-    <link name="left_finger">
+    <link name="${prefix}left_finger">
       <inertial>
         <origin rpy="0 0 0" xyz="0.02262 -0.00759 0.00738"/>
@@ -50,9 +50,9 @@
       </collision>
     </link>
-    <gazebo reference="left_finger">
+    <gazebo reference="${prefix}left_finger">
       <material>Gazebo/Grey</material>
       <selfCollide>True</selfCollide>
     </gazebo>
-    <link name="right_finger">
+    <link name="${prefix}right_finger">
       <inertial>
         <origin rpy="0 0 0" xyz="-0.02262 0.00759 0.00738"/>
@@ -76,37 +76,37 @@
       </collision>
     </link>
-    <gazebo reference="right_finger">
+    <gazebo reference="${prefix}right_finger">
       <material>Gazebo/Grey</material>
       <selfCollide>True</selfCollide>
     </gazebo>
-    <joint name="joint_finger" type="prismatic">
+    <joint name="${prefix}joint_finger" type="prismatic">
       <origin rpy="0 0 0" xyz="0 0 0.099"/>
-      <parent link="robotiq_hande_base_link"/>
-      <child link="left_finger"/>
+      <parent link="${prefix}robotiq_hande_base_link"/>
+      <child link="${prefix}left_finger"/>
       <axis xyz="-1 0 0"/>
       <limit effort="130" lower="0" upper="0.025" velocity="0.15"/>
     </joint>
-    <joint name="robotiq_hande_base_to_right_finger" type="prismatic">
+    <joint name="robotiq_hande_base_to_${prefix}right_finger" type="prismatic">
       <origin rpy="0 0 0" xyz="0 0 0.099"/>
-      <parent link="robotiq_hande_base_link"/>
-      <child link="right_finger"/>
+      <parent link="${prefix}robotiq_hande_base_link"/>
+      <child link="${prefix}right_finger"/>
       <axis xyz="1 0 0"/>
       <limit effort="130" lower="0" upper="0.025" velocity="0.15"/>
-      <mimic joint="joint_finger" multiplier="1" offset="0"/>
+      <mimic joint="${prefix}joint_finger" multiplier="1" offset="0"/>
     </joint>
     <gazebo>
-      <plugin filename="librobotiq_gripper_gazebo_plugin.so" name="robotiq_hande_gripper">
+      <plugin filename="librobotiq_gripper_gazebo_plugin.so" name="hrim_actuator_gripper${MAC}">
         <kp>100</kp>
         <ki>3</ki>
         <kd>9</kd>
-        <joint>joint_finger</joint>
-        <joint>robotiq_hande_base_to_right_finger</joint>
+        <joint>${prefix}joint_finger</joint>
+        <joint>robotiq_hande_base_to_${prefix}right_finger</joint>
       </plugin>
-      <plugin filename="libgazebo_ros_joint_state_publisher.so" name="mara_joint_state">
+      <plugin filename="libgazebo_ros_joint_state_publisher.so" name="${prefix}joint_state">
         <ros>
           <argument>~/out:=joint_states</argument>
         </ros>
         <update_rate>25</update_rate>
-        <joint_name>joint_finger</joint_name>
+        <joint_name>${prefix}joint_finger</joint_name>
       </plugin>
     </gazebo>

File: robotiq_hande_gripper_description/urdf/robotiq_hande_world.urdf.xacro (robot description, xacro)
@@ -2,5 +2,5 @@
 <robot xmlns:xacro="http://ros.org/wiki/xacro" name="robotiq_hande" >
   <xacro:include filename="$(find robotiq_hande_gripper_description)/urdf/hande_gripper.urdf.xacro" />
-  <xacro:robotiq_hande prefix=""/>
+  <xacro:robotiq_hande prefix="hande" MAC="_000000000004"/>
   <link name="world" />
   <joint name="world_to_robotiq_adapter" type="fixed">
