Commit message: fix - libgazebo_ros_joint_state_publisher plugin - launch files - passive_joints

File: mara_description/urdf/mara_gazebo.urdf.xacro (robot description, xacro)
@@ -3,7 +3,7 @@
   <xacro:macro name="mara_gazebo" params="prefix MAC1 MAC2 MAC3">
     <gazebo>
-      <plugin name="mara_joint_state" filename="libgazebo_ros_joint_state_publisher.so">
+      <plugin name="${prefix}joint_state" filename="libgazebo_ros_joint_state_publisher.so">
         <ros>
-          <argument>~/out:=joint_states</argument>
+          <argument>~/out:=${prefix}joint_states</argument>
         </ros>
         <update_rate>25</update_rate>

File: robotiq_140_gripper_description/urdf/robotiq_140.urdf.xacro (robot description, xacro)
@@ -331,4 +331,11 @@
         <joint>${prefix}joint_finger</joint>
       </plugin>
+      <plugin filename="libgazebo_ros_joint_state_publisher.so" name="${prefix}joint_state">
+        <ros>
+          <argument>~/out:=${prefix}joint_states</argument>
+        </ros>
+        <update_rate>25</update_rate>
+        <joint_name>${prefix}joint_finger</joint_name>
+      </plugin>
     </gazebo>
   </xacro:macro>

File: robotiq_85_gripper_description/urdf/robotiq_85.urdf.xacro (robot description, xacro)
@@ -331,4 +331,11 @@
         <joint>${prefix}joint_finger</joint>
       </plugin>
+      <plugin filename="libgazebo_ros_joint_state_publisher.so" name="${prefix}joint_state">
+        <ros>
+          <argument>~/out:=${prefix}joint_states</argument>
+        </ros>
+        <update_rate>25</update_rate>
+        <joint_name>${prefix}joint_finger</joint_name>
+      </plugin>
     </gazebo>
   </xacro:macro>

File: robotiq_85_gripper_description/urdf/robotiq_85_world.urdf.xacro (robot description, xacro)
@@ -2,10 +2,10 @@
 <robot xmlns:xacro="http://ros.org/wiki/xacro" name="robotiq_85" >
   <xacro:include filename="$(find robotiq_85_gripper_description)/urdf/robotiq_85.urdf.xacro" />
-  <xacro:robotiq_85 prefix="robotiq85" MAC="_000000000004"/>
+  <xacro:robotiq_85 prefix="robotiq_85_" MAC="_000000000004"/>
   <link name="world" />
   <joint name="world_to_robotiq_arg2f_base" type="fixed">
     <origin rpy="0 0 0" xyz="0 0 0.5"/>
     <parent link="world"/>
-    <child link="robotiq_arg2f_base_link"/>
+    <child link="robotiq_85_robotiq_arg2f_base_link"/>
   </joint>
 </robot>

File: robotiq_hande_gripper_description/urdf/robotiq_hande.urdf.xacro (robot description, xacro)
@@ -105,5 +105,5 @@
       <plugin filename="libgazebo_ros_joint_state_publisher.so" name="${prefix}joint_state">
         <ros>
-          <argument>~/out:=joint_states</argument>
+          <argument>~/out:=${prefix}joint_states</argument>
         </ros>
         <update_rate>25</update_rate>

File: robotiq_hande_gripper_description/urdf/robotiq_hande_world.urdf.xacro (robot description, xacro)
@@ -2,10 +2,10 @@
 <robot xmlns:xacro="http://ros.org/wiki/xacro" name="robotiq_hande" >
   <xacro:include filename="$(find robotiq_hande_gripper_description)/urdf/hande_gripper.urdf.xacro" />
-  <xacro:robotiq_hande prefix="hande" MAC="_000000000004"/>
+  <xacro:robotiq_hande prefix="hande_" MAC="_000000000004"/>
   <link name="world" />
   <joint name="world_to_robotiq_adapter" type="fixed">
     <origin rpy="0 0 0" xyz="0 0 0.5"/>
     <parent link="world"/>
-    <child link="robotiq_hande_base_link"/>
+    <child link="hande_robotiq_hande_base_link"/>
   </joint>
 </robot>
