Commit message: Updating URDF modular robotiq 85 gripper

File: robotiq_85_gripper_description/urdf/robotiq_85.urdf.xacro (robot description, xacro)
@@ -28,4 +28,108 @@
       <selfCollide>True</selfCollide>
     </gazebo>
+    <link name="left_outer_knuckle">
+      <inertial>
+        <origin xyz="8.625E-08 -4.6583E-06 0.03145" rpy="0 0 0" />
+        <mass value="0.22652" />
+        <inertia ixx="0.00020005" ixy="0" ixz="0" iyy="0.00017832" iyz="0" izz="0.00013478" />
+      </inertial>
+      <visual>
+        <origin xyz="0 0 0" rpy="0 0 0" />
+        <geometry>
+          <mesh filename="package://robotiq_85_gripper_description/meshes/2-F-85_1_l.dae" scale="0.001 0.001 0.001"/>
+        </geometry>
+        <material name="Gazebo/Grey">
+          <color rgba="0.1 0.1 0.1 1" />
+        </material>
+      </visual>
+      <collision>
+        <origin xyz="0 0 0" rpy="0 0 0" />
+        <geometry>
+          <mesh filename="package://robotiq_85_gripper_description/meshes/2-F-85_1_l.dae" scale="0.001 0.001 0.001"/>
+        </geometry>
+      </collision>
+    </link>
+    <gazebo reference="left_outer_knuckle">
+      <material>Gazebo/Grey</material>
+      <selfCollide>True</selfCollide>
+    </gazebo>
+    <link name="right_outer_knuckle">
+      <inertial>
+        <origin xyz="8.625E-08 -4.6583E-06 0.03145" rpy="0 0 0" />
+        <mass value="0.22652" />
+        <inertia ixx="0.00020005" ixy="0" ixz="0" iyy="0.00017832" iyz="0" izz="0.00013478" />
+      </inertial>
+      <visual>
+        <origin xyz="0 0 0" rpy="0 0 0" />
+        <geometry>
+          <mesh filename="package://robotiq_85_gripper_description/meshes/2-F-85_1_r.dae" scale="0.001 0.001 0.001"/>
+        </geometry>
+        <material name="Gazebo/Grey">
+          <color rgba="0.1 0.1 0.1 1" />
+        </material>
+      </visual>
+      <collision>
+        <origin xyz="0 0 0" rpy="0 0 0" />
+        <geometry>
+          <mesh filename="package://robotiq_85_gripper_description/meshes/2-F-85_1_r.dae" scale="0.001 0.001 0.001"/>
+        </geometry>
+      </collision>
+    </link>
+    <gazebo reference="right_outer_knuckle">
+      <material>Gazebo/Grey</material>
+      <selfCollide>True</selfCollide>
+    </gazebo>
+    <link name="left_outer_finger">
+      <inertial>
+        <origin xyz="8.625E-08 -4.6583E-06 0.03145" rpy="0 0 0" />
+        <mass value="0.22652" />
+        <inertia ixx="0.00020005" ixy="0" ixz="0" iyy="0.00017832" iyz="0" izz="0.00013478" />
+      </inertial>
+      <visual>
+        <origin xyz="0 0 0" rpy="0 0 0" />
+        <geometry>
+          <mesh filename="package://robotiq_85_gripper_description/meshes/2-F-85_3_l.dae" scale="0.001 0.001 0.001"/>
+        </geometry>
+        <material name="Gazebo/Black">
+          <color rgba="0.1 0.1 0.1 1" />
+        </material>
+      </visual>
+      <collision>
+        <origin xyz="0 0 0" rpy="0 0 0" />
+        <geometry>
+          <mesh filename="package://robotiq_85_gripper_description/meshes/2-F-85_3_l.dae" scale="0.001 0.001 0.001"/>
+        </geometry>
+      </collision>
+    </link>
+    <gazebo reference="left_outer_finger">
+      <material>Gazebo/Black</material>
+      <selfCollide>True</selfCollide>
+    </gazebo>
+    <link name="right_outer_finger">
+      <inertial>
+        <origin xyz="8.625E-08 -4.6583E-06 0.03145" rpy="0 0 0" />
+        <mass value="0.22652" />
+        <inertia ixx="0.00020005" ixy="0" ixz="0" iyy="0.00017832" iyz="0" izz="0.00013478" />
+      </inertial>
+      <visual>
+        <origin xyz="0 0 0" rpy="0 0 0" />
+        <geometry>
+          <mesh filename="package://robotiq_85_gripper_description/meshes/2-F-85_3_r.dae" scale="0.001 0.001 0.001"/>
+        </geometry>
+        <material name="Gazebo/Black">
+          <color rgba="0.1 0.1 0.1 1" />
+        </material>
+      </visual>
+      <collision>
+        <origin xyz="0 0 0" rpy="0 0 0" />
+        <geometry>
+          <mesh filename="package://robotiq_85_gripper_description/meshes/2-F-85_3_r.dae" scale="0.001 0.001 0.001"/>
+        </geometry>
+      </collision>
+    </link>
+    <gazebo reference="right_outer_finger">
+      <material>Gazebo/Black</material>
+      <selfCollide>True</selfCollide>
+    </gazebo>
     <link name="left_inner_knuckle">
       <inertial>
@@ -37,19 +141,19 @@
         <origin xyz="0 0 0" rpy="0 0 0" />
         <geometry>
-          <mesh filename="package://robotiq_85_gripper_description/meshes/2-F-85_1_l.dae" scale="0.001 0.001 0.001"/>
-        </geometry>
-        <material name="Gazebo/Grey">
-          <color rgba="0.1 0.1 0.1 1" />
-        </material>
-      </visual>
-      <collision>
-        <origin xyz="0 0 0" rpy="0 0 0" />
-        <geometry>
-          <mesh filename="package://robotiq_85_gripper_description/meshes/2-F-85_1_l.dae" scale="0.001 0.001 0.001"/>
+          <mesh filename="package://robotiq_85_gripper_description/meshes/2-F-85_2_l.dae" scale="0.001 0.001 0.001"/>
+        </geometry>
+        <material name="Gazebo/Black">
+          <color rgba="0.1 0.1 0.1 1" />
+        </material>
+      </visual>
+      <collision>
+        <origin xyz="0 0 0" rpy="0 0 0" />
+        <geometry>
+          <mesh filename="package://robotiq_85_gripper_description/meshes/2-F-85_2_l.dae" scale="0.001 0.001 0.001"/>
         </geometry>
       </collision>
     </link>
     <gazebo reference="left_inner_knuckle">
-      <material>Gazebo/Grey</material>
+      <material>Gazebo/Black</material>
       <selfCollide>True</selfCollide>
     </gazebo>
@@ -63,70 +167,18 @@
         <origin xyz="0 0 0" rpy="0 0 0" />
         <geometry>
-          <mesh filename="package://robotiq_85_gripper_description/meshes/2-F-85_1_r.dae" scale="0.001 0.001 0.001"/>
-        </geometry>
-        <material name="Gazebo/Grey">
-          <color rgba="0.1 0.1 0.1 1" />
-        </material>
-      </visual>
-      <collision>
-        <origin xyz="0 0 0" rpy="0 0 0" />
-        <geometry>
-          <mesh filename="package://robotiq_85_gripper_description/meshes/2-F-85_1_r.dae" scale="0.001 0.001 0.001"/>
+          <mesh filename="package://robotiq_85_gripper_description/meshes/2-F-85_2_r.dae" scale="0.001 0.001 0.001"/>
+        </geometry>
+        <material name="Gazebo/Black">
+          <color rgba="0.1 0.1 0.1 1" />
+        </material>
+      </visual>
+      <collision>
+        <origin xyz="0 0 0" rpy="0 0 0" />
+        <geometry>
+          <mesh filename="package://robotiq_85_gripper_description/meshes/2-F-85_2_r.dae" scale="0.001 0.001 0.001"/>
         </geometry>
       </collision>
     </link>
     <gazebo reference="right_inner_knuckle">
-      <material>Gazebo/Grey</material>
-      <selfCollide>True</selfCollide>
-    </gazebo>
-    <link name="left_outer_knuckle">
-      <inertial>
-        <origin xyz="8.625E-08 -4.6583E-06 0.03145" rpy="0 0 0" />
-        <mass value="0.22652" />
-        <inertia ixx="0.00020005" ixy="0" ixz="0" iyy="0.00017832" iyz="0" izz="0.00013478" />
-      </inertial>
-      <visual>
-        <origin xyz="0 0 0" rpy="0 0 0" />
-        <geometry>
-          <mesh filename="package://robotiq_85_gripper_description/meshes/2-F-85_3_l.dae" scale="0.001 0.001 0.001"/>
-        </geometry>
-        <material name="Gazebo/Black">
-          <color rgba="0.1 0.1 0.1 1" />
-        </material>
-      </visual>
-      <collision>
-        <origin xyz="0 0 0" rpy="0 0 0" />
-        <geometry>
-          <mesh filename="package://robotiq_85_gripper_description/meshes/2-F-85_3_l.dae" scale="0.001 0.001 0.001"/>
-        </geometry>
-      </collision>
-    </link>
-    <gazebo reference="left_outer_knuckle">
-      <material>Gazebo/Black</material>
-      <selfCollide>True</selfCollide>
-    </gazebo>
-    <link name="right_outer_knuckle">
-      <inertial>
-        <origin xyz="8.625E-08 -4.6583E-06 0.03145" rpy="0 0 0" />
-        <mass value="0.22652" />
-        <inertia ixx="0.00020005" ixy="0" ixz="0" iyy="0.00017832" iyz="0" izz="0.00013478" />
-      </inertial>
-      <visual>
-        <origin xyz="0 0 0" rpy="0 0 0" />
-        <geometry>
-          <mesh filename="package://robotiq_85_gripper_description/meshes/2-F-85_3_r.dae" scale="0.001 0.001 0.001"/>
-        </geometry>
-        <material name="Gazebo/Black">
-          <color rgba="0.1 0.1 0.1 1" />
-        </material>
-      </visual>
-      <collision>
-        <origin xyz="0 0 0" rpy="0 0 0" />
-        <geometry>
-          <mesh filename="package://robotiq_85_gripper_description/meshes/2-F-85_3_r.dae" scale="0.001 0.001 0.001"/>
-        </geometry>
-      </collision>
-    </link>
-    <gazebo reference="right_outer_knuckle">
       <material>Gazebo/Black</material>
       <selfCollide>True</selfCollide>
@@ -141,14 +193,14 @@
         <origin xyz="0 0 0" rpy="0 0 0" />
         <geometry>
-          <mesh filename="package://robotiq_85_gripper_description/meshes/2-F-85_2_l.dae" scale="0.001 0.001 0.001"/>
-        </geometry>
-        <material name="Gazebo/Black">
-          <color rgba="0.1 0.1 0.1 1" />
-        </material>
-      </visual>
-      <collision>
-        <origin xyz="0 0 0" rpy="0 0 0" />
-        <geometry>
-          <mesh filename="package://robotiq_85_gripper_description/meshes/2-F-85_2_l.dae" scale="0.001 0.001 0.001"/>
+          <mesh filename="package://robotiq_85_gripper_description/meshes/2-F-85_4_l.dae" scale="0.001 0.001 0.001"/>
+        </geometry>
+        <material name="Gazebo/Black">
+          <color rgba="0.1 0.1 0.1 1" />
+        </material>
+      </visual>
+      <collision>
+        <origin xyz="0 0 0" rpy="0 0 0" />
+        <geometry>
+          <mesh filename="package://robotiq_85_gripper_description/meshes/2-F-85_4_l.dae" scale="0.001 0.001 0.001"/>
         </geometry>
       </collision>
@@ -167,14 +219,14 @@
         <origin xyz="0 0 0" rpy="0 0 0" />
         <geometry>
-          <mesh filename="package://robotiq_85_gripper_description/meshes/2-F-85_2_r.dae" scale="0.001 0.001 0.001"/>
-        </geometry>
-        <material name="Gazebo/Black">
-          <color rgba="0.1 0.1 0.1 1" />
-        </material>
-      </visual>
-      <collision>
-        <origin xyz="0 0 0" rpy="0 0 0" />
-        <geometry>
-          <mesh filename="package://robotiq_85_gripper_description/meshes/2-F-85_2_r.dae" scale="0.001 0.001 0.001"/>
+          <mesh filename="package://robotiq_85_gripper_description/meshes/2-F-85_4_r.dae" scale="0.001 0.001 0.001"/>
+        </geometry>
+        <material name="Gazebo/Black">
+          <color rgba="0.1 0.1 0.1 1" />
+        </material>
+      </visual>
+      <collision>
+        <origin xyz="0 0 0" rpy="0 0 0" />
+        <geometry>
+          <mesh filename="package://robotiq_85_gripper_description/meshes/2-F-85_4_r.dae" scale="0.001 0.001 0.001"/>
         </geometry>
       </collision>
@@ -184,127 +236,70 @@
       <selfCollide>True</selfCollide>
     </gazebo>
-    <link name="left_finger">
-      <inertial>
-        <origin xyz="8.625E-08 -4.6583E-06 0.03145" rpy="0 0 0" />
-        <mass value="0.22652" />
-        <inertia ixx="0.00020005" ixy="0" ixz="0" iyy="0.00017832" iyz="0" izz="0.00013478" />
-      </inertial>
-      <visual>
-        <origin xyz="0 0 0" rpy="0 0 0" />
-        <geometry>
-          <mesh filename="package://robotiq_85_gripper_description/meshes/2-F-85_4_l.dae" scale="0.001 0.001 0.001"/>
-        </geometry>
-        <material name="Gazebo/Black">
-          <color rgba="0.1 0.1 0.1 1" />
-        </material>
-      </visual>
-      <collision>
-        <origin xyz="0 0 0" rpy="0 0 0" />
-        <geometry>
-          <mesh filename="package://robotiq_85_gripper_description/meshes/2-F-85_4_l.dae" scale="0.001 0.001 0.001"/>
-        </geometry>
-      </collision>
-    </link>
-    <gazebo reference="left_finger">
-      <material>Gazebo/Black</material>
-      <selfCollide>True</selfCollide>
-    </gazebo>
-    <link name="right_finger">
-      <inertial>
-        <origin xyz="8.625E-08 -4.6583E-06 0.03145" rpy="0 0 0" />
-        <mass value="0.22652" />
-        <inertia ixx="0.00020005" ixy="0" ixz="0" iyy="0.00017832" iyz="0" izz="0.00013478" />
-      </inertial>
-      <visual>
-        <origin xyz="0 0 0" rpy="0 0 0" />
-        <geometry>
-          <mesh filename="package://robotiq_85_gripper_description/meshes/2-F-85_4_r.dae" scale="0.001 0.001 0.001"/>
-        </geometry>
-        <material name="Gazebo/Black">
-          <color rgba="0.1 0.1 0.1 1" />
-        </material>
-      </visual>
-      <collision>
-        <origin xyz="0 0 0" rpy="0 0 0" />
-        <geometry>
-          <mesh filename="package://robotiq_85_gripper_description/meshes/2-F-85_4_r.dae" scale="0.001 0.001 0.001"/>
-        </geometry>
-      </collision>
-    </link>
-    <gazebo reference="right_finger">
-      <material>Gazebo/Black</material>
-      <selfCollide>True</selfCollide>
-    </gazebo>
+    <joint name="left_outer_knuckle_joint" type="revolute">
+      <origin xyz="-0.0306 0 0.05490" rpy="0 0 0" />
+      <parent link="robotiq_arg2f_base" />
+      <child link="left_outer_knuckle" />
+      <axis xyz="0 1 0" />
+      <limit lower="0.0" upper="0.78" velocity="2.0" effort="1000" />
+      <mimic joint="joint_finger" multiplier="1" offset="0"/>
+    </joint>
+    <joint name="joint_finger" type="revolute">
+      <origin xyz="0.0306 0 0.05490" rpy="0 0 3.1416" />
+      <parent link="robotiq_arg2f_base" />
+      <child link="right_outer_knuckle" />
+      <axis xyz="0 1 0" />
+      <limit lower="0" upper="0.78" velocity="2.0" effort="1000" />
+    </joint>
     <joint name="left_inner_knuckle_joint" type="revolute">
-      <origin xyz="-0.0306 0 0.05490" rpy="0 0 0" />
+      <origin xyz="-0.0127 0 0.06142" rpy="0 0 0" />
       <parent link="robotiq_arg2f_base" />
       <child link="left_inner_knuckle" />
       <axis xyz="0 1 0" />
-      <limit lower="0.0" upper="0.794" velocity="2.0" effort="1000" />
+      <limit lower="0" upper="0.8757" velocity="2.0" effort="1000" />
+      <mimic joint="joint_finger" multiplier="1" offset="0"/>
     </joint>
     <joint name="right_inner_knuckle_joint" type="revolute">
-      <origin xyz="0.0306 0 0.05490" rpy="0 0 3.1416" />
+      <origin xyz="0.0127 0 0.06142" rpy="0 0 3.1416" />
       <parent link="robotiq_arg2f_base" />
       <child link="right_inner_knuckle" />
       <axis xyz="0 1 0" />
-      <limit lower="0" upper="0.794" velocity="2.0" effort="1000" />
-    </joint>
-    <joint name="left_outer_knuckle_joint" type="revolute">
+      <limit lower="0" upper="0.8757" velocity="2.0" effort="1000" />
+      <mimic joint="joint_finger" multiplier="1" offset="0"/>
+    </joint>
+    <joint name="left_inner_finger_joint" type="revolute">
+      <origin xyz="-0.005625 0 0.04718" rpy="0 0.0 0" />
+      <parent link="left_outer_finger" />
+      <child link="left_inner_finger" />
+      <axis xyz="0 -1 0" />
+      <limit lower="0" upper="0.775" velocity="2.0" effort="1000" />
+      <mimic joint="joint_finger" multiplier="1" offset="0"/>
+    </joint>
+    <joint name="right_inner_finger_joint" type="revolute">
+      <origin xyz="-0.005625 0 0.04718" rpy="0 0 0" />
+      <parent link="right_outer_finger" />
+      <child link="right_inner_finger" />
+      <axis xyz="0 -1 0" />
+      <limit lower="0" upper="0.775" velocity="2.0" effort="1000" />
+      <mimic joint="joint_finger" multiplier="1" offset="0"/>
+    </joint>
+    <joint name="left_outer_finger_joint" type="fixed">
       <origin xyz="-0.03156 0 -0.003758" rpy="0 0 0" />
-      <parent link="left_inner_knuckle" />
-      <child link="left_outer_knuckle" />
-      <axis xyz="0 -1 0" />
-      <limit lower="0" upper="0.8757" velocity="2.0" effort="1000" />
-    </joint>
-    <joint name="right_outer_knuckle_joint" type="revolute">
+      <parent link="left_outer_knuckle" />
+      <child link="left_outer_finger" />
+    </joint>
+    <joint name="right_outer_finger_joint" type="fixed">
       <origin xyz="-0.03156 0 -0.003758" rpy="0 0 0" />
-      <parent link="right_inner_knuckle" />
-      <child link="right_outer_knuckle" />
-      <axis xyz="0 -1 0" />
-      <limit lower="0" upper="0.8757" velocity="2.0" effort="1000" />
-    </joint>
-    <joint name="left_inner_finger_joint" type="revolute">
-      <origin xyz="-0.0127 0 0.06142" rpy="0 0 0" />
-      <parent link="robotiq_arg2f_base" />
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