Commit message: Updating URDF modular robotiq 85 gripper

File: robotiq_85_gripper_description/urdf/robotiq_85_hros_support.urdf.xacro (robot description, xacro)
@@ -54,5 +54,5 @@
       <selfCollide>True</selfCollide>
     </gazebo>
-    <link name="robotiq_85_left_inner_knuckle_link">
+    <link name="left_outer_knuckle">
       <inertial>
         <origin xyz="8.625E-08 -4.6583E-06 0.03145" rpy="0 0 0" />
@@ -76,9 +76,9 @@
       </collision>
     </link>
-    <gazebo reference="robotiq_85_left_inner_knuckle_link">
+    <gazebo reference="left_outer_knuckle">
       <material>Gazebo/Grey</material>
       <selfCollide>True</selfCollide>
     </gazebo>
-    <link name="robotiq_85_right_inner_knuckle_link">
+    <link name="right_outer_knuckle">
       <inertial>
         <origin xyz="8.625E-08 -4.6583E-06 0.03145" rpy="0 0 0" />
@@ -102,9 +102,9 @@
       </collision>
     </link>
-    <gazebo reference="robotiq_85_right_inner_knuckle_link">
+    <gazebo reference="right_outer_knuckle">
       <material>Gazebo/Grey</material>
       <selfCollide>True</selfCollide>
     </gazebo>
-    <link name="robotiq_85_left_outer_knuckle_link">
+    <link name="left_outer_finger">
       <inertial>
         <origin xyz="8.625E-08 -4.6583E-06 0.03145" rpy="0 0 0" />
@@ -128,9 +128,9 @@
       </collision>
     </link>
-    <gazebo reference="robotiq_85_left_outer_knuckle_link">
-      <material>Gazebo/Black</material>
-      <selfCollide>True</selfCollide>
-    </gazebo>
-    <link name="robotiq_85_right_outer_knuckle_link">
+    <gazebo reference="left_outer_finger">
+      <material>Gazebo/Black</material>
+      <selfCollide>True</selfCollide>
+    </gazebo>
+    <link name="right_outer_finger">
       <inertial>
         <origin xyz="8.625E-08 -4.6583E-06 0.03145" rpy="0 0 0" />
@@ -154,9 +154,9 @@
       </collision>
     </link>
-    <gazebo reference="robotiq_85_right_outer_knuckle_link">
-      <material>Gazebo/Black</material>
-      <selfCollide>True</selfCollide>
-    </gazebo>
-    <link name="robotiq_85_left_inner_finger_link">
+    <gazebo reference="right_outer_finger">
+      <material>Gazebo/Black</material>
+      <selfCollide>True</selfCollide>
+    </gazebo>
+    <link name="left_inner_knuckle">
       <inertial>
         <origin xyz="8.625E-08 -4.6583E-06 0.03145" rpy="0 0 0" />
@@ -180,9 +180,9 @@
       </collision>
     </link>
-    <gazebo reference="robotiq_85_left_inner_finger_link">
-      <material>Gazebo/Black</material>
-      <selfCollide>True</selfCollide>
-    </gazebo>
-    <link name="robotiq_85_right_inner_finger_link">
+    <gazebo reference="left_inner_knuckle">
+      <material>Gazebo/Black</material>
+      <selfCollide>True</selfCollide>
+    </gazebo>
+    <link name="right_inner_knuckle">
       <inertial>
         <origin xyz="8.625E-08 -4.6583E-06 0.03145" rpy="0 0 0" />
@@ -206,9 +206,9 @@
       </collision>
     </link>
-    <gazebo reference="robotiq_85_right_inner_finger_link">
-      <material>Gazebo/Black</material>
-      <selfCollide>True</selfCollide>
-    </gazebo>
-    <link name="robotiq_85_left_finger_link">
+    <gazebo reference="right_inner_knuckle">
+      <material>Gazebo/Black</material>
+      <selfCollide>True</selfCollide>
+    </gazebo>
+    <link name="left_inner_finger">
       <inertial>
         <origin xyz="8.625E-08 -4.6583E-06 0.03145" rpy="0 0 0" />
@@ -232,9 +232,9 @@
       </collision>
     </link>
-    <gazebo reference="robotiq_85_left_finger_link">
-      <material>Gazebo/Black</material>
-      <selfCollide>True</selfCollide>
-    </gazebo>
-    <link name="robotiq_85_right_finger_link">
+    <gazebo reference="left_inner_finger">
+      <material>Gazebo/Black</material>
+      <selfCollide>True</selfCollide>
+    </gazebo>
+    <link name="right_inner_finger">
       <inertial>
         <origin xyz="8.625E-08 -4.6583E-06 0.03145" rpy="0 0 0" />
@@ -258,5 +258,5 @@
       </collision>
     </link>
-    <gazebo reference="robotiq_85_right_finger_link">
+    <gazebo reference="right_inner_finger">
       <material>Gazebo/Black</material>
       <selfCollide>True</selfCollide>
@@ -267,75 +267,70 @@
       <child link="robotiq_85_base_link"/>
     </joint>
+    <joint name="left_outer_knuckle_joint" type="revolute">
+      <origin xyz="-0.0306 0 0.05490" rpy="0 0 0" />
+      <parent link="robotiq_arg2f_base" />
+      <child link="left_outer_knuckle" />
+      <axis xyz="0 1 0" />
+      <limit lower="0.0" upper="0.78" velocity="2.0" effort="1000" />
+      <mimic joint="joint_finger" multiplier="1" offset="0"/>
+    </joint>
+    <joint name="joint_finger" type="revolute">
+      <origin xyz="0.0306 0 0.05490" rpy="0 0 3.1416" />
+      <parent link="robotiq_arg2f_base" />
+      <child link="right_outer_knuckle" />
+      <axis xyz="0 1 0" />
+      <limit lower="0" upper="0.78" velocity="2.0" effort="1000" />
+    </joint>
     <joint name="left_inner_knuckle_joint" type="revolute">
-      <origin xyz="-0.0306 0 0.05490" rpy="0 0 0" />
-      <parent link="robotiq_85_base_link" />
-      <child link="robotiq_85_left_inner_knuckle_link" />
-      <axis xyz="0 1 0" />
-      <limit lower="0.0" upper="0.794" velocity="2.0" effort="1000" />
-    </joint>
-    <joint name="right_inner_knuckle_joint" type="revolute">
-      <origin xyz="0.0306 0 0.05490" rpy="0 0 3.1416" />
-      <parent link="robotiq_85_base_link" />
-      <child link="robotiq_85_right_inner_knuckle_link" />
-      <axis xyz="0 1 0" />
-      <limit lower="0" upper="0.794" velocity="2.0" effort="1000" />
-    </joint>
-    <joint name="left_outer_knuckle_joint" type="revolute">
-      <origin xyz="-0.03156 0 -0.003758" rpy="0 0 0" />
-      <parent link="robotiq_85_left_inner_knuckle_link" />
-      <child link="robotiq_85_left_outer_knuckle_link" />
-      <axis xyz="0 -1 0" />
-      <limit lower="0" upper="0.8757" velocity="2.0" effort="1000" />
-    </joint>
-    <joint name="right_outer_knuckle_joint" type="revolute">
-      <origin xyz="-0.03156 0 -0.003758" rpy="0 0 0" />
-      <parent link="robotiq_85_right_inner_knuckle_link" />
-      <child link="robotiq_85_right_outer_knuckle_link" />
-      <axis xyz="0 -1 0" />
-      <limit lower="0" upper="0.8757" velocity="2.0" effort="1000" />
-    </joint>
-    <joint name="left_inner_finger_joint" type="revolute">
       <origin xyz="-0.0127 0 0.06142" rpy="0 0 0" />
-      <parent link="robotiq_85_base_link" />
-      <child link="robotiq_85_left_inner_finger_link" />
+      <parent link="robotiq_arg2f_base" />
+      <child link="left_inner_knuckle" />
       <axis xyz="0 1 0" />
       <limit lower="0" upper="0.8757" velocity="2.0" effort="1000" />
-    </joint>
-    <joint name="right_inner_finger_joint" type="revolute">
+      <mimic joint="joint_finger" multiplier="1" offset="0"/>
+    </joint>
+    <joint name="right_inner_knuckle_joint" type="revolute">
       <origin xyz="0.0127 0 0.06142" rpy="0 0 3.1416" />
-      <parent link="robotiq_85_base_link" />
-      <child link="robotiq_85_right_inner_finger_link" />
+      <parent link="robotiq_arg2f_base" />
+      <child link="right_inner_knuckle" />
       <axis xyz="0 1 0" />
       <limit lower="0" upper="0.8757" velocity="2.0" effort="1000" />
-    </joint>
-    <joint name="left_finger_joint" type="revolute">
+      <mimic joint="joint_finger" multiplier="1" offset="0"/>
+    </joint>
+    <joint name="left_inner_finger_joint" type="revolute">
       <origin xyz="-0.005625 0 0.04718" rpy="0 0.0 0" />
-      <parent link="robotiq_85_left_outer_knuckle_link" />
-      <child link="robotiq_85_left_finger_link" />
+      <parent link="left_outer_finger" />
+      <child link="left_inner_finger" />
       <axis xyz="0 -1 0" />
-      <limit lower="-0.1" upper="0.8757" velocity="2.0" effort="1000" />
-    </joint>
-    <joint name="right_finger_joint" type="revolute">
+      <limit lower="0" upper="0.775" velocity="2.0" effort="1000" />
+      <mimic joint="joint_finger" multiplier="1" offset="0"/>
+    </joint>
+    <joint name="right_inner_finger_joint" type="revolute">
       <origin xyz="-0.005625 0 0.04718" rpy="0 0 0" />
-      <parent link="robotiq_85_right_outer_knuckle_link" />
-      <child link="robotiq_85_right_finger_link" />
-      <axis xyz="0 -1 0"/>
-      <limit lower="-0.1" upper="0.8757" velocity="2.0" effort="1000" />
+      <parent link="right_outer_finger" />
+      <child link="right_inner_finger" />
+      <axis xyz="0 -1 0" />
+      <limit lower="0" upper="0.775" velocity="2.0" effort="1000" />
+      <mimic joint="joint_finger" multiplier="1" offset="0"/>
+    </joint>
+    <joint name="left_outer_finger_joint" type="fixed">
+      <origin xyz="-0.03156 0 -0.003758" rpy="0 0 0" />
+      <parent link="left_outer_knuckle" />
+      <child link="left_outer_finger" />
+    </joint>
+    <joint name="right_outer_finger_joint" type="fixed">
+      <origin xyz="-0.03156 0 -0.003758" rpy="0 0 0" />
+      <parent link="right_outer_knuckle" />
+      <child link="right_outer_finger" />
     </joint>
     <gazebo>
-      <plugin filename="librobotiq_gripper_gazebo_plugin.so" name="hros_actuation_gripper_000000000004">
-        <left_joint>left_inner_knuckle_joint</left_joint>
-        <left_joint>left_inner_finger_joint</left_joint>
-        <right_joint>right_inner_knuckle_joint</right_joint>
-        <right_joint>right_inner_finger_joint</right_joint>
-      </plugin>
       <joint name="left_finger_joint2" type="revolute">
         <pose frame="">0.017901 0 0.00651469 0 0 0</pose>
-        <parent>${prefix}::robotiq_85_left_inner_finger_link</parent>
-        <child>${prefix}::robotiq_85_left_finger_link</child>
+        <parent>${prefix}::left_inner_knuckle</parent>
+        <child>${prefix}::left_inner_finger</child>
         <axis>
           <xyz>0 -1 0</xyz>
           <limit>
-            <lower>-0.1</lower>
+            <lower>-0.8</lower>
             <upper>0.8</upper>
             <velocity>2.0</velocity>
@@ -346,10 +341,10 @@
       <joint name="right_finger_joint2" type="revolute">
         <pose frame="">0.017901 0 0.00651469 0 0 0</pose>
-        <parent>${prefix}::robotiq_85_right_inner_finger_link</parent>
-        <child>${prefix}::robotiq_85_right_finger_link</child>
+        <parent>${prefix}::right_inner_knuckle</parent>
+        <child>${prefix}::right_inner_finger</child>
         <axis>
           <xyz>0 1 0</xyz>
           <limit>
-            <lower>-0.1</lower>
+            <lower>-0.8</lower>
             <upper>0.8</upper>
             <velocity>2.0</velocity>

Commit message: replace robotiq_arg2f_base with robotiq_arg2f_base_link
In order not to complain about the collisions when planning the trajectory

File: robotiq_85_gripper_description/urdf/robotiq_85.urdf.xacro (robot description, xacro)
@@ -31,7 +31,7 @@
       <origin rpy="0 0 0" xyz=" 0 0 0.03653"/>
       <parent link="robotiq_adapter_link" />
-      <child link="robotiq_arg2f_base"/>
-    </joint>
-    <link name="robotiq_arg2f_base">
+      <child link="robotiq_arg2f_base_link"/>
+    </joint>
+    <link name="robotiq_arg2f_base_link">
       <inertial>
         <origin xyz="8.625E-08 -4.6583E-06 0.03145" rpy="0 0 0" />
@@ -55,5 +55,5 @@
       </collision>
     </link>
-    <gazebo reference="robotiq_arg2f_base">
+    <gazebo reference="robotiq_arg2f_base_link">
       <material>Gazebo/Black</material>
       <selfCollide>True</selfCollide>
@@ -269,5 +269,5 @@
     <joint name="left_outer_knuckle_joint" type="revolute">
       <origin xyz="-0.0306 0 0.05490" rpy="0 0 0" />
-      <parent link="robotiq_arg2f_base" />
+      <parent link="robotiq_arg2f_base_link" />
       <child link="left_outer_knuckle" />
       <axis xyz="0 1 0" />
@@ -277,5 +277,5 @@
     <joint name="joint_finger" type="revolute">
       <origin xyz="0.0306 0 0.05490" rpy="0 0 3.1416" />
-      <parent link="robotiq_arg2f_base" />
+      <parent link="robotiq_arg2f_base_link" />
       <child link="right_outer_knuckle" />
       <axis xyz="0 1 0" />
@@ -284,5 +284,5 @@
     <joint name="left_inner_knuckle_joint" type="revolute">
       <origin xyz="-0.0127 0 0.06142" rpy="0 0 0" />
-      <parent link="robotiq_arg2f_base" />
+      <parent link="robotiq_arg2f_base_link" />
       <child link="left_inner_knuckle" />
       <axis xyz="0 1 0" />
@@ -292,5 +292,5 @@
     <joint name="right_inner_knuckle_joint" type="revolute">
       <origin xyz="0.0127 0 0.06142" rpy="0 0 3.1416" />
-      <parent link="robotiq_arg2f_base" />
+      <parent link="robotiq_arg2f_base_link" />
       <child link="right_inner_knuckle" />
       <axis xyz="0 1 0" />
