Commit message: update S85 meshes and update values accordingly

File: robotiq_85_gripper_description/urdf/robotiq_85.urdf.xacro (robot description, xacro)
@@ -2,40 +2,9 @@
 <robot xmlns:xacro="http://ros.org/wiki/xacro">
   <xacro:macro name="robotiq_85"  params="prefix">
-    <link name="robotiq_adapter_link">
-      <inertial>
-        <origin xyz="8.625E-08 -4.6583E-06 0.03145" rpy="0 0 0" />
-        <mass value="0.22652" />
-        <inertia ixx="0.00020005" ixy="0" ixz="0" iyy="0.00017832" iyz="0" izz="0.00013478" />
-      </inertial>
-      <visual>
-        <origin xyz="0 0 0" rpy="0 0 1.57" />
-        <geometry>
-          <mesh filename="package://robotiq_85_gripper_description/meshes/hros_robotiq_adapter.dae" scale="0.001 0.001 0.001"/>
-        </geometry>
-        <material name="Gazebo/Black">
-          <color rgba="0.0 0.0 0.0 1" />
-        </material>
-      </visual>
-      <collision>
-        <origin xyz="0 0 0" rpy="0 0 1.57" />
-        <geometry>
-          <mesh filename="package://robotiq_85_gripper_description/meshes/hros_robotiq_adapter.dae" scale="0.001 0.001 0.001"/>
-        </geometry>
-      </collision>
-    </link>
-    <gazebo reference="robotiq_adapter_link">
-      <material>Gazebo/Black</material>
-      <selfCollide>False</selfCollide>
-    </gazebo>
-    <joint name="base_adapter_to_base_robotiq_joint" type="fixed">
-      <origin rpy="0 0 0" xyz=" 0 0 0.03653"/>
-      <parent link="robotiq_adapter_link" />
-      <child link="robotiq_arg2f_base_link"/>
-    </joint>
     <link name="robotiq_arg2f_base_link">
       <inertial>
-        <origin xyz="8.625E-08 -4.6583E-06 0.03145" rpy="0 0 0" />
-        <mass value="0.22652" />
-        <inertia ixx="0.00020005" ixy="0" ixz="0" iyy="0.00017832" iyz="0" izz="0.00013478" />
+        <origin xyz="-0.00013 -0.00011 0.03284" rpy="0 0 0" />
+        <mass value="0.55938" />
+        <inertia ixx="605783E-9" ixy="-579.95E-9" ixz="2765.53E-9" iyy="720148E-9" iyz="618E-9" izz="510534E-9" />
       </inertial>
       <visual>
@@ -57,11 +26,11 @@
     <gazebo reference="robotiq_arg2f_base_link">
       <material>Gazebo/Black</material>
-      <selfCollide>True</selfCollide>
+      <selfCollide>False</selfCollide>
     </gazebo>
     <link name="left_outer_knuckle">
       <inertial>
-        <origin xyz="8.625E-08 -4.6583E-06 0.03145" rpy="0 0 0" />
-        <mass value="0.22652" />
-        <inertia ixx="0.00020005" ixy="0" ixz="0" iyy="0.00017832" iyz="0" izz="0.00013478" />
+        <origin xyz="0.01545 0 -0.00118" rpy="0 0 0" />
+        <mass value="0.01252" />
+        <inertia ixx="312.44E-9" ixy="0" ixz="-168.09E-9" iyy="2156E-9" iyz="0" izz="2027.51E-9" />
       </inertial>
       <visual>
@@ -83,11 +52,11 @@
     <gazebo reference="left_outer_knuckle">
       <material>Gazebo/Grey</material>
-      <selfCollide>True</selfCollide>
+      <selfCollide>False</selfCollide>
     </gazebo>
     <link name="right_outer_knuckle">
       <inertial>
-        <origin xyz="8.625E-08 -4.6583E-06 0.03145" rpy="0 0 0" />
-        <mass value="0.22652" />
-        <inertia ixx="0.00020005" ixy="0" ixz="0" iyy="0.00017832" iyz="0" izz="0.00013478" />
+        <origin xyz="-0.01545 0 -0.00118" rpy="0 0 0" />
+        <mass value="0.01252" />
+        <inertia ixx="312.44E-9" ixy="0" ixz="-168.09E-9" iyy="2156E-9" iyz="0" izz="2027.51E-9" />
       </inertial>
       <visual>
@@ -109,11 +78,11 @@
     <gazebo reference="right_outer_knuckle">
       <material>Gazebo/Grey</material>
-      <selfCollide>True</selfCollide>
+      <selfCollide>False</selfCollide>
     </gazebo>
     <link name="left_outer_finger">
       <inertial>
-        <origin xyz="8.625E-08 -4.6583E-06 0.03145" rpy="0 0 0" />
-        <mass value="0.22652" />
-        <inertia ixx="0.00020005" ixy="0" ixz="0" iyy="0.00017832" iyz="0" izz="0.00013478" />
+        <origin xyz="0.004 0 0.01892" rpy="0 0 0" />
+        <mass value="0.03848" />
+        <inertia ixx="12341E-9" ixy="0" ixz="-2152.21E-9" iyy="10617E-9" iyz="0" izz="4812.09E-9" />
       </inertial>
       <visual>
@@ -135,11 +104,11 @@
     <gazebo reference="left_outer_finger">
       <material>Gazebo/Black</material>
-      <selfCollide>True</selfCollide>
+      <selfCollide>False</selfCollide>
     </gazebo>
     <link name="right_outer_finger">
       <inertial>
-        <origin xyz="8.625E-08 -4.6583E-06 0.03145" rpy="0 0 0" />
-        <mass value="0.22652" />
-        <inertia ixx="0.00020005" ixy="0" ixz="0" iyy="0.00017832" iyz="0" izz="0.00013478" />
+        <origin xyz="-0.004 0 0.01892" rpy="0 0 0" />
+        <mass value="0.03848" />
+        <inertia ixx="12341E-9" ixy="0" ixz="-2152.21E-9" iyy="10617E-9" iyz="0" izz="4812.09E-9" />
       </inertial>
       <visual>
@@ -161,11 +130,11 @@
     <gazebo reference="right_outer_finger">
       <material>Gazebo/Black</material>
-      <selfCollide>True</selfCollide>
+      <selfCollide>False</selfCollide>
     </gazebo>
     <link name="left_inner_knuckle">
       <inertial>
-        <origin xyz="8.625E-08 -4.6583E-06 0.03145" rpy="0 0 0" />
-        <mass value="0.22652" />
-        <inertia ixx="0.00020005" ixy="0" ixz="0" iyy="0.00017832" iyz="0" izz="0.00013478" />
+        <origin xyz="0.01952 0 0.022" rpy="0 0 0" />
+        <mass value="0.02731" />
+        <inertia ixx="8621.3E-9" ixy="0" ixz="-3646.49E-9" iyy="8004.28E-9" iyz="0" izz="7704.42E-9" />
       </inertial>
       <visual>
@@ -187,11 +156,11 @@
     <gazebo reference="left_inner_knuckle">
       <material>Gazebo/Black</material>
-      <selfCollide>True</selfCollide>
+      <selfCollide>False</selfCollide>
     </gazebo>
     <link name="right_inner_knuckle">
       <inertial>
-        <origin xyz="8.625E-08 -4.6583E-06 0.03145" rpy="0 0 0" />
-        <mass value="0.22652" />
-        <inertia ixx="0.00020005" ixy="0" ixz="0" iyy="0.00017832" iyz="0" izz="0.00013478" />
+        <origin xyz="-0.01952 0 0.022" rpy="0 0 0" />
+        <mass value="0.02731" />
+        <inertia ixx="8621.3E-9" ixy="0" ixz="-3646.49E-9" iyy="8004.28E-9" iyz="0" izz="7704.42E-9" />
       </inertial>
       <visual>
@@ -213,11 +182,11 @@
     <gazebo reference="right_inner_knuckle">
       <material>Gazebo/Black</material>
-      <selfCollide>True</selfCollide>
+      <selfCollide>False</selfCollide>
     </gazebo>
     <link name="left_inner_finger">
       <inertial>
-        <origin xyz="8.625E-08 -4.6583E-06 0.03145" rpy="0 0 0" />
-        <mass value="0.22652" />
-        <inertia ixx="0.00020005" ixy="0" ixz="0" iyy="0.00017832" iyz="0" izz="0.00013478" />
+        <origin xyz="-0.01409 0 0.01569" rpy="0 0 0" />
+        <mass value="0.037" />
+        <inertia ixx="12446.57E-9" ixy="0" ixz="4167.81E-9" iyy="14201.18E-9" iyz="0" izz="4979.86E-9" />
       </inertial>
       <visual>
@@ -239,11 +208,11 @@
     <gazebo reference="left_inner_finger">
       <material>Gazebo/Black</material>
-      <selfCollide>True</selfCollide>
+      <selfCollide>False</selfCollide>
     </gazebo>
     <link name="right_inner_finger">
       <inertial>
-        <origin xyz="8.625E-08 -4.6583E-06 0.03145" rpy="0 0 0" />
-        <mass value="0.22652" />
-        <inertia ixx="0.00020005" ixy="0" ixz="0" iyy="0.00017832" iyz="0" izz="0.00013478" />
+        <origin xyz="0.01409 0 0.01569" rpy="0 0 0" />
+        <mass value="0.037" />
+        <inertia ixx="12446.57E-9" ixy="0" ixz="4167.81E-9" iyy="14201.18E-9" iyz="0" izz="4979.86E-9" />
       </inertial>
       <visual>
@@ -265,96 +234,99 @@
     <gazebo reference="right_inner_finger">
       <material>Gazebo/Black</material>
-      <selfCollide>True</selfCollide>
-    </gazebo>
-    <joint name="left_outer_knuckle_joint" type="revolute">
-      <origin xyz="-0.0306 0 0.05490" rpy="0 0 0" />
+      <selfCollide>False</selfCollide>
+    </gazebo>
+    <joint name="robotiq_arg2f_base_link_to_left_outer_knuckle" type="revolute">
+      <origin xyz="0.0306 0 0.05466" rpy="0 0 0" />
       <parent link="robotiq_arg2f_base_link" />
       <child link="left_outer_knuckle" />
-      <axis xyz="0 1 0" />
-      <limit lower="0.0" upper="0.78" velocity="2.0" effort="1000" />
+      <axis xyz="0 -1 0" />
+      <limit lower="0" upper="0.82589" velocity="3.87" effort="21.03" />
       <mimic joint="joint_finger" multiplier="1" offset="0"/>
     </joint>
     <joint name="joint_finger" type="revolute">
-      <origin xyz="0.0306 0 0.05490" rpy="0 0 3.1416" />
+      <origin xyz="-0.0306 0 0.05466" rpy="0 0 0" />
       <parent link="robotiq_arg2f_base_link" />
       <child link="right_outer_knuckle" />
       <axis xyz="0 1 0" />
-      <limit lower="0" upper="0.78" velocity="2.0" effort="1000" />
-    </joint>
-    <joint name="left_inner_knuckle_joint" type="revolute">
-      <origin xyz="-0.0127 0 0.06142" rpy="0 0 0" />
+      <limit lower="0" upper="0.82589" velocity="3.87" effort="21.03" />
+    </joint>
+    <joint name="robotiq_arg2f_base_link_to_left_inner_knuckle" type="revolute">
+      <origin xyz="0.0127 0 0.06118" rpy="0 0 0" />
       <parent link="robotiq_arg2f_base_link" />
       <child link="left_inner_knuckle" />
-      <axis xyz="0 1 0" />
-      <limit lower="0" upper="0.8757" velocity="2.0" effort="1000" />
-      <mimic joint="joint_finger" multiplier="1" offset="0"/>
-    </joint>
-    <joint name="right_inner_knuckle_joint" type="revolute">
-      <origin xyz="0.0127 0 0.06142" rpy="0 0 3.1416" />
+      <axis xyz="0 -1 0" />
+      <limit lower="0" upper="0.82589" velocity="3.87" effort="21.03" />
+      <mimic joint="joint_finger" multiplier="1" offset="0"/>
+    </joint>
+    <joint name="robotiq_arg2f_base_link_to_right_inner_knuckle" type="revolute">
+      <origin xyz="-0.0127 0 0.06118" rpy="0 0 0" />
       <parent link="robotiq_arg2f_base_link" />
       <child link="right_inner_knuckle" />
       <axis xyz="0 1 0" />
-      <limit lower="0" upper="0.8757" velocity="2.0" effort="1000" />
-      <mimic joint="joint_finger" multiplier="1" offset="0"/>
-    </joint>
-    <joint name="left_inner_finger_joint" type="revolute">
-      <origin xyz="-0.005625 0 0.04718" rpy="0 0.0 0" />
+      <limit lower="0" upper="0.82589" velocity="3.87" effort="21.03" />
+      <mimic joint="joint_finger" multiplier="1" offset="0"/>
+    </joint>
+    <joint name="left_outer_finger_to_inner" type="revolute">
+      <origin xyz="0.00678 0 0.04703" rpy="0 0 0" />
       <parent link="left_outer_finger" />
       <child link="left_inner_finger" />
-      <axis xyz="0 -1 0" />
-      <limit lower="0" upper="0.775" velocity="2.0" effort="1000" />
-      <mimic joint="joint_finger" multiplier="1" offset="0"/>
-    </joint>
-    <joint name="right_inner_finger_joint" type="revolute">
-      <origin xyz="-0.005625 0 0.04718" rpy="0 0 0" />
+      <axis xyz="0 1 0" />
+      <limit lower="0" upper="0.82589" velocity="3.87" effort="21.03" />
+      <mimic joint="joint_finger" multiplier="1" offset="0"/>
+    </joint>
+    <joint name="right_outer_finger_to_inner" type="revolute">
+      <origin xyz="-0.00678 0 0.04703" rpy="0 0 0" />
       <parent link="right_outer_finger" />
       <child link="right_inner_finger" />
       <axis xyz="0 -1 0" />
-      <limit lower="0" upper="0.775" velocity="2.0" effort="1000" />
-      <mimic joint="joint_finger" multiplier="1" offset="0"/>
-    </joint>
-    <joint name="left_outer_finger_joint" type="fixed">
-      <origin xyz="-0.03156 0 -0.003758" rpy="0 0 0" />
+      <limit lower="0" upper="0.82589" velocity="3.87" effort="21.03" />
+      <mimic joint="joint_finger" multiplier="1" offset="0"/>
+    </joint>
+    <joint name="left_outer_knuckle_to_finger" type="fixed">
+      <origin xyz="0.03142 0 -0.00453" rpy="0 0 0" />
       <parent link="left_outer_knuckle" />
       <child link="left_outer_finger" />
     </joint>
-    <joint name="right_outer_finger_joint" type="fixed">
-      <origin xyz="-0.03156 0 -0.003758" rpy="0 0 0" />
+    <joint name="right_outer_knuckle_to_finger" type="fixed">
+      <origin xyz="-0.03142 0 -0.00453" rpy="0 0 0" />
       <parent link="right_outer_knuckle" />
       <child link="right_outer_finger" />
     </joint>
     <gazebo>
-      <joint name="left_finger_joint2" type="revolute">
-        <pose frame="">0.017901 0 0.00651469 0 0 0</pose>
+      <joint name="left_inner_knuckle_to_finger" type="revolute">
+        <pose frame="">-0.0179 0 0.00652 0 0 0</pose>
         <parent>${prefix}::left_inner_knuckle</parent>
         <child>${prefix}::left_inner_finger</child>
         <axis>
-          <xyz>0 -1 0</xyz>
+          <xyz>0 1 0</xyz>
           <limit>
-            <lower>-0.8</lower>
-            <upper>0.8</upper>
-            <velocity>2.0</velocity>
-            <effort>1000</effort>
+            <lower>0</lower>
+            <upper>0.82589</upper>
+            <velocity>3.87</velocity>
+            <effort>21.03</effort>
           </limit>
         </axis>
       </joint>
-      <joint name="right_finger_joint2" type="revolute">
-        <pose frame="">0.017901 0 0.00651469 0 0 0</pose>
+      <joint name="right_inner_knuckle_to_finger" type="revolute">
+        <pose frame="">0.0179 0 0.00652 0 0 0</pose>
         <parent>${prefix}::right_inner_knuckle</parent>
         <child>${prefix}::right_inner_finger</child>
         <axis>
-          <xyz>0 1 0</xyz>
+          <xyz>0 -1 0</xyz>
           <limit>
-            <lower>-0.8</lower>
-            <upper>0.8</upper>
-            <velocity>2.0</velocity>
-            <effort>1000</effort>
+            <lower>0</lower>
+            <upper>0.82589</upper>
+            <velocity>3.87</velocity>
+            <effort>21.03</effort>
           </limit>
         </axis>
       </joint>
       <plugin filename="librobotiq_gripper_gazebo_plugin.so" name="robotiq_85_gripper">
-        <joint>left_inner_knuckle_joint</joint>
-        <joint>left_outer_knuckle_joint</joint>
-        <joint>right_inner_knuckle_joint</joint>
+        <kp>10</kp>
+        <ki>10</ki>
+        <kd>0.1</kd>
+        <joint>robotiq_arg2f_base_link_to_left_inner_knuckle</joint>
+        <joint>robotiq_arg2f_base_link_to_left_outer_knuckle</joint>
+        <joint>robotiq_arg2f_base_link_to_right_inner_knuckle</joint>
         <joint>joint_finger</joint>
       </plugin>
