Commit message: rename and fix rename module_gripper urdf files to the corresponding robotiq_world

File: robotiq_85_gripper_description/urdf/robotiq_85_world.urdf.xacro (robot description, xacro)
@@ -1,13 +1,11 @@
 <?xml version="1.0"?>
-<robot xmlns:xacro="http://ros.org/wiki/xacro"
-       name="robotiq_85" >
-  <!-- robotiq hande_gripper -->
+<robot xmlns:xacro="http://ros.org/wiki/xacro" name="robotiq_85" >
   <xacro:include filename="$(find robotiq_85_gripper_description)/urdf/robotiq_85.urdf.xacro" />
   <xacro:robotiq_85 prefix="robotiq85"/>
   <link name="world" />
-  <joint name="world_to_hande_joint" type="fixed">
+  <joint name="world_to_robotiq_arg2f_base" type="fixed">
     <origin rpy="0 0 0" xyz="0 0 0.5"/>
     <parent link="world"/>
-    <child link="robotiq_adapter_link"/>
+    <child link="robotiq_arg2f_base_link"/>
   </joint>
 </robot>

File: robotiq_hande_gripper_description/urdf/robotiq_hande_world.urdf.xacro (robot description, xacro)
@@ -1,11 +1,9 @@
 <?xml version="1.0"?>
-<robot xmlns:xacro="http://ros.org/wiki/xacro"
-       name="robotiq_hande" >
-  <!-- robotiq hande_gripper -->
+<robot xmlns:xacro="http://ros.org/wiki/xacro" name="robotiq_hande" >
   <xacro:include filename="$(find robotiq_hande_gripper_description)/urdf/hande_gripper.urdf.xacro" />
   <xacro:robotiq_hande prefix=""/>
   <link name="world" />
-  <joint name="world_to_hande_joint" type="fixed">
-    <origin rpy="0 1.57 0" xyz="0 0 0.5"/>
+  <joint name="world_to_robotiq_adapter" type="fixed">
+    <origin rpy="0 0 0" xyz="0 0 0.5"/>
     <parent link="world"/>
     <child link="robotiq_hande_base_link"/>
