Commit message: updating hande URDF

File: robotiq_hande_gripper_description/urdf/robotiq_hande.urdf.xacro (robot description, xacro)
@@ -82,17 +82,22 @@
     <gazebo>
       <plugin filename="librobotiq_linear_gripper_gazebo_plugin.so" name="robotiq_hande_gripper">
-        <left_joint>finger1_joint</left_joint>
+        <left_joint>joint_finger</left_joint>
         <right_joint>finger2_joint</right_joint>
       </plugin>
     </gazebo>
-    <joint name="finger1_joint" type="fixed">
+    <joint name="joint_finger" type="prismatic">
       <origin rpy="0 0 0" xyz="0 0 0.0"/>
       <parent link="robotiq_hande_base_link"/>
       <child link="finger1"/>
+      <axis xyz="0 0 -1"/>
+      <limit effort="1000" lower="0" upper="0.024858" velocity="2.0"/>
     </joint>
-    <joint name="finger2_joint" type="fixed">
+    <joint name="finger2_joint" type="prismatic">
       <origin rpy="0 0 0" xyz="0 0 0.0"/>
       <parent link="robotiq_hande_base_link"/>
       <child link="finger2"/>
+      <axis xyz="0 0 1"/>
+      <limit effort="1000" lower="0" upper="0.024858" velocity="2.0"/>
+      <mimic joint="joint_finger" multiplier="1" offset="0"/>
     </joint>
   </xacro:macro>

Commit message: update hande meshes and update values accordingly

File: robotiq_hande_gripper_description/urdf/robotiq_hande.urdf.xacro (robot description, xacro)
@@ -2,38 +2,12 @@
 <robot xmlns:xacro="http://ros.org/wiki/xacro">
   <xacro:macro name="robotiq_hande"  params="prefix">
-    <link name="robotiq_adapter_link">
+    <link name="robotiq_hande_base_link">
       <inertial>
-        <origin xyz="8.625E-08 -4.6583E-06 0.03145" rpy="0 0 0" />
-        <mass value="0.22652" />
-        <inertia ixx="0.00020005" ixy="0" ixz="0" iyy="0.00017832" iyz="0" izz="0.00013478" />
+        <origin xyz="0 0 0.04607" rpy="0 0 0" />
+        <mass value="0.86387" />
+        <inertia ixx="1017560E-9" ixy="0" ixz="2235E-9" iyy="1028041E-9" iyz="0" izz="489810E-9" />
       </inertial>
       <visual>
-        <origin xyz="0 0 0" rpy="0 0 1.57" />
-        <geometry>
-          <mesh filename="package://robotiq_hande_gripper_description/meshes/hros_robotiq_adapter.dae" scale="0.001 0.001 0.001"/>
-        </geometry>
-        <material name="Gazebo/Black">
-          <color rgba="0.0 0.0 0.0 1" />
-        </material>
-      </visual>
-      <collision>
-        <origin xyz="0 0 0" rpy="0 0 1.57" />
-        <geometry>
-          <mesh filename="package://robotiq_hande_gripper_description/meshes/hros_robotiq_adapter.dae" scale="0.001 0.001 0.001"/>
-        </geometry>
-      </collision>
-    </link>
-    <gazebo reference="robotiq_adapter_link">
-      <material>Gazebo/Black</material>
-      <selfCollide>False</selfCollide>
-    </gazebo>
-    <link name="robotiq_hande_base_link">
-      <inertial>
-        <origin xyz="8.625E-08 -4.6583E-06 0.03145" rpy="0 0 0" />
-        <mass value="0.22652" />
-        <inertia ixx="0.00020005" ixy="0" ixz="0" iyy="0.00017832" iyz="0" izz="0.00013478" />
-      </inertial>
-      <visual>
-        <origin xyz="0 0 0" rpy="0 0 1.57" />
+        <origin xyz="0 0 0" rpy="0 0 0" />
         <geometry>
           <mesh filename="package://robotiq_hande_gripper_description/meshes/hand-e.dae" scale="0.001 0.001 0.001"/>
@@ -44,5 +18,5 @@
       </visual>
       <collision>
-        <origin xyz="0 0 0" rpy="0 0 1.57" />
+        <origin xyz="0 0 0" rpy="0 0 0" />
         <geometry>
           <mesh filename="package://robotiq_hande_gripper_description/meshes/hand-e.dae" scale="0.001 0.001 0.001"/>
@@ -52,14 +26,14 @@
     <gazebo reference="robotiq_hande_base_link">
       <material>Gazebo/Black</material>
-      <selfCollide>True</selfCollide>
+      <selfCollide>False</selfCollide>
     </gazebo>
-    <link name="finger1">
+    <link name="left_finger">
       <inertial>
-        <origin rpy="0 0 0" xyz="8.625E-08 -4.6583E-06 0.03145"/>
-        <mass value="0.22652"/>
-        <inertia ixx="0.00020005" ixy="0" ixz="0" iyy="0.00017832" iyz="0" izz="0.00013478"/>
+        <origin rpy="0 0 0" xyz="0.02262 -0.00759 0.00738"/>
+        <mass value="0.03804"/>
+        <inertia ixx="13567E-9" ixy="1849E-9" ixz="3622E-9" iyy="15784E-9" iyz="3616E-9" izz="7478E-9"/>
       </inertial>
       <visual>
-        <origin rpy="0 0 1.57" xyz="0 0 0"/>
+        <origin rpy="0 0 0" xyz="0 0 0"/>
         <geometry>
           <mesh filename="package://robotiq_hande_gripper_description/meshes/finger_1.dae" scale="0.001 0.001 0.001"/>
@@ -70,5 +44,5 @@
       </visual>
       <collision>
-        <origin rpy="0 0 1.57" xyz="0 0 0"/>
+        <origin rpy="0 0 0" xyz="0 0 0"/>
         <geometry>
           <mesh filename="package://robotiq_hande_gripper_description/meshes/finger_1.dae" scale="0.001 0.001 0.001"/>
@@ -76,16 +50,16 @@
       </collision>
     </link>
-    <gazebo reference="finger1">
+    <gazebo reference="left_finger">
       <material>Gazebo/Grey</material>
-      <selfCollide>True</selfCollide>
+      <selfCollide>False</selfCollide>
     </gazebo>
-    <link name="finger2">
+    <link name="right_finger">
       <inertial>
-        <origin rpy="0 0 0" xyz="8.625E-08 -4.6583E-06 0.03145"/>
-        <mass value="0.22652"/>
-        <inertia ixx="0.00020005" ixy="0" ixz="0" iyy="0.00017832" iyz="0" izz="0.00013478"/>
+        <origin rpy="0 0 0" xyz="-0.02262 0.00759 0.00738"/>
+        <mass value="0.03804"/>
+        <inertia ixx="13567E-9" ixy="1849E-9" ixz="-3622E-9" iyy="15784E-9" iyz="-3616E-9" izz="7478E-9"/>
       </inertial>
       <visual>
-        <origin rpy="0 0 1.57" xyz="0 0 0"/>
+        <origin rpy="0 0 0" xyz="0 0 0"/>
         <geometry>
           <mesh filename="package://robotiq_hande_gripper_description/meshes/finger_2.dae" scale="0.001 0.001 0.001"/>
@@ -96,5 +70,5 @@
       </visual>
       <collision>
-        <origin rpy="0 0 1.57" xyz="0 0 0"/>
+        <origin rpy="0 0 0" xyz="0 0 0"/>
         <geometry>
           <mesh filename="package://robotiq_hande_gripper_description/meshes/finger_2.dae" scale="0.001 0.001 0.001"/>
@@ -102,37 +76,39 @@
       </collision>
     </link>
-    <gazebo reference="finger2">
+    <gazebo reference="right_finger">
       <material>Gazebo/Grey</material>
-      <selfCollide>True</selfCollide>
+      <selfCollide>False</selfCollide>
     </gazebo>
+    <joint name="joint_finger" type="prismatic">
+      <origin rpy="0 0 0" xyz="0 0 0.099"/>
+      <parent link="robotiq_hande_base_link"/>
+      <child link="left_finger"/>
+      <axis xyz="-1 0 0"/>
+      <limit effort="130" lower="0" upper="0.025" velocity="0.15"/>
+    </joint>
+    <joint name="robotiq_hande_base_to_right_finger" type="prismatic">
+      <origin rpy="0 0 0" xyz="0 0 0.099"/>
+      <parent link="robotiq_hande_base_link"/>
+      <child link="right_finger"/>
+      <axis xyz="1 0 0"/>
+      <limit effort="130" lower="0" upper="0.025" velocity="0.15"/>
+      <mimic joint="joint_finger" multiplier="1" offset="0"/>
+    </joint>
     <gazebo>
       <plugin filename="librobotiq_gripper_gazebo_plugin.so" name="robotiq_hande_gripper">
-        <kp>10</kp>
+        <kp>100</kp>
         <ki>3</ki>
-        <kd>5</kd>
+        <kd>9</kd>
         <joint>joint_finger</joint>
-        <joint>finger2_joint</joint>
+        <joint>robotiq_hande_base_to_right_finger</joint>
+      </plugin>
+      <plugin filename="libgazebo_ros_joint_state_publisher.so" name="mara_joint_state">
+        <ros>
+          <argument>~/out:=joint_states</argument>
+        </ros>
+        <update_rate>25</update_rate>
+        <joint_name>joint_finger</joint_name>
       </plugin>
     </gazebo>
-    <joint name="base_adapter_to_base_robotiq_joint" type="fixed">
-      <origin rpy="0 1.57 0" xyz=" 0 0 0.10653"/>
-      <parent link="robotiq_adapter_link" />
-      <child link="robotiq_hande_base_link"/>
-    </joint>
-    <joint name="joint_finger" type="prismatic">
-      <origin rpy="0 0 0" xyz="0 0 0.0"/>
-      <parent link="robotiq_hande_base_link"/>
-      <child link="finger1"/>
-      <axis xyz="0 0 -1"/>
-      <limit effort="1000" lower="0" upper="0.024858" velocity="2.0"/>
-    </joint>
-    <joint name="finger2_joint" type="prismatic">
-      <origin rpy="0 0 0" xyz="0 0 0.0"/>
-      <parent link="robotiq_hande_base_link"/>
-      <child link="finger2"/>
-      <axis xyz="0 0 1"/>
-      <limit effort="1000" lower="0" upper="0.024858" velocity="2.0"/>
-      <mimic joint="joint_finger" multiplier="1" offset="0"/>
-    </joint>
   </xacro:macro>
 </robot>
