Commit message: Fixing URDFs

File: robotiq_140_gripper_description/urdf/robotiq_140.urdf.xacro (robot description, xacro)
@@ -34,6 +34,6 @@
         <inertia
             ixx="2.89328108496468E-06"
-            ixy="0"
-            ixz="0"
+            ixy="-1.57935047237397E-19"
+            ixz="-1.93980378593255E-19"
             iyy="1.86719750325683E-06"
             iyz="-1.21858577871576E-06"
@@ -66,6 +66,6 @@
         <inertia
             ixx="2.89328108496468E-06"
-            ixy="0"
-            ixz="0"
+            ixy="-1.57935047237397E-19"
+            ixz="-1.93980378593255E-19"
             iyy="1.86719750325683E-06"
             iyz="-1.21858577871576E-06"
@@ -149,10 +149,10 @@
         <mass value="0.0104003125914103" />
         <inertia
-            ixx="6.06863499e-06"
-            ixy="0"
-            ixz="0"
-            iyy="7.46305064e-07"
-            iyz="0"
-            izz="6.21796490e-06" />
+            ixx="2.71909453810972E-06"
+            ixy="1.35402465472579E-21"
+            ixz="-7.1817349065269E-22"
+            iyy="7.69100314106116E-07"
+            iyz="6.74715432769696E-07"
+            izz="2.30315190420171E-06" />
       </inertial>
       <visual>
@@ -181,10 +181,10 @@
         <mass value="0.0104003125914103" />
         <inertia
-            ixx="6.06863499e-06"
-            ixy="0"
-            ixz="0"
-            iyy="7.46305064e-07"
-            iyz="0"
-            izz="6.21796490e-06" />
+            ixx="2.71909453810972E-06"
+            ixy="1.35402465472579E-21"
+            ixz="-7.1817349065269E-22"
+            iyy="7.69100314106116E-07"
+            iyz="6.74715432769696E-07"
+            izz="2.30315190420171E-06" />
       </inertial>
       <visual>
@@ -277,12 +277,13 @@
       <child link="left_outer_knuckle" />
       <axis xyz="-1 0 0" />
-      <limit lower="0" upper="0.78"  velocity="2.0" effort="1000" />
-    </joint>
-    <joint name="right_outer_knuckle_joint" type="revolute">
+      <limit lower="0" upper="0.775"  velocity="2.0" effort="1000" />
+      <mimic joint="joint_finger" multiplier="1" offset="0"/>
+    </joint>
+    <joint name="joint_finger" type="revolute">
       <origin xyz="0 0.030601 0.054905" rpy="2.31 0 3.14159265359" />
       <parent link="robotiq_arg2f_base_link" />
       <child link="right_outer_knuckle" />
       <axis xyz="-1 0 0" />
-      <limit lower="0" upper="0.78" velocity="2.0" effort="1000" />
+      <limit lower="0" upper="0.775" velocity="2.0" effort="1000" />
     </joint>
     <joint name="left_inner_knuckle_joint" type="revolute">
@@ -292,4 +293,5 @@
       <axis xyz="-1 0 0" />
       <limit lower="0" upper="0.78" velocity="2.0" effort="1000" />
+      <mimic joint="joint_finger" multiplier="1" offset="0"/>
     </joint>
     <joint name="right_inner_knuckle_joint" type="revolute">
@@ -299,18 +301,15 @@
       <axis xyz="-1 0 0" />
       <limit lower="0" upper="0.78" velocity="2.0" effort="1000" />
-    </joint>
-    <joint name="left_outer_finger_joint" type="revolute">
+      <mimic joint="joint_finger" multiplier="1" offset="0"/>
+    </joint>
+    <joint name="left_outer_finger_joint" type="fixed">
       <origin xyz="0 0.01821998610742 0.0260018192872234" rpy="0 0 0" />
       <parent link="left_outer_knuckle" />
       <child link="left_outer_finger" />
-      <axis xyz="-1 0 0" />
-      <limit lower="-0.875" upper="-0.0075" velocity="2.0" effort="1000" />
-    </joint>
-    <joint name="right_outer_finger_joint" type="revolute">
+    </joint>
+    <joint name="right_outer_finger_joint" type="fixed">
       <origin xyz="0 0.01821998610742 0.0260018192872234" rpy="0 0 0" />
       <parent link="right_outer_knuckle" />
       <child link="right_outer_finger" />
-      <axis xyz="-1 0 0" />
-      <limit lower="-0.875" upper="-0.0075" velocity="2.0" effort="1000" />
     </joint>
     <joint name="left_inner_finger_joint" type="revolute">
@@ -319,5 +318,6 @@
       <child link="left_inner_finger" />
       <axis xyz="1 0 0" />
-      <limit lower="-0.875" upper="0.8757" velocity="2.0" effort="1000" />
+      <limit lower="0" upper="0.8757" velocity="2.0" effort="1000" />
+      <mimic joint="joint_finger" multiplier="1" offset="0"/>
     </joint>
     <joint name="right_inner_finger_joint" type="revolute">
@@ -326,5 +326,6 @@
       <child link="right_inner_finger" />
       <axis xyz="1 0 0" />
-      <limit lower="-0.875" upper="0.8757" velocity="2.0" effort="1000" />
+      <limit lower="0" upper="0.8757" velocity="2.0" effort="1000" />
+      <mimic joint="joint_finger" multiplier="1" offset="0"/>
     </joint>
     <gazebo>
@@ -361,5 +362,5 @@
         <left_joint>left_outer_knuckle_joint</left_joint>
         <right_joint>right_inner_knuckle_joint</right_joint>
-        <right_joint>right_outer_knuckle_joint</right_joint>
+        <right_joint>joint_finger</right_joint>
       </plugin>
     </gazebo>

File: robotiq_140_gripper_description/urdf/robotiq_140_hros_support.urdf.xacro (robot description, xacro)
@@ -308,12 +308,13 @@
       <child link="left_outer_knuckle" />
       <axis xyz="-1 0 0" />
-      <limit lower="0" upper="0.78"  velocity="2.0" effort="1000" />
-    </joint>
-    <joint name="right_outer_knuckle_joint" type="revolute">
+      <limit lower="0" upper="0.775"  velocity="2.0" effort="1000" />
+      <mimic joint="joint_finger" multiplier="1" offset="0"/>
+    </joint>
+    <joint name="joint_finger" type="revolute">
       <origin xyz="0 0.030601 0.054905" rpy="2.31 0 3.14159265359" />
       <parent link="robotiq_arg2f_base_link" />
       <child link="right_outer_knuckle" />
       <axis xyz="-1 0 0" />
-      <limit lower="0" upper="0.78" velocity="2.0" effort="1000" />
+      <limit lower="0" upper="0.775" velocity="2.0" effort="1000" />
     </joint>
     <joint name="left_inner_knuckle_joint" type="revolute">
@@ -323,4 +324,5 @@
       <axis xyz="-1 0 0" />
       <limit lower="0" upper="0.78" velocity="2.0" effort="1000" />
+      <mimic joint="joint_finger" multiplier="1" offset="0"/>
     </joint>
     <joint name="right_inner_knuckle_joint" type="revolute">
@@ -330,18 +332,15 @@
       <axis xyz="-1 0 0" />
       <limit lower="0" upper="0.78" velocity="2.0" effort="1000" />
-    </joint>
-    <joint name="left_outer_finger_joint" type="revolute">
+      <mimic joint="joint_finger" multiplier="1" offset="0"/>
+    </joint>
+    <joint name="left_outer_finger_joint" type="fixed">
       <origin xyz="0 0.01821998610742 0.0260018192872234" rpy="0 0 0" />
       <parent link="left_outer_knuckle" />
       <child link="left_outer_finger" />
-      <axis xyz="-1 0 0" />
-      <limit lower="-0.875" upper="-0.0075" velocity="2.0" effort="1000" />
-    </joint>
-    <joint name="right_outer_finger_joint" type="revolute">
+    </joint>
+    <joint name="right_outer_finger_joint" type="fixed">
       <origin xyz="0 0.01821998610742 0.0260018192872234" rpy="0 0 0" />
       <parent link="right_outer_knuckle" />
       <child link="right_outer_finger" />
-      <axis xyz="-1 0 0" />
-      <limit lower="-0.875" upper="-0.0075" velocity="2.0" effort="1000" />
     </joint>
     <joint name="left_inner_finger_joint" type="revolute">
@@ -350,5 +349,6 @@
       <child link="left_inner_finger" />
       <axis xyz="1 0 0" />
-      <limit lower="-0.875" upper="0.8757" velocity="2.0" effort="1000" />
+      <limit lower="0" upper="0.8757" velocity="2.0" effort="1000" />
+      <mimic joint="joint_finger" multiplier="1" offset="0"/>
     </joint>
     <joint name="right_inner_finger_joint" type="revolute">
@@ -357,5 +357,6 @@
       <child link="right_inner_finger" />
       <axis xyz="1 0 0" />
-      <limit lower="-0.875" upper="0.8757" velocity="2.0" effort="1000" />
+      <limit lower="0" upper="0.8757" velocity="2.0" effort="1000" />
+      <mimic joint="joint_finger" multiplier="1" offset="0"/>
     </joint>
     <gazebo>
